File: Power_Mux_12V.kicad_sch (KiCad schematic)
At the start: 11 parts, among them U4 TPS2121RUXR

Commit message: reviewnotes
Changed lines of the file:
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@@
+		)
+	)
+	(label "diode or gate instead? normal beefy shocky diode would probably be fine"
+		(at 181.61 55.88 0)
+		(effects
+			(font
+				(size 1.27 1.27)
+			)
+			(justify left bottom)
 		)
 	)
@@
 		(effects
 			(font
+				(size 1.27 1.27)
+			)
+			(justify left bottom)
+		)
+	)
+	(label "basically diode on each end of each output and then outputs are tied together"
+		(at 184.15 64.77 0)
+		(effects
+			(font

Commit message: schematic1
Other:
- note added: "basically diode on each end of each output and then outputs are tied together"
- note added: "diode or gate instead? normal beefy shocky diode would probably be fine"
Changed lines of the file:
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@@
 	(generator_version "10.0")
 	(paper "A4")
+	(text "diode or gate instead? normal beefy shocky diode would probably be fine"
+		(exclude_from_sim no)
+		(at 220.98 74.676 0)
+		(effects
+			(font
+				(size 1.27 1.27)
+			)
+		)
+	)
 	(text "Resistor Divider Settings"
 		(exclude_from_sim no)
@@
 			)
 			(justify left top)
+		)
+	)
+	(text "basically diode on each end of each output and then outputs are tied together\n"
+		(exclude_from_sim no)
+		(at 216.662 81.026 0)
+		(effects
+			(font
+				(size 1.27 1.27)
+			)
 		)
 	)
@@
 		)
 	)
-	(label "diode or gate instead? normal beefy shocky diode would probably be fine"
-		(at 181.61 55.88 0)
-		(effects
-			(font
-				(size 1.27 1.27)
-			)
-			(justify left bottom)
-		)
-	)
 	(label "CP2"
 		(at 112.395 82.55 0)
 		(effects
 			(font
-				(size 1.27 1.27)
-			)
-			(justify left bottom)
-		)
-	)
-	(label "basically diode on each end of each output and then outputs are tied together"
-		(at 184.15 64.77 0)
-		(effects
-			(font
