File: Display.kicad_sch (KiCad schematic)
At the start: 0 parts

Commit message: root2
Parts:
- added NHD-0208BZ-FSW-GBW-33V1: (no value), symbol PS-SuppCharger_Library:NHD-0208BZ-FSW-GBW-33V3
- added R46, R47, R48, R49: R, symbol Device:R
Connections:
- new net DB4: NHD-0208BZ-FSW-GBW-33V1.11 (DB4)
- new net DB5: NHD-0208BZ-FSW-GBW-33V1.12 (DB5)
- new net DB6: NHD-0208BZ-FSW-GBW-33V1.13 (DB6)
- new net DB7: NHD-0208BZ-FSW-GBW-33V1.14 (DB7)
- new net E: NHD-0208BZ-FSW-GBW-33V1.6 (E)
- new net GND: NHD-0208BZ-FSW-GBW-33V1.1 (VSS), NHD-0208BZ-FSW-GBW-33V1.K (LED-), R47.2, R49.2
- new net LED+: NHD-0208BZ-FSW-GBW-33V1.A (LED+), R48.2, R49.1
- new net RS: NHD-0208BZ-FSW-GBW-33V1.4 (RS)
- new net RW: NHD-0208BZ-FSW-GBW-33V1.5 (RW)
- new net V0: NHD-0208BZ-FSW-GBW-33V1.3 (V0), R46.2, R47.1
- new net Vin: NHD-0208BZ-FSW-GBW-33V1.2 (VDD), R46.1, R48.1

Commit message: root3
Connections:
- net LED+ renamed LED_2V9
- net LED_2V9: no longer NHD-0208BZ-FSW-GBW-33V1.A (LED+)
- net V0 renamed V0_0V1
- new net LEV_2V9: NHD-0208BZ-FSW-GBW-33V1.A (LED+)
Other:
- note added: "LED+ 2.9V Input"
- note added: "VSS 0.1V input"
Changed lines of the file:
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@@
 	(generator_version "10.0")
 	(paper "A4")
+	(text "VSS 0.1V input"
+		(exclude_from_sim no)
+		(at 112.776 115.316 0)
+		(effects
+			(font
+				(size 1.27 1.27)
+			)
+		)
+	)
+	(text "LED+ 2.9V Input"
+		(exclude_from_sim no)
+		(at 112.776 118.11 0)
+		(effects
+			(font
+				(size 1.27 1.27)
+			)
+		)
+	)
 	(junction
 		(at 91.44 91.44)
@@
 	(wire
 		(pts
-			(xy 110.49 85.09) (xy 124.46 85.09)
+			(xy 111.76 85.09) (xy 124.46 85.09)
 		)
 		(stroke
@@
 		)
 	)
-	(label "V0"
-		(at 110.49 85.09 180)
+	(label "V0_0V1"
+		(at 111.76 85.09 180)
 		(effects
 			(font
@@
 		)
 	)
-	(label "LED+"
+	(label "LEV_2V9"
 		(at 165.1 95.25 0)
 		(effects
@@
 		)
 	)
-	(label "V0"
+	(label "V0_0V1"
 		(at 72.39 91.44 0)
 		(effects
@@
 		)
 	)
-	(label "LED+"
+	(label "LED_2V9"
 		(at 93.98 91.44 0)
 		(effects

Commit message: reviewnotes
Other:
- note added: "TFT LCD Display Module Screen - 2.0in., 240x320 (SPI Interface)"
- note added: "change display and go from there:"
- note added: "highletgo display"
- note added: "stack 3 diodes to make 2.9v? cant do voltage divider"
Changed lines of the file:
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@@
 	(generator_version "10.0")
 	(paper "A4")
+	(text " TFT LCD Display Module Screen - 2.0in., 240x320 (SPI Interface) \n"
+		(exclude_from_sim no)
+		(at 131.318 154.178 0)
+		(effects
+			(font
+				(size 1.27 1.27)
+			)
+		)
+	)
+	(text "highletgo display"
+		(exclude_from_sim no)
+		(at 129.54 136.398 0)
+		(effects
+			(font
+				(size 1.27 1.27)
+			)
+		)
+	)
 	(text "VSS 0.1V input"
 		(exclude_from_sim no)
 		(at 112.776 115.316 0)
+		(effects
+			(font
+				(size 1.27 1.27)
+			)
+		)
+	)
+	(text "stack 3 diodes to make 2.9v? cant do voltage divider\n"
+		(exclude_from_sim no)
+		(at 120.65 127.254 0)
 		(effects
 			(font
@@
 		(effects
 			(font
+				(size 1.27 1.27)
+			)
+		)
+	)
+	(text "change display and go from there:"
+		(exclude_from_sim no)
+		(at 157.48 132.08 0)
+		(effects
+			(font

Commit message: schematic1
Parts:
- removed NHD-0208BZ-FSW-GBW-33V1: (no value), symbol PS-SuppCharger_Library:NHD-0208BZ-FSW-GBW-33V3
- removed R46, R47, R48, R49: R, symbol Device:R
- added C54: 0.1u, symbol Device:C
- added DS1: (no value), symbol PS-SuppCharger_Library:ZJY200S0800TG01
Connections:
- net GND: now also C54.2, DS1.1 (GND)
- net Vin: now also C54.1, DS1.2 (VCC)
- new net BLK: DS1.8 (BLK)
- new net CS: DS1.7 (CS)
- new net DC: DS1.6 (DC)
- new net RES: DS1.5 (RES)
- new net SCL: DS1.3 (SCL)
- new net SDA: DS1.4 (SDA)
Other:
- note added: "hiletgo display"
- note removed: "highletgo display"

Commit message: schematic3
Connections:
- net Vin renamed DS_Vin
Changed lines of the file:
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@@
 		)
 	)
-	(hierarchical_label "Vin"
+	(hierarchical_label "DS_Vin"
 		(shape input)
 		(at 102.87 74.93 180)

Commit message: schematic5
Parts:
- DS1: value (none) -> ZJY200S0800TG01
Other:
- note removed: "LED+ 2.9V Input"
- note removed: "VSS 0.1V input"
- note removed: "change display and go from there:"
- note removed: "hiletgo display"
- note removed: "stack 3 diodes to make 2.9v? cant do voltage divider"
Changed lines of the file:
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@@
 	(text " TFT LCD Display Module Screen - 2.0in., 240x320 (SPI Interface) \n"
 		(exclude_from_sim no)
-		(at 131.318 154.178 0)
-		(effects
-			(font
-				(size 1.27 1.27)
-			)
-		)
-	)
-	(text "hiletgo display"
-		(exclude_from_sim no)
-		(at 129.54 136.398 0)
-		(effects
-			(font
-				(size 1.27 1.27)
-			)
-		)
-	)
-	(text "VSS 0.1V input"
-		(exclude_from_sim no)
-		(at 112.776 115.316 0)
-		(effects
-			(font
-				(size 1.27 1.27)
-			)
-		)
-	)
-	(text "stack 3 diodes to make 2.9v? cant do voltage divider\n"
-		(exclude_from_sim no)
-		(at 120.65 127.254 0)
-		(effects
-			(font
-				(size 1.27 1.27)
-			)
-		)
-	)
-	(text "LED+ 2.9V Input"
-		(exclude_from_sim no)
-		(at 112.776 118.11 0)
-		(effects
-			(font
-				(size 1.27 1.27)
-			)
-		)
-	)
-	(text "change display and go from there:"
-		(exclude_from_sim no)
-		(at 157.48 132.08 0)
+		(at 128.27 100.838 0)
 		(effects
 			(font
@@
 		(in_pos_files yes)
 		(dnp no)
-		(fields_autoplaced yes)
 		(property "Reference" "DS1"
-			(at 127 64.77 0)
-			(show_name no)
-			(do_not_autoplace no)
-			(effects
-				(font
-					(size 1.27 1.27)
-				)
-			)
-		)
-		(property "Value" ""
-			(at 127 76.2 0)
+			(at 127.254 64.008 0)
+			(show_name no)
+			(do_not_autoplace no)
+			(effects
+				(font
+					(size 1.27 1.27)
+				)
+			)
+		)
+		(property "Value" "ZJY200S0800TG01"
+			(at 127.254 66.294 0)
 			(show_name no)
 			(do_not_autoplace no)
@@
 			)
 		)
-		(property "Datasheet" ""
+		(property "Datasheet" "https://cdn.sparkfun.com/assets/0/2/3/0/c/ZJY200S0800TG01.pdf"
 			(at 127 76.2 0)
 			(hide yes)

Commit message: schematic6
Parts:
- added R26: 22, symbol Device:R
Connections:
- net SDA: now also R26.1; no longer DS1.4 (SDA)
- new net: DS1.4 (SDA), R26.2
Changed lines of the file:
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@@
 	(wire
 		(pts
-			(xy 116.84 69.85) (xy 118.11 69.85)
+			(xy 115.57 69.85) (xy 118.11 69.85)
 		)
 		(stroke
@@
 	(wire
 		(pts
-			(xy 135.89 72.39) (xy 137.16 72.39)
+			(xy 102.87 69.85) (xy 107.95 69.85)
 		)
 		(stroke
@@
 		)
 	)
+	(wire
+		(pts
+			(xy 135.89 72.39) (xy 137.16 72.39)
+		)
+		(stroke
+			(width 0)
+			(type default)
+		)
+	)
 	(hierarchical_label "DC"
 		(shape input)
@@
 	(hierarchical_label "SDA"
 		(shape input)
-		(at 116.84 69.85 180)
+		(at 102.87 69.85 180)
 		(effects
 			(font
@@
 					(unit 1)
 				)
+			)
+		)
+	)
+	(symbol
+		(lib_id "Device:R")
+		(at 111.76 69.85 90)
+		(unit 1)
+		(body_style 1)
+		(exclude_from_sim no)
+		(in_bom yes)
+		(on_board yes)
+		(in_pos_files yes)
+		(dnp no)
+		(property "Reference" "R26"
+			(at 111.76 65.278 90)
+			(show_name no)
+			(do_not_autoplace no)
+			(effects
+				(font
+					(size 1.27 1.27)
+				)
+			)
+		)
+		(property "Value" "22"
+			(at 111.76 67.31 90)
+			(show_name no)
+			(do_not_autoplace no)
+			(effects
+				(font
+					(size 1.27 1.27)
+				)
+			)
+		)
+		(property "Footprint" ""
+			(at 111.76 71.628 90)
+			(hide yes)
+			(show_name no)
+			(do_not_autoplace no)
+			(effects
+				(font
+					(size 1.27 1.27)
+				)
+			)
+		)
+		(property "Datasheet" ""
+			(at 111.76 69.85 0)
+			(hide yes)
+			(show_name no)
+			(do_not_autoplace no)
+			(effects
+				(font
+					(size 1.27 1.27)
+				)
+			)
+		)
+		(property "Description" "Resistor"
+			(at 111.76 69.85 0)
+			(hide yes)
+			(show_name no)
+			(do_not_autoplace no)
+			(effects
+				(font
+					(size 1.27 1.27)
+				)
+			)
+		)
+		(pin "1"
+		)
+		(pin "2"
+		)
+		(instances
+			(project "PS-SuppChargerPCB"
+				(path "/bb6ce8fd-e1af-464e-bfef-c3b4f18a2cee/a0f50f41-4e30-4c40-9c76-1d295d27d660"
+					(reference "R26")
+					(unit 1)
+				)

Commit message: schematic7
Other:
- moved on the sheet: C54, DS1, R26
