File: Display.kicad_sch (KiCad schematic)
At the start: 3 parts

Commit message: schematic10
Other:
- moved on the sheet: C54, R26
Changed lines of the file:
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@@
 	(generator "eeschema")
 	(generator_version "10.0")
-	(paper "A4")
+	(paper "A5")
 	(text " TFT LCD Display Module Screen - 2.0in., 240x320 (SPI Interface) \n"
 		(exclude_from_sim no)
-		(at 88.646 95.504 0)
+		(at 110.236 54.864 0)
 		(effects
 			(font
@@
 	)
 	(junction
-		(at 72.39 76.2)
+		(at 93.98 35.56)
 		(diameter 0)
 		(color 0 0 0 0)
 	)
 	(junction
-		(at 72.39 83.82)
+		(at 93.98 43.18)
 		(diameter 0)
 		(color 0 0 0 0)
@@
 	(wire
 		(pts
-			(xy 77.47 73.66) (xy 78.74 73.66)
+			(xy 99.06 33.02) (xy 100.33 33.02)
 		)
 		(stroke
@@
 	(wire
 		(pts
-			(xy 63.5 83.82) (xy 72.39 83.82)
+			(xy 85.09 43.18) (xy 93.98 43.18)
 		)
 		(stroke
@@
 	(wire
 		(pts
-			(xy 96.52 76.2) (xy 97.79 76.2)
+			(xy 118.11 35.56) (xy 119.38 35.56)
 		)
 		(stroke
@@
 	(wire
 		(pts
-			(xy 63.5 76.2) (xy 72.39 76.2)
+			(xy 85.09 35.56) (xy 93.98 35.56)
 		)
 		(stroke
@@
 	(wire
 		(pts
-			(xy 72.39 76.2) (xy 78.74 76.2)
+			(xy 93.98 35.56) (xy 100.33 35.56)
 		)
 		(stroke
@@
 	(wire
 		(pts
-			(xy 72.39 83.82) (xy 78.74 83.82)
+			(xy 93.98 43.18) (xy 100.33 43.18)
 		)
 		(stroke
@@
 	(wire
 		(pts
-			(xy 96.52 78.74) (xy 97.79 78.74)
+			(xy 118.11 38.1) (xy 119.38 38.1)
 		)
 		(stroke
@@
 	(wire
 		(pts
-			(xy 76.2 71.12) (xy 78.74 71.12)
+			(xy 97.79 30.48) (xy 100.33 30.48)
 		)
 		(stroke
@@
 	(wire
 		(pts
-			(xy 96.52 71.12) (xy 97.79 71.12)
+			(xy 118.11 30.48) (xy 119.38 30.48)
 		)
 		(stroke
@@
 	(wire
 		(pts
-			(xy 63.5 71.12) (xy 68.58 71.12)
+			(xy 85.09 30.48) (xy 90.17 30.48)
 		)
 		(stroke
@@
 	(wire
 		(pts
-			(xy 96.52 73.66) (xy 97.79 73.66)
+			(xy 118.11 33.02) (xy 119.38 33.02)
 		)
 		(stroke
@@
 	)
 	(image
-		(at 213.36 137.16)
-		(scale 0.208967)
+		(at 149.86 78.74)
+		(scale 0.188656)
 		(data "iVBORw0KGgoAAAANSUhEUgAACGYAAAQuCAYAAACUWKk1AAAMTGlDQ1BJQ0MgUHJvZmlsZQAASImV"
 			"VwdYU1cbPndkQggQiICMsJcgIiOAjBBWANlbVEISIIwYE4KKGymtYN0ighOtgihYrYAUF2pdFMW9"
@@
 	)
 	(image
-		(at 93.98 137.16)
-		(scale 0.422028)
+		(at 62.23 78.74)
+		(scale 0.289272)
 		(data "iVBORw0KGgoAAAANSUhEUgAABvgAAAIYCAYAAACov+vjAAAMTGlDQ1BJQ0MgUHJvZmlsZQAASImV"
 			"VwdYU1cbPndkQggQiICMsJcgIiOAjBBWANlbVEISIIwYE4KKGymtYN0ighOtgihYrYAUF2pdFMW9"
@@
 	(hierarchical_label "DC"
 		(shape input)
-		(at 97.79 76.2 0)
+		(at 119.38 35.56 0)
 		(effects
 			(font
@@
 	(hierarchical_label "CS"
 		(shape input)
-		(at 97.79 73.66 0)
+		(at 119.38 33.02 0)
 		(effects
 			(font
@@
 	(hierarchical_label "DS_Vin"
 		(shape input)
-		(at 63.5 76.2 180)
+		(at 85.09 35.56 180)
 		(effects
 			(font
@@
 	(hierarchical_label "GND"
 		(shape input)
-		(at 63.5 83.82 180)
+		(at 85.09 43.18 180)
 		(effects
 			(font
@@
 	(hierarchical_label "RES"
 		(shape input)
-		(at 97.79 78.74 0)
+		(at 119.38 38.1 0)
 		(effects
 			(font
@@
 	(hierarchical_label "BLK"
 		(shape input)
-		(at 97.79 71.12 0)
+		(at 119.38 30.48 0)
 		(effects
 			(font
@@
 	(hierarchical_label "SDA"
 		(shape input)
-		(at 63.5 71.12 180)
+		(at 85.09 30.48 180)
 		(effects
 			(font
@@
 	(hierarchical_label "SCL"
 		(shape input)
-		(at 77.47 73.66 180)
+		(at 99.06 33.02 180)
 		(effects
 			(font
@@
 	(symbol
 		(lib_id "Device:C")
-		(at 72.39 80.01 0)
+		(at 93.98 39.37 0)
 		(unit 1)
 		(body_style 1)
@@
 		(dnp no)
 		(property "Reference" "C54"
-			(at 65.786 78.994 0)
+			(at 87.376 38.354 0)
 			(show_name no)
 			(do_not_autoplace no)
@@
 		)
 		(property "Value" "0.1u"
-			(at 65.786 80.772 0)
+			(at 87.376 40.132 0)
 			(show_name no)
 			(do_not_autoplace no)
@@
 		)
 		(property "Footprint" ""
-			(at 73.3552 83.82 0)
+			(at 94.9452 43.18 0)
 			(hide yes)
 			(show_name no)
@@
 		)
 		(property "Datasheet" ""
-			(at 72.39 80.01 0)
+			(at 93.98 39.37 0)
 			(hide yes)
 			(show_name no)
@@
 		)
 		(property "Description" "Unpolarized capacitor"
-			(at 72.39 80.01 0)
+			(at 93.98 39.37 0)
 			(hide yes)
 			(show_name no)
@@
 	(symbol
 		(lib_id "PS-SuppCharger_Library:ZJY200S0800TG01")
-		(at 87.63 77.47 0)
+		(at 109.22 36.83 0)
 		(unit 1)
 		(body_style 1)
@@
 		(dnp no)
 		(property "Reference" "DS1"
-			(at 87.884 65.278 0)
+			(at 109.474 24.638 0)
 			(show_name no)
 			(do_not_autoplace no)
@@
 		)
 		(property "Value" "ZJY200S0800TG01"
-			(at 87.884 67.564 0)
+			(at 109.474 26.924 0)
 			(show_name no)
 			(do_not_autoplace no)
@@
 		)
 		(property "Footprint" ""
-			(at 87.63 77.47 0)
+			(at 109.22 36.83 0)
 			(hide yes)
 			(show_name no)
@@
 			)
 		)
-		(property "Datasheet" "kicad-embed://ZJY200S0800TG01.pdf"
-			(at 87.63 77.47 0)
+		(property "Datasheet" "https://cdn.sparkfun.com/assets/0/2/3/0/c/ZJY200S0800TG01.pdf"
+			(at 109.22 36.83 0)
 			(hide yes)
 			(show_name no)
@@
 		)
 		(property "Description" ""
-			(at 87.63 77.47 0)
+			(at 109.22 36.83 0)
 			(hide yes)
 			(show_name no)
@@
 	(symbol
 		(lib_id "Device:R")
-		(at 72.39 71.12 90)
+		(at 93.98 30.48 90)
 		(unit 1)
 		(body_style 1)
@@
 		(dnp no)
 		(property "Reference" "R26"
-			(at 72.39 66.548 90)
+			(at 93.98 25.908 90)
 			(show_name no)
 			(do_not_autoplace no)
@@
 		)
 		(property "Value" "22"
-			(at 72.39 68.58 90)
+			(at 93.98 27.94 90)
 			(show_name no)
 			(do_not_autoplace no)
@@
 		)
 		(property "Footprint" ""
-			(at 72.39 72.898 90)
+			(at 93.98 32.258 90)
 			(hide yes)
 			(show_name no)
@@
 		)
 		(property "Datasheet" ""
-			(at 72.39 71.12 0)
+			(at 93.98 30.48 0)
 			(hide yes)
 			(show_name no)
@@
 		)
 		(property "Description" "Resistor"
-			(at 72.39 71.12 0)
+			(at 93.98 30.48 0)
 			(hide yes)
 			(show_name no)

Commit message: halleffectsense
Parts:
- renumbered C54 to C47, R26 to R49
Changed lines of the file:
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@@
 		(in_pos_files yes)
 		(dnp no)
-		(property "Reference" "C54"
+		(property "Reference" "C47"
 			(at 87.376 38.354 0)
 			(show_name no)
@@
 			(project "PS-SuppChargerPCB"
 				(path "/bb6ce8fd-e1af-464e-bfef-c3b4f18a2cee/62959a0d-7d46-4ab6-879a-37e4e873f375"
-					(reference "C54")
+					(reference "C47")
 					(unit 1)
 				)
@@
 		(in_pos_files yes)
 		(dnp no)
-		(property "Reference" "R26"
+		(property "Reference" "R49"
 			(at 93.98 25.908 90)
 			(show_name no)
@@
 			(project "PS-SuppChargerPCB"
 				(path "/bb6ce8fd-e1af-464e-bfef-c3b4f18a2cee/62959a0d-7d46-4ab6-879a-37e4e873f375"
-					(reference "R26")
+					(reference "R49")
 					(unit 1)
 				)

Commit message: footprints1
Parts:
- C45: renamed from C47; footprint (none) -> Capacitor_SMD:C_0603_1608Metric_Pad1.08x0.95mm_HandSolder
- R48: renamed from R49; footprint (none) -> Resistor_SMD:R_0603_1608Metric_Pad0.98x0.95mm_HandSolder
Changed lines of the file:
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@@
 		(in_pos_files yes)
 		(dnp no)
-		(property "Reference" "C47"
+		(property "Reference" "C45"
 			(at 87.376 38.354 0)
 			(show_name no)
@@
 			)
 		)
-		(property "Footprint" ""
+		(property "Footprint" "Capacitor_SMD:C_0603_1608Metric_Pad1.08x0.95mm_HandSolder"
 			(at 94.9452 43.18 0)
 			(hide yes)
@@
 			(project "PS-SuppChargerPCB"
 				(path "/bb6ce8fd-e1af-464e-bfef-c3b4f18a2cee/62959a0d-7d46-4ab6-879a-37e4e873f375"
-					(reference "C47")
+					(reference "C45")
 					(unit 1)
 				)
@@
 		(in_pos_files yes)
 		(dnp no)
-		(property "Reference" "R49"
+		(property "Reference" "R48"
 			(at 93.98 25.908 90)
 			(show_name no)
@@
 			)
 		)
-		(property "Footprint" ""
+		(property "Footprint" "Resistor_SMD:R_0603_1608Metric_Pad0.98x0.95mm_HandSolder"
 			(at 93.98 32.258 90)
 			(hide yes)
@@
 			(project "PS-SuppChargerPCB"
 				(path "/bb6ce8fd-e1af-464e-bfef-c3b4f18a2cee/62959a0d-7d46-4ab6-879a-37e4e873f375"
-					(reference "R49")
+					(reference "R48")
 					(unit 1)
 				)

Commit message: layout0
Parts:
- DS1: footprint (none) -> PS-Supp-Footprints:ZJY200S0800TG01
Changed lines of the file:
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@@
 			)
 		)
-		(property "Footprint" ""
+		(property "Footprint" "PS-Supp-Footprints:ZJY200S0800TG01"
 			(at 109.22 36.83 0)
 			(hide yes)

Commit message: layout1
Parts:
- C45, R48: KiLib_Generator (none) -> SMD_2terminal_chip_molded
Changed lines of the file:
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@@
+			)
+		)
+		(property "KiLib_Generator" "SMD_2terminal_chip_molded"
+			(at 93.98 39.37 0)
+			(hide yes)
+			(show_name no)
+			(do_not_autoplace no)
+			(effects
+				(font
+					(size 1.27 1.27)
+				)
 			)
 		)
@@
 			(at 93.98 30.48 0)
 			(hide yes)
+			(show_name no)
+			(do_not_autoplace no)
+			(effects
+				(font
+					(size 1.27 1.27)
+				)
+			)
+		)
+		(property "KiLib_Generator" "SMD_2terminal_chip_molded"
+			(at 93.98 30.48 0)
+			(hide yes)
