File: PowerSupply.kicad_sch (KiCad schematic)
At the start: 0 parts

Commit message: reviewnotes
Other:
- note added: "make them bananajacks in footprint"
- note added: "two one by one connectors"
Changed lines of the file:
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@@
 	(generator_version "10.0")
 	(paper "A4")
+	(text "make them bananajacks in footprint"
+		(exclude_from_sim no)
+		(at 116.332 46.482 0)
+		(effects
+			(font
+				(size 1.27 1.27)
+			)
+		)
+	)
+	(text "two one by one connectors\n"
+		(exclude_from_sim no)
+		(at 117.094 33.274 0)
+		(effects
+			(font
+				(size 1.27 1.27)
+			)
+		)
+	)
 )

Commit message: schematic1
Parts:
- added J5: PS_Banana_+, symbol Connector_Generic:Conn_01x01
- added J6: PS_Banana_-, symbol Connector_Generic:Conn_01x01
Connections:
- new net GND: J6.1 (Pin_1)
- new net Vout: J5.1 (Pin_1)
Changed lines of the file:
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@@
 	(text "two one by one connectors\n"
 		(exclude_from_sim no)
-		(at 117.094 33.274 0)
+		(at 116.078 43.18 0)
 		(effects
 			(font
@@
 			)
 		)
+	)
+	(wire
+		(pts
+			(xy 88.9 78.74) (xy 92.71 78.74)
+		)
+		(stroke
+			(width 0)
+			(type default)
+		)
+	)
+	(wire
+		(pts
+			(xy 88.9 69.85) (xy 92.71 69.85)
+		)
+		(stroke
+			(width 0)
+			(type default)
+		)
+	)
+	(hierarchical_label "GND"
+		(shape input)
+		(at 88.9 78.74 180)
+		(effects
+			(font
+				(size 1.27 1.27)
+			)
+			(justify right)
+		)
+	)
+	(hierarchical_label "Vout"
+		(shape output)
+		(at 88.9 69.85 180)
+		(effects
+			(font
+				(size 1.27 1.27)
+			)
+			(justify right)
+		)
+	)
+	(symbol
+		(lib_id "Connector_Generic:Conn_01x01")
+		(at 97.79 78.74 0)
+		(unit 1)
+		(body_style 1)
+		(exclude_from_sim no)
+		(in_bom yes)
+		(on_board yes)
+		(in_pos_files yes)
+		(dnp no)
+		(fields_autoplaced yes)
+		(property "Reference" "J6"
+			(at 100.33 77.4699 0)
+			(show_name no)
+			(do_not_autoplace no)
+			(effects
+				(font
+					(size 1.27 1.27)
+				)
+				(justify left)
+			)
+		)
+		(property "Value" "PS_Banana_-"
+			(at 100.33 80.0099 0)
+			(show_name no)
+			(do_not_autoplace no)
+			(effects
+				(font
+					(size 1.27 1.27)
+				)
+				(justify left)
+			)
+		)
+		(property "Footprint" ""
+			(at 97.79 78.74 0)
+			(hide yes)
+			(show_name no)
+			(do_not_autoplace no)
+			(effects
+				(font
+					(size 1.27 1.27)
+				)
+			)
+		)
+		(property "Datasheet" ""
+			(at 97.79 78.74 0)
+			(hide yes)
+			(show_name no)
+			(do_not_autoplace no)
+			(effects
+				(font
+					(size 1.27 1.27)
+				)
+			)
+		)
+		(property "Description" "Generic connector, single row, 01x01, script generated (kicad-library-utils/schlib/autogen/connector/)"
+			(at 97.79 78.74 0)
+			(hide yes)
+			(show_name no)
+			(do_not_autoplace no)
+			(effects
+				(font
+					(size 1.27 1.27)
+				)
+			)
+		)
+		(pin "1"
+		)
+		(instances
+			(project "PS-SuppChargerPCB"
+				(path "/bb6ce8fd-e1af-464e-bfef-c3b4f18a2cee/b453130c-e9c7-412e-8bc8-36da0f20a61a"
+					(reference "J6")
+					(unit 1)
+				)
+			)
+		)
+	)
+	(symbol
+		(lib_id "Connector_Generic:Conn_01x01")
+		(at 97.79 69.85 0)
+		(unit 1)
+		(body_style 1)
+		(exclude_from_sim no)
+		(in_bom yes)
+		(on_board yes)
+		(in_pos_files yes)
+		(dnp no)
+		(fields_autoplaced yes)
+		(property "Reference" "J5"
+			(at 100.33 68.5799 0)
+			(show_name no)
+			(do_not_autoplace no)
+			(effects
+				(font
+					(size 1.27 1.27)
+				)
+				(justify left)
+			)
+		)
+		(property "Value" "PS_Banana_+"
+			(at 100.33 71.1199 0)
+			(show_name no)
+			(do_not_autoplace no)
+			(effects
+				(font
+					(size 1.27 1.27)
+				)
+				(justify left)
+			)
+		)
+		(property "Footprint" ""
+			(at 97.79 69.85 0)
+			(hide yes)
+			(show_name no)
+			(do_not_autoplace no)
+			(effects
+				(font
+					(size 1.27 1.27)
+				)
+			)
+		)
+		(property "Datasheet" ""
+			(at 97.79 69.85 0)
+			(hide yes)
+			(show_name no)
+			(do_not_autoplace no)
+			(effects
+				(font
+					(size 1.27 1.27)
+				)
+			)
+		)
+		(property "Description" "Generic connector, single row, 01x01, script generated (kicad-library-utils/schlib/autogen/connector/)"
+			(at 97.79 69.85 0)
+			(hide yes)
+			(show_name no)
+			(do_not_autoplace no)
+			(effects
+				(font
+					(size 1.27 1.27)
+				)
+			)
+		)
+		(pin "1"
+		)
+		(instances
+			(project "PS-SuppChargerPCB"
+				(path "/bb6ce8fd-e1af-464e-bfef-c3b4f18a2cee/b453130c-e9c7-412e-8bc8-36da0f20a61a"
+					(reference "J5")
+					(unit 1)
+				)
+			)
+		)

Commit message: schematic2
Connections:
- net Vout renamed PS_Vout
Changed lines of the file:
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@@
 		)
 	)
-	(hierarchical_label "Vout"
+	(hierarchical_label "PS_Vout"
 		(shape output)
 		(at 88.9 69.85 180)

Commit message: schematic6
Other:
- moved on the sheet: J5
Changed lines of the file:
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@@
 	(wire
 		(pts
-			(xy 88.9 69.85) (xy 92.71 69.85)
+			(xy 88.9 73.66) (xy 92.71 73.66)
 		)
 		(stroke
@@
 	(hierarchical_label "PS_Vout"
 		(shape output)
-		(at 88.9 69.85 180)
+		(at 88.9 73.66 180)
 		(effects
 			(font
@@
 	(symbol
 		(lib_id "Connector_Generic:Conn_01x01")
-		(at 97.79 69.85 0)
+		(at 97.79 73.66 0)
 		(unit 1)
 		(body_style 1)
@@
 		(fields_autoplaced yes)
 		(property "Reference" "J5"
-			(at 100.33 68.5799 0)
+			(at 100.33 72.3899 0)
 			(show_name no)
 			(do_not_autoplace no)
@@
 		)
 		(property "Value" "PS_Banana_+"
-			(at 100.33 71.1199 0)
+			(at 100.33 74.9299 0)
 			(show_name no)
 			(do_not_autoplace no)
@@
 		)
 		(property "Footprint" ""
-			(at 97.79 69.85 0)
+			(at 97.79 73.66 0)
 			(hide yes)
 			(show_name no)
@@
 		)
 		(property "Datasheet" ""
-			(at 97.79 69.85 0)
+			(at 97.79 73.66 0)
 			(hide yes)
 			(show_name no)
@@
 		)
 		(property "Description" "Generic connector, single row, 01x01, script generated (kicad-library-utils/schlib/autogen/connector/)"
-			(at 97.79 69.85 0)
+			(at 97.79 73.66 0)
 			(hide yes)
 			(show_name no)

Commit message: schematicrev1
Parts:
- added C34, C61, C62: 0.1u, Capacitor_SMD:C_0603_1608Metric_Pad1.08x0.95mm_HandSolder, symbol Device:C
- added C47: 1u, Capacitor_SMD:C_0603_1608Metric_Pad1.08x0.95mm_HandSolder, symbol Device:C
- added C58: 220n, Capacitor_SMD:C_0603_1608Metric_Pad1.08x0.95mm_HandSolder, symbol Device:C
- added C59: 10n, Capacitor_SMD:C_0603_1608Metric_Pad1.08x0.95mm_HandSolder, symbol ECE319H:C
- added C60: 10u, Capacitor_SMD:C_0805_2012Metric_Pad1.18x1.45mm_HandSolder, symbol Device:C
- added D13: SMBJ15CA, Diode_SMD:D_SMB, symbol lhrs_power:SMBJ15CA
- added D14: SMAF4758A, LHRS_Passives:SODFL5026X125N, symbol lhrs_power:SMAF4758A
- added IC3: LM74502DDFR, LHRS_Power:LM74502DDFR, symbol lhrs_power:LM74502HDDFR
- added J7: CarLVPowerConnector, LHRS_Connectors:Molex_Nano-Fit_105309-xx02_1x02_P2.50mm_Vertical, symbol lhrs_connectors:CarLVPowerConnector
- added Q4, Q5: PSMN012-100YS, Package_TO_SOT_SMD:LFPAK56, symbol lhrs_power:PSMN012-100YS
- added R29: 10k, Resistor_SMD:R_0603_1608Metric_Pad0.98x0.95mm_HandSolder, symbol Device:R_US
- added R30: 33, Resistor_SMD:R_0603_1608Metric_Pad0.98x0.95mm_HandSolder, symbol Device:R_US
- added R35, R43: 100k, Resistor_SMD:R_0603_1608Metric_Pad0.98x0.95mm_HandSolder, symbol Device:R_US
- added R36: 7.32k, Resistor_SMD:R_0603_1608Metric_Pad0.98x0.95mm_HandSolder, symbol Device:R_US
- added R44: 15.8k, Resistor_SMD:R_0603_1608Metric_Pad0.98x0.95mm_HandSolder, symbol Device:R_US
Connections:
- net GND: now also C34.2, C47.1, C59.2, C60.2, C61.2, C62.2, D13.1 (A1), D14.2 (A), IC3.2 (GND), J7.2 (GND), R36.2, R44.1
- net PS_Vout: now also C34.1, D13.2 (A2), J7.1 (+24V), Q4.5, R29.2, R35.1, R43.1
- new net: C47.2, C58.1, D14.1 (K), IC3.5 (VS), R29.1
- new net: C58.2, IC3.4 (VCAP)
- new net: C59.1, R30.1
- new net EN/UVLO: C62.1, IC3.1 (EN/UVLO), R43.2, R44.2
- new net OV: C61.1, IC3.7 (OV), R35.2, R36.1
- new net PP_Vout: C60.1, Q5.5
- new net gate: IC3.6 (GATE), Q4.4, Q5.4, R30.2
- new net source: IC3.8 (SRC), Q4.1, Q4.2, Q4.3, Q5.1, Q5.2, Q5.3
Other:
- note added: "4.84ms = 75us + 220nF * 6.5V/300uA 6.5V recommended on datasheet 4.84ms power up delay"
- note added: "Kell Harpole"
- note added: "Make them bananajacks in footprint"
- note added: "Output of Python Calulations for Resistor Values"
- note added: "Two one by one connectors"
- note removed: "make them bananajacks in footprint"
- note removed: "two one by one connectors"
- moved on the sheet: J5, J6

Commit message: schematic7
Parts:
- removed J5: PS_Banana_+, symbol Connector_Generic:Conn_01x01
- removed J6: PS_Banana_-, symbol Connector_Generic:Conn_01x01
- removed J7: CarLVPowerConnector, LHRS_Connectors:Molex_Nano-Fit_105309-xx02_1x02_P2.50mm_Vertical, symbol lhrs_connectors:CarLVPowerConnector
Connections:
- net PS_Vout: no longer C34.1, D13.2 (A2), Q4.5, R29.2
- new net Vin: C34.1, D13.2 (A2), Q4.5, R29.2
