File: 12VBuckBoost.kicad_sch (KiCad schematic)
At the start: 21 parts, among them IC2 TPS552872RYQR

Commit message: root3
Changed lines of the file:
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@@
 		(fields_autoplaced yes)
 		(property "Reference" "IC2"
-			(at 147.32 46.736 0)
+			(at 150.7333 73.66 0)
 			(show_name no)
 			(do_not_autoplace no)
@@
 					(size 1.27 1.27)
 				)
+				(justify left)
 			)
 		)
 		(property "Value" "TPS552872RYQR"
-			(at 147.32 49.276 0)
+			(at 150.7333 76.2 0)
 			(show_name no)
 			(do_not_autoplace no)
@@
 					(size 1.27 1.27)
 				)
+				(justify left)
 			)
 		)

Commit message: reviewnotes
Other:
- note added: "look at bps leader"
Changed lines of the file:
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@@
+		)
+	)
+	(text "look at bps leader"
+		(exclude_from_sim no)
+		(at 43.688 23.876 0)
+		(effects
+			(font
+				(size 1.27 1.27)
+			)
 		)
 	)

Commit message: schematic2
Other:
- note removed: "look at bps leader"
Changed lines of the file:
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@@
 		)
 	)
-	(text "look at bps leader"
-		(exclude_from_sim no)
-		(at 43.688 23.876 0)
-		(effects
-			(font
-				(size 1.27 1.27)
-			)
-		)
-	)
 	(text "C4"
 		(exclude_from_sim no)
@@
 	(wire
 		(pts
+			(xy 18.524 0.8257) (xy 19.794 0.8257)
+		)
+		(stroke
+			(width 0)
+			(type default)
+		)
+	)
+	(wire
+		(pts
+			(xy 2.6162 2.6162) (xy 3.8862 2.6162)
+		)
+		(stroke
+			(width 0)
+			(type default)
+		)
+	)
+	(wire
+		(pts
 			(xy 96.52 55.88) (xy 120.65 55.88)
 		)
@@
 		)
 	)
+	(label "12V_MUX_OUT"
+		(at 13.444 2.0957 180)
+		(effects
+			(font
+				(size 1.27 1.27)
+			)
+			(justify right bottom)
+		)
+	)

Commit message: schematic5
Changed lines of the file:
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@@
 	(wire
 		(pts
-			(xy 18.524 0.8257) (xy 19.794 0.8257)
-		)
-		(stroke
-			(width 0)
-			(type default)
-		)
-	)
-	(wire
-		(pts
-			(xy 2.6162 2.6162) (xy 3.8862 2.6162)
-		)
-		(stroke
-			(width 0)
-			(type default)
-		)
-	)
-	(wire
-		(pts
 			(xy 96.52 55.88) (xy 120.65 55.88)
 		)
@@
 		)
 	)
-	(label "12V_MUX_OUT"
-		(at 13.444 2.0957 180)
-		(effects
-			(font
-				(size 1.27 1.27)
-			)
-			(justify right bottom)
-		)
-	)

Commit message: schematic6
Changed lines of the file:
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@@
 	)
 	(hierarchical_label "VOUT"
-		(shape input)
+		(shape output)
 		(at 243.84 35.56 0)
 		(effects

Commit message: schematic7
Parts:
- IC2: footprint TPS552892QWRYQRQ1 -> LHRS_ICs:TPS552892QWRYQRQ1
Changed lines of the file:
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@@
 			)
 		)
-		(property "Footprint" "TPS552892QWRYQRQ1"
+		(property "Footprint" "LHRS_ICs:TPS552892QWRYQRQ1"
 			(at 154.94 130.48 0)
 			(hide yes)

Commit message: fixedsharepoint
Parts:
- IC1: renamed from IC2; footprint LHRS_ICs:TPS552892QWRYQRQ1 -> TPS552892QWRYQRQ1; Height 1 -> (none); Manufacturer_Name Texas Instruments -> (none); Manufacturer_Part_Number TPS552872RYQR -> (none); Mouser Part Number 595-TPS552872RYQR -> (none); Mouser Price/Stock https://www.mouser.co.uk/ProductDetail/Texas-Instruments/TP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 -> (none); P/N (none) -> TPS552872RYQR
- renumbered C35 to C1, C36 to C2, C37 to C3, C44 to C35, C45 to C36, C46 to C37, C38 to C4, C39 to C5, C40 to C6, C41 to C7, C42 to C8, C43 to C9, R37 to R1, R38 to R2, R39 to R3, R40 to R4, R41 to R5, R42 to R6

Commit message: schematic9
Parts:
- IC1: footprint TPS552892QWRYQRQ1 -> LHRS_ICs:TPS552892QWRYQRQ1
Changed lines of the file:
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@@
 			)
 		)
-		(property "Footprint" "TPS552892QWRYQRQ1"
+		(property "Footprint" "LHRS_ICs:TPS552892QWRYQRQ1"
 			(at 154.94 130.48 0)
 			(hide yes)
