File: CurrentVoltageSensing.kicad_sch (KiCad schematic)
At the start: 0 parts

Commit message: root2
Parts:
- added C47: 100n, Capacitor_SMD:C_0603_1608Metric_Pad1.08x0.95mm_HandSolder, symbol Device:C_Small
- added C48: 47n, Capacitor_SMD:C_0603_1608Metric_Pad1.08x0.95mm_HandSolder, symbol Device:C_Small
- added C49: 0.1u, Capacitor_SMD:C_0603_1608Metric_Pad1.08x0.95mm_HandSolder, symbol Device:C_Small
- added R43: 10k, Resistor_SMD:R_0603_1608Metric_Pad0.98x0.95mm_HandSolder, symbol Device:R
- added R44: 1k, Resistor_SMD:R_0603_1608Metric_Pad0.98x0.95mm_HandSolder, symbol Device:R
- added R45: 4.7k, Resistor_SMD:R_0603_1608Metric_Pad0.98x0.95mm_HandSolder, symbol Device:R
- added U5: TMCS1107A2UQDR, OBBB Footprints:TMCS1107A3BQDR, symbol OBBB Symbols:TMCS1107A3BQDR
Connections:
- new net: R45.1, U5.7 (VOUT)
- new net I_ADC: C48.1, R45.2
- new net LV_GND: C47.2, C48.2, C49.1, R44.2, U5.5 (GND), U5.6 (NC)
- new net SENSE_IN: R43.1, U5.1 (IN+), U5.2 (IN+)
- new net SENSE_OUT: U5.3 (IN-), U5.4 (IN-)
- new net VS: C49.2, U5.8 (VS)
- new net V_ADC: C47.1, R43.2, R44.1
Other:
- note added: "Divider of 11 Max SuppReg Voltage = 25, divided = 2.27V Min supp Voltage = 23.9, divided = 2.27V"
- note added: "TMCS1107A2U 100 mV/A, V_OUT = 0.33V + 0.1 × I Range: −2.8A to 27.7A"
- note added: "Use a 10× probe or a DMM"
- note added: "place close to VS pin Low ESR"
- note added: "use 1% resistors for dividers"

Commit message: reviewnotes
Other:
- note added: "make it non isolated"
Changed lines of the file:
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@@
+		)
+	)
+	(text "make it non isolated"
+		(exclude_from_sim no)
+		(at 214.376 113.03 0)
+		(effects
+			(font
+				(size 1.27 1.27)
+			)
 		)
 	)
@@
 		)
 	)
+	(label "look at bps leader"
+		(at 205.74 109.22 0)
+		(effects
+			(font
+				(size 1.27 1.27)
+			)
+			(justify left bottom)
+		)
+	)

Commit message: schematic2
Parts:
- renumbered C47 to C34, C48 to C47, C49 to C48, R43 to R28, R44 to R29, R45 to R30, U5 to U4
Other:
- note added: "look at bps leader"
Changed lines of the file:
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@@
+		)
+	)
+	(text "look at bps leader"
+		(exclude_from_sim no)
+		(at 223.774 103.378 0)
+		(effects
+			(font
+				(size 1.27 1.27)
+			)
 		)
 	)
@@
 			(width 0)
 			(type default)
-		)
-	)
-	(label "look at bps leader"
-		(at 205.74 109.22 0)
-		(effects
-			(font
-				(size 1.27 1.27)
-			)
-			(justify left bottom)
 		)
 	)
@@
 		(in_pos_files yes)
 		(dnp no)
-		(property "Reference" "R44"
+		(property "Reference" "R29"
 			(at 96.52 87.6299 0)
 			(show_name no)
@@
 		(instances
 			(project "PS-SuppChargerPCB"
-				(path "/bb6ce8fd-e1af-464e-bfef-c3b4f18a2cee/8d46c906-880b-4ae9-bef9-10e6557421b5"
-					(reference "R44")
+				(path "/bb6ce8fd-e1af-464e-bfef-c3b4f18a2cee/7814c951-9095-4f8d-9e56-f938c21b373e"
+					(reference "R29")
 					(unit 1)
 				)
@@
 		(in_pos_files yes)
 		(dnp no)
-		(property "Reference" "R45"
+		(property "Reference" "R30"
 			(at 161.036 77.216 0)
 			(show_name no)
@@
 		(instances
 			(project "PS-SuppChargerPCB"
-				(path "/bb6ce8fd-e1af-464e-bfef-c3b4f18a2cee/8d46c906-880b-4ae9-bef9-10e6557421b5"
-					(reference "R45")
+				(path "/bb6ce8fd-e1af-464e-bfef-c3b4f18a2cee/7814c951-9095-4f8d-9e56-f938c21b373e"
+					(reference "R30")
 					(unit 1)
 				)
@@
 		(in_pos_files yes)
 		(dnp no)
-		(property "Reference" "R43"
+		(property "Reference" "R28"
 			(at 96.52 74.9299 0)
 			(show_name no)
@@
 		(instances
 			(project "PS-SuppChargerPCB"
-				(path "/bb6ce8fd-e1af-464e-bfef-c3b4f18a2cee/8d46c906-880b-4ae9-bef9-10e6557421b5"
-					(reference "R43")
+				(path "/bb6ce8fd-e1af-464e-bfef-c3b4f18a2cee/7814c951-9095-4f8d-9e56-f938c21b373e"
+					(reference "R28")
 					(unit 1)
 				)
@@
 		(in_pos_files yes)
 		(dnp no)
-		(property "Reference" "C47"
+		(property "Reference" "C34"
 			(at 82.55 87.6362 0)
 			(show_name no)
@@
 		(instances
 			(project "PS-SuppChargerPCB"
-				(path "/bb6ce8fd-e1af-464e-bfef-c3b4f18a2cee/8d46c906-880b-4ae9-bef9-10e6557421b5"
-					(reference "C47")
+				(path "/bb6ce8fd-e1af-464e-bfef-c3b4f18a2cee/7814c951-9095-4f8d-9e56-f938c21b373e"
+					(reference "C34")
 					(unit 1)
 				)
@@
 		(in_pos_files yes)
 		(dnp no)
-		(property "Reference" "C48"
+		(property "Reference" "C47"
 			(at 158.75 88.9062 0)
 			(show_name no)
@@
 		(instances
 			(project "PS-SuppChargerPCB"
-				(path "/bb6ce8fd-e1af-464e-bfef-c3b4f18a2cee/8d46c906-880b-4ae9-bef9-10e6557421b5"
-					(reference "C48")
+				(path "/bb6ce8fd-e1af-464e-bfef-c3b4f18a2cee/7814c951-9095-4f8d-9e56-f938c21b373e"
+					(reference "C47")
 					(unit 1)
 				)
@@
 		(in_pos_files yes)
 		(dnp no)
-		(property "Reference" "C49"
+		(property "Reference" "C48"
 			(at 178.308 77.724 0)
 			(show_name no)
@@
 		(instances
 			(project "PS-SuppChargerPCB"
-				(path "/bb6ce8fd-e1af-464e-bfef-c3b4f18a2cee/8d46c906-880b-4ae9-bef9-10e6557421b5"
-					(reference "C49")
+				(path "/bb6ce8fd-e1af-464e-bfef-c3b4f18a2cee/7814c951-9095-4f8d-9e56-f938c21b373e"
+					(reference "C48")
 					(unit 1)
 				)
@@
 		(dnp no)
 		(fields_autoplaced yes)
-		(property "Reference" "U5"
+		(property "Reference" "U4"
 			(at 129.54 58.42 0)
 			(show_name no)
@@
 		(instances
 			(project "PS-SuppChargerPCB"
-				(path "/bb6ce8fd-e1af-464e-bfef-c3b4f18a2cee/8d46c906-880b-4ae9-bef9-10e6557421b5"
-					(reference "U5")
+				(path "/bb6ce8fd-e1af-464e-bfef-c3b4f18a2cee/7814c951-9095-4f8d-9e56-f938c21b373e"
+					(reference "U4")
 					(unit 1)
 				)

Commit message: schematic3
Parts:
- removed C34: 100n, Capacitor_SMD:C_0603_1608Metric_Pad1.08x0.95mm_HandSolder, symbol Device:C_Small
- removed C47: 47n, Capacitor_SMD:C_0603_1608Metric_Pad1.08x0.95mm_HandSolder, symbol Device:C_Small
- removed R28: 10k, Resistor_SMD:R_0603_1608Metric_Pad0.98x0.95mm_HandSolder, symbol Device:R
- removed R29: 1k, Resistor_SMD:R_0603_1608Metric_Pad0.98x0.95mm_HandSolder, symbol Device:R
- removed R30: 4.7k, Resistor_SMD:R_0603_1608Metric_Pad0.98x0.95mm_HandSolder, symbol Device:R
- removed U4: TMCS1107A2UQDR, OBBB Footprints:TMCS1107A3BQDR, symbol OBBB Symbols:TMCS1107A3BQDR
- added C49: 100n, Capacitor_SMD:C_0603_1608Metric_Pad1.08x0.95mm_HandSolder, symbol Device:C_Small
- added C56: 47n, Capacitor_SMD:C_0603_1608Metric_Pad1.08x0.95mm_HandSolder, symbol Device:C_Small
- added R31: 10k, Resistor_SMD:R_0603_1608Metric_Pad0.98x0.95mm_HandSolder, symbol Device:R
- added R32: 1k, Resistor_SMD:R_0603_1608Metric_Pad0.98x0.95mm_HandSolder, symbol Device:R
- added R33: 4.7k, Resistor_SMD:R_0603_1608Metric_Pad0.98x0.95mm_HandSolder, symbol Device:R
- added U5: TMCS1170, symbol PS-SuppCharger_Library:TMCS1170
Connections:
- net I_ADC: now also C56.1, R33.2
- net SENSE_IN: now also R31.1, U5.1 (IN+), U5.2 (IN+)
- net SENSE_OUT: now also U5.3 (IN-), U5.4 (IN-)
- net VS: now also U5.12 (VS)
- net V_ADC: now also C49.1, R31.2, R32.1
- net LV_GND renamed CV_GND
- net CV_GND: now also C49.2, C56.2, R32.2, U5.10 (NC), U5.7 (NC), U5.8 (NC), U5.9 (NC)
- new net CV_GNDA: U5.5 (GND)
- new net VOUT: R33.1, U5.11 (VOUT)
- no-connect marks 0 -> 1
Other:
- note added: "Divider of 11 Max SuppReg Voltage = 14.7, divided = 2.27V Min supp Voltage = 12, divided = 2.27V"
- note removed: "Divider of 11 Max SuppReg Voltage = 25, divided = 2.27V Min supp Voltage = 23.9, divided = 2.27V"
- note removed: "TMCS1107A2U 100 mV/A, V_OUT = 0.33V + 0.1 × I Range: −2.8A to 27.7A"
- note removed: "Use a 10× probe or a DMM"
- note removed: "look at bps leader"
- note removed: "make it non isolated"
- note removed: "use 1% resistors for dividers"
- moved on the sheet: C48

Commit message: schematic6
Parts:
- added C57: 47n, Capacitor_SMD:C_0603_1608Metric_Pad1.08x0.95mm_HandSolder, symbol Device:C_Small
- added R34: 4.7k, Resistor_SMD:R_0603_1608Metric_Pad0.98x0.95mm_HandSolder, symbol Device:R
- C49: value 100n -> 0.1u
Connections:
- net CV_GND: now also C57.2
- net V_ADC: now also C57.1, R34.2; no longer C49.1, R31.2, R32.1
- new net: C49.1, R31.2, R32.1, R34.1
Other:
- note added: "Divider of 11 Max SuppReg Voltage = 14.7, divided = --V Min supp Voltage = 9.8 , divided = --V"
- note removed: "Divider of 11 Max SuppReg Voltage = 14.7, divided = 2.27V Min supp Voltage = 12, divided = 2.27V"
- moved on the sheet: C49, C56, R31, R32, R33

Commit message: schematicrev1
Parts:
- R32: value 1k -> 2.2k
Other:
- note added: "Divider of ~5.5454 -> (1/(2.2/2.2+10)) Max SuppReg Voltage = 15V, divided = 2.705V Min supp Voltage = 9.8, divided = 1.767V"
- note removed: "Divider of 11 Max SuppReg Voltage = 14.7, divided = --V Min supp Voltage = 9.8 , divided = --V"
Changed lines of the file:
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@@
 		)
 	)
-	(text "Divider of 11\nMax SuppReg Voltage = 14.7, divided = --V\nMin supp Voltage = 9.8\n, divided = --V"
+	(text "Divider of ~5.5454 -> (1/(2.2/2.2+10))\nMax SuppReg Voltage = 15V, divided = 2.705V\nMin supp Voltage = 9.8, divided = 1.767V"
 		(exclude_from_sim no)
-		(at 49.276 112.776 0)
+		(at 49.276 112.268 0)
 		(effects
 			(font
@@
 			)
 		)
-		(property "Value" "1k"
+		(property "Value" "2.2k"
 			(at 55.88 95.2499 0)
 			(show_name no)

Commit message: schematic7
Other:
- note added: "Cuttoff Frequency fc = 1/(2πRC) = 720.48Hz"
- note added: "Divider of ~5.5454 -> (1/(2.2/2.2+10)) Max SuppReg Voltage = 15V, divided = 2.705V Min supp Voltage = 9.8, divided = 1.767V Cuttoff Frequency fc = 1/(2πRC) = 720.48Hz"
- note removed: "Divider of ~5.5454 -> (1/(2.2/2.2+10)) Max SuppReg Voltage = 15V, divided = 2.705V Min supp Voltage = 9.8, divided = 1.767V"
Changed lines of the file:
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@@
 		)
 	)
-	(text "Divider of ~5.5454 -> (1/(2.2/2.2+10))\nMax SuppReg Voltage = 15V, divided = 2.705V\nMin supp Voltage = 9.8, divided = 1.767V"
+	(text "Divider of ~5.5454 -> (1/(2.2/2.2+10))\nMax SuppReg Voltage = 15V, divided = 2.705V\nMin supp Voltage = 9.8, divided = 1.767V\n\nCuttoff Frequency\nfc = 1/(2πRC) = 720.48Hz"
 		(exclude_from_sim no)
-		(at 49.276 112.268 0)
+		(at 49.276 113.284 0)
+		(effects
+			(font
+				(size 1.27 1.27)
+			)
+			(justify left)
+		)
+	)
+	(text "Cuttoff Frequency\nfc = 1/(2πRC) = 720.48Hz"
+		(exclude_from_sim no)
+		(at 184.15 104.394 0)
 		(effects
 			(font
@@
 			)
 		)
-		(property "Datasheet" "https://www.ti.com/lit/ds/symlink/tmcs1170.pdf?ts=1791411836090&ref_url=https%253A%252F%252Fwww.ti.com%252Fproduct%252FTMCS1170"
+		(property "Datasheet" "kicad-embed://TMCS1170.pdf"
 			(at 143.51 83.82 0)
 			(hide yes)

Commit message: schematic10
Other:
- moved on the sheet: C48, C49, C56, C57, R31, R32, R33, R34, U5
