File: CurrentVoltageSensing.kicad_sch (KiCad schematic)
At the start: 9 parts, among them U5 TMCS1170

Commit message: halleffectsense
Parts:
- renumbered C49 to C31, C57 to C32, C48 to C33, C56 to C34, R31 to R42, R32 to R43, R34 to R44, R33 to R45, U5 to U1
Changed lines of the file:
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@@
 		(dnp no)
 		(fields_autoplaced yes)
-		(property "Reference" "U5"
+		(property "Reference" "U1"
 			(at 116.84 45.72 0)
 			(show_name no)
@@
 			(project "PS-SuppChargerPCB"
 				(path "/bb6ce8fd-e1af-464e-bfef-c3b4f18a2cee/7814c951-9095-4f8d-9e56-f938c21b373e"
-					(reference "U5")
+					(reference "U1")
 					(unit 1)
 				)
@@
 		(in_pos_files yes)
 		(dnp no)
-		(property "Reference" "C49"
+		(property "Reference" "C31"
 			(at 43.18 66.0462 0)
 			(show_name no)
@@
 			(project "PS-SuppChargerPCB"
 				(path "/bb6ce8fd-e1af-464e-bfef-c3b4f18a2cee/7814c951-9095-4f8d-9e56-f938c21b373e"
-					(reference "C49")
+					(reference "C31")
 					(unit 1)
 				)
@@
 		(in_pos_files yes)
 		(dnp no)
-		(property "Reference" "C56"
+		(property "Reference" "C34"
 			(at 168.91 62.2362 0)
 			(show_name no)
@@
 			(project "PS-SuppChargerPCB"
 				(path "/bb6ce8fd-e1af-464e-bfef-c3b4f18a2cee/7814c951-9095-4f8d-9e56-f938c21b373e"
-					(reference "C56")
+					(reference "C34")
 					(unit 1)
 				)
@@
 		(in_pos_files yes)
 		(dnp no)
-		(property "Reference" "R31"
+		(property "Reference" "R42"
 			(at 29.21 53.3399 0)
 			(show_name no)
@@
 			(project "PS-SuppChargerPCB"
 				(path "/bb6ce8fd-e1af-464e-bfef-c3b4f18a2cee/7814c951-9095-4f8d-9e56-f938c21b373e"
-					(reference "R31")
+					(reference "R42")
 					(unit 1)
 				)
@@
 		(in_pos_files yes)
 		(dnp no)
-		(property "Reference" "C57"
+		(property "Reference" "C32"
 			(at 63.5 63.5062 0)
 			(show_name no)
@@
 			(project "PS-SuppChargerPCB"
 				(path "/bb6ce8fd-e1af-464e-bfef-c3b4f18a2cee/7814c951-9095-4f8d-9e56-f938c21b373e"
-					(reference "C57")
+					(reference "C32")
 					(unit 1)
 				)
@@
 		(in_pos_files yes)
 		(dnp no)
-		(property "Reference" "R34"
+		(property "Reference" "R44"
 			(at 54.356 55.118 90)
 			(show_name no)
@@
 			(project "PS-SuppChargerPCB"
 				(path "/bb6ce8fd-e1af-464e-bfef-c3b4f18a2cee/7814c951-9095-4f8d-9e56-f938c21b373e"
-					(reference "R34")
+					(reference "R44")
 					(unit 1)
 				)
@@
 		(in_pos_files yes)
 		(dnp no)
-		(property "Reference" "R33"
+		(property "Reference" "R45"
 			(at 159.766 53.848 90)
 			(show_name no)
@@
 			(project "PS-SuppChargerPCB"
 				(path "/bb6ce8fd-e1af-464e-bfef-c3b4f18a2cee/7814c951-9095-4f8d-9e56-f938c21b373e"
-					(reference "R33")
+					(reference "R45")
 					(unit 1)
 				)
@@
 		(in_pos_files yes)
 		(dnp no)
-		(property "Reference" "R32"
+		(property "Reference" "R43"
 			(at 29.21 66.0399 0)
 			(show_name no)
@@
 			(project "PS-SuppChargerPCB"
 				(path "/bb6ce8fd-e1af-464e-bfef-c3b4f18a2cee/7814c951-9095-4f8d-9e56-f938c21b373e"
-					(reference "R32")
+					(reference "R43")
 					(unit 1)
 				)
@@
 		(in_pos_files yes)
 		(dnp no)
-		(property "Reference" "C48"
+		(property "Reference" "C33"
 			(at 132.588 65.024 0)
 			(show_name no)
@@
 			(project "PS-SuppChargerPCB"
 				(path "/bb6ce8fd-e1af-464e-bfef-c3b4f18a2cee/7814c951-9095-4f8d-9e56-f938c21b373e"
-					(reference "C48")
+					(reference "C33")
 					(unit 1)
 				)

Commit message: newcvsense
Parts:
- removed C31, C33: 0.1u, Capacitor_SMD:C_0603_1608Metric_Pad1.08x0.95mm_HandSolder, symbol Device:C_Small
- removed C32, C34: 47n, Capacitor_SMD:C_0603_1608Metric_Pad1.08x0.95mm_HandSolder, symbol Device:C_Small
- removed R43: 2.2k, Resistor_SMD:R_0603_1608Metric_Pad0.98x0.95mm_HandSolder, symbol Device:R
- removed R44, R45: 4.7k, Resistor_SMD:R_0603_1608Metric_Pad0.98x0.95mm_HandSolder, symbol Device:R
- removed U1: TMCS1170, symbol PS-SuppCharger_Library:TMCS1170
- added C63: 0.1u, symbol Device:C
- added R65: 20m, symbol Device:R_Shunt
- added R66, R67: 10, symbol Device:R
- added U7: INA226AIDGST, Package_SO:TSSOP-10_3x3mm_P0.5mm, symbol Sensor_Energy:INA226
- R42: footprint Resistor_SMD:R_0603_1608Metric_Pad0.98x0.95mm_HandSolder -> (none); Assemble -- mixed values -- -> (none); LCSC P/N C25804 -> (none); Mouser Part Number -- mixed values -- -> (none); P/N -- mixed values -- -> (none)
Connections:
- net SENSE_IN: now also R65.1; no longer R42.1
- net SENSE_OUT: now also R65.4, U7.8 (Vbus)
- net INA_ALERT: now reaches R42.2
- net INA_ALERT: now also U7.3 (~{Alert})
- new net: R65.2, R66.2
- new net: R65.3, R67.2
- new net +3V3: R42.1, U7.6 (VS)
- new net GND: U7.1 (A1), U7.2 (A0), U7.7 (GND)
- new net INA_SCL: U7.5 (SCL)
- new net INA_SDA: U7.4 (SDA)
- new net Vin+: C63.1, R66.1, U7.10 (Vin+)
- new net Vin-: C63.2, R67.1, U7.9 (Vin-)
- no-connect marks 1 -> 0
Other:
- note added: "Alert Pullup"
- note removed: "Cuttoff Frequency fc = 1/(2πRC) = 720.48Hz"
- note removed: "Divider of ~5.5454 -> (1/(2.2/2.2+10)) Max SuppReg Voltage = 15V, divided = 2.705V Min supp Voltage = 9.8, divided = 1.767V Cuttoff Frequency fc = 1/(2πRC) = 720.48Hz"
- note removed: "place close to VS pin Low ESR"

Commit message: shuntschem2
Parts:
- added C64: 0.1u, symbol Device:C
- R65: value 20m -> 2m
Connections:
- net +3V3: now also C64.1
- net GND: now also C64.2
Other:
- note added: "Bypass Cap"
- moved on the sheet: C63, R42, R65, R66, R67, U7

Commit message: shuntschem3
Other:
- note added: "Address Pins and Target Address A1 <- GND A2 <- GND Target address: 1000000"
- moved on the sheet: C63, C64, R42, R65, R66, R67, U7

Commit message: footprints1
Parts:
- C31: renamed from C63; footprint (none) -> Capacitor_SMD:C_0603_1608Metric_Pad1.08x0.95mm_HandSolder
- C32: renamed from C64; footprint (none) -> Capacitor_SMD:C_0603_1608Metric_Pad1.08x0.95mm_HandSolder
- R41: renamed from R65; footprint (none) -> PS-Supp-Footprints:PSR100KTQFJ2L00_ROM
- R42: renamed from R66; footprint (none) -> Resistor_SMD:R_0603_1608Metric_Pad0.98x0.95mm_HandSolder
- R43: renamed from R67; footprint (none) -> Resistor_SMD:R_0603_1608Metric_Pad0.98x0.95mm_HandSolder
- R44: renamed from R42; footprint (none) -> Resistor_SMD:R_0603_1608Metric_Pad0.98x0.95mm_HandSolder
- renumbered U7 to U1
Changed lines of the file:
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@@
 		(in_pos_files yes)
 		(dnp no)
-		(property "Reference" "C64"
+		(property "Reference" "C32"
 			(at 237.744 69.85 0)
 			(show_name no)
@@
 			)
 		)
-		(property "Footprint" ""
+		(property "Footprint" "Capacitor_SMD:C_0603_1608Metric_Pad1.08x0.95mm_HandSolder"
 			(at 235.9152 74.93 0)
 			(hide yes)
@@
 			(project "PS-SuppChargerPCB"
 				(path "/bb6ce8fd-e1af-464e-bfef-c3b4f18a2cee/7814c951-9095-4f8d-9e56-f938c21b373e"
-					(reference "C64")
+					(reference "C32")
 					(unit 1)
 				)
@@
 		(dnp no)
 		(fields_autoplaced yes)
-		(property "Reference" "U7"
+		(property "Reference" "U1"
 			(at 153.2733 43.18 0)
 			(show_name no)
@@
 			(project "PS-SuppChargerPCB"
 				(path "/bb6ce8fd-e1af-464e-bfef-c3b4f18a2cee/7814c951-9095-4f8d-9e56-f938c21b373e"
-					(reference "U7")
+					(reference "U1")
 					(unit 1)
 				)
@@
 		(in_pos_files yes)
 		(dnp no)
-		(property "Reference" "C63"
+		(property "Reference" "C31"
 			(at 92.964 58.42 0)
 			(show_name no)
@@
 			)
 		)
-		(property "Footprint" ""
+		(property "Footprint" "Capacitor_SMD:C_0603_1608Metric_Pad1.08x0.95mm_HandSolder"
 			(at 91.1352 63.5 0)
 			(hide yes)
@@
 			(project "PS-SuppChargerPCB"
 				(path "/bb6ce8fd-e1af-464e-bfef-c3b4f18a2cee/7814c951-9095-4f8d-9e56-f938c21b373e"
-					(reference "C63")
+					(reference "C31")
 					(unit 1)
 				)
@@
 		(dnp no)
 		(fields_autoplaced yes)
-		(property "Reference" "R65"
+		(property "Reference" "R41"
 			(at 67.31 58.4199 0)
 			(show_name no)
@@
 			)
 		)
-		(property "Footprint" ""
+		(property "Footprint" "PS-Supp-Footprints:PSR100KTQFJ2L00_ROM"
 			(at 68.072 59.69 90)
 			(hide yes)
@@
 			(project "PS-SuppChargerPCB"
 				(path "/bb6ce8fd-e1af-464e-bfef-c3b4f18a2cee/7814c951-9095-4f8d-9e56-f938c21b373e"
-					(reference "R65")
+					(reference "R41")
 					(unit 1)
 				)
@@
 		(in_pos_files yes)
 		(dnp no)
-		(property "Reference" "R67"
+		(property "Reference" "R43"
 			(at 82.55 66.04 90)
 			(show_name no)
@@
 			)
 		)
-		(property "Footprint" ""
+		(property "Footprint" "Resistor_SMD:R_0603_1608Metric_Pad0.98x0.95mm_HandSolder"
 			(at 82.55 65.278 90)
 			(hide yes)
@@
 			(project "PS-SuppChargerPCB"
 				(path "/bb6ce8fd-e1af-464e-bfef-c3b4f18a2cee/7814c951-9095-4f8d-9e56-f938c21b373e"
-					(reference "R67")
+					(reference "R43")
 					(unit 1)
 				)
@@
 		(in_pos_files yes)
 		(dnp no)
-		(property "Reference" "R66"
+		(property "Reference" "R42"
 			(at 82.55 52.07 90)
 			(show_name no)
@@
 			)
 		)
-		(property "Footprint" ""
+		(property "Footprint" "Resistor_SMD:R_0603_1608Metric_Pad0.98x0.95mm_HandSolder"
 			(at 82.55 57.658 90)
 			(hide yes)
@@
 			(project "PS-SuppChargerPCB"
 				(path "/bb6ce8fd-e1af-464e-bfef-c3b4f18a2cee/7814c951-9095-4f8d-9e56-f938c21b373e"
-					(reference "R66")
+					(reference "R42")
 					(unit 1)
 				)
@@
 		(dnp no)
 		(fields_autoplaced yes)
-		(property "Reference" "R42"
+		(property "Reference" "R44"
 			(at 240.03 39.3699 0)
 			(show_name no)
@@
 			)
 		)
-		(property "Footprint" ""
+		(property "Footprint" "Resistor_SMD:R_0603_1608Metric_Pad0.98x0.95mm_HandSolder"
 			(at 235.712 40.64 90)
 			(hide yes)
@@
 			(project "PS-SuppChargerPCB"
 				(path "/bb6ce8fd-e1af-464e-bfef-c3b4f18a2cee/7814c951-9095-4f8d-9e56-f938c21b373e"
-					(reference "R42")
-					(unit 1)
-				)
+					(reference "R44")
+					(unit 1)
+				)

Commit message: layout1
Parts:
- removed R41: 2m, PS-Supp-Footprints:PSR100KTQFJ2L00_ROM, symbol Device:R_Shunt
- added R41: 10m, PS-Supp-Footprints:PSR100KTQFJ2L00_ROM, symbol Device:R
- C31, C32, R42, R43, R44: KiLib_Generator (none) -> SMD_2terminal_chip_molded
- U1: KiLib_Generator (none) -> package/gullwing
Connections:
- net SENSE_IN: now also R42.2, R41.1
- net SENSE_OUT: now also R43.2, R41.2
Other:
- note added: "Shunt Input Voltage: Shunt Resistance = 10m Max Current = 3A Max Shunt Input Voltage = 10m * 3A = 30mv -81.9175 < 30mV < 81.9175"
- moved on the sheet: C31, R42, R43

Commit message: alayout2
Parts:
- R41: footprint PS-Supp-Footprints:PSR100KTQFJ2L00_ROM -> PS-Supp-Footprints:PMR100HZPFU10L0
Changed lines of the file:
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@@
 			)
 		)
-		(property "Footprint" "PS-Supp-Footprints:PSR100KTQFJ2L00_ROM"
+		(property "Footprint" "PS-Supp-Footprints:PMR100HZPFU10L0"
 			(at 71.628 58.42 90)
 			(hide yes)
