File: 48PinMCU.kicad_sch (KiCad schematic)
At the start: 34 parts, among them J1 SWD_Header, J2 SWD, SW1 Reset, SW2 SW_SPDT, U2 STM32G473CETx, Y1 Crystal

Commit message: fixedsharepoint
Parts:
- C18, C20, C21, C22, C23, C24, C25, C26, C27, C28, C29: Mouser Part Number MLASH168SB7104KTNA01 -> (none)
- C19: Mouser Part Number 08055D475KAT4A -> (none)
- D5: MANUFACTURER Everlight -> (none)
- D6: Color Blue -> (none); Mouser P/N 771-PESD15VL1BA-T/R -> (none)
- J1: LSCS P/N C17492485 -> (none)
- R12: renamed from R19; Mouser Part Number CRCW060310K0FKEI -> (none)
- R18: renamed from R24; Mouser Part Number CRCW060310K0FKEI -> (none)
- SW1: Mouser Part Number 612-TL3365AF180QG -> (none)
- renumbered R18 to R11, R20 to R13, R21 to R14, R22 to R16, R23 to R17, R25 to R19

Commit message: halleffectsense
Parts:
- renumbered C16 to C48, C17 to C49, C18 to C50, C19 to C51, C20 to C52, C21 to C53, C22 to C54, C23 to C55, C24 to C56, C25 to C57, C26 to C58, C27 to C59, C28 to C60, C29 to C61, C30 to C62, D5 to D22, D6 to D23, D7 to D24, J2 to J10, J1 to J9, R11 to R50, R12 to R51, R13 to R52, R14 to R53, R16 to R54, R17 to R55, R18 to R56, R19 to R57, U2 to U5
