File: 48PinMCU.kicad_sch (KiCad schematic)
At the start: 34 parts, among them J10 SWD, J9 SWD_Header, SW1 Reset, SW2 SW_SPDT, U5 STM32G473CETx, Y1 Crystal

Commit message: footprints1
Parts:
- renumbered C48 to C46, C49 to C47, C50 to C48, C51 to C49, C52 to C50, C53 to C51, C54 to C52, C55 to C53, C56 to C54, C57 to C55, C58 to C56, C59 to C57, C60 to C58, C61 to C59, C62 to C60, D22 to D23, D23 to D24, D24 to D25, R50 to R49, R51 to R50, R52 to R51, R53 to R52, R54 to R53, R55 to R54, R56 to R55, R57 to R56
Changed lines of the file:
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@@
 		(dnp no)
 		(fields_autoplaced yes)
-		(property "Reference" "C56"
+		(property "Reference" "C54"
 			(at 204.597 57.4039 0)
 			(show_name no)
@@
 			(project "PS-SuppChargerPCB"
 				(path "/bb6ce8fd-e1af-464e-bfef-c3b4f18a2cee/a08c0d72-2b4d-4df5-af0e-616f80f6e7bf/dc00c9b9-366d-4632-b955-a9cb4062bc78"
-					(reference "C56")
+					(reference "C54")
 					(unit 1)
 				)
@@
 		(in_pos_files yes)
 		(dnp no)
-		(property "Reference" "R52"
+		(property "Reference" "R51"
 			(at 183.388 154.686 0)
 			(show_name no)
@@
 			(project "PS-SuppChargerPCB"
 				(path "/bb6ce8fd-e1af-464e-bfef-c3b4f18a2cee/a08c0d72-2b4d-4df5-af0e-616f80f6e7bf/dc00c9b9-366d-4632-b955-a9cb4062bc78"
-					(reference "R52")
+					(reference "R51")
 					(unit 1)
 				)
@@
 		(dnp no)
 		(fields_autoplaced yes)
-		(property "Reference" "R51"
+		(property "Reference" "R50"
 			(at 180.848 96.0119 0)
 			(show_name no)
@@
 			(project "PS-SuppChargerPCB"
 				(path "/bb6ce8fd-e1af-464e-bfef-c3b4f18a2cee/a08c0d72-2b4d-4df5-af0e-616f80f6e7bf/dc00c9b9-366d-4632-b955-a9cb4062bc78"
-					(reference "R51")
+					(reference "R50")
 					(unit 1)
 				)
@@
 		(dnp no)
 		(fields_autoplaced yes)
-		(property "Reference" "D23"
+		(property "Reference" "D24"
 			(at 238.76 101.5999 90)
 			(show_name no)
@@
 			(project "PS-SuppChargerPCB"
 				(path "/bb6ce8fd-e1af-464e-bfef-c3b4f18a2cee/a08c0d72-2b4d-4df5-af0e-616f80f6e7bf/dc00c9b9-366d-4632-b955-a9cb4062bc78"
-					(reference "D23")
+					(reference "D24")
 					(unit 1)
 				)
@@
 		(in_pos_files yes)
 		(dnp no)
-		(property "Reference" "C61"
+		(property "Reference" "C59"
 			(at 247.142 32.258 0)
 			(show_name no)
@@
 			(project "PS-SuppChargerPCB"
 				(path "/bb6ce8fd-e1af-464e-bfef-c3b4f18a2cee/a08c0d72-2b4d-4df5-af0e-616f80f6e7bf/dc00c9b9-366d-4632-b955-a9cb4062bc78"
-					(reference "C61")
+					(reference "C59")
 					(unit 1)
 				)
@@
 		(dnp no)
 		(fields_autoplaced yes)
-		(property "Reference" "C54"
+		(property "Reference" "C52"
 			(at 189.992 57.4039 0)
 			(show_name no)
@@
 			(project "PS-SuppChargerPCB"
 				(path "/bb6ce8fd-e1af-464e-bfef-c3b4f18a2cee/a08c0d72-2b4d-4df5-af0e-616f80f6e7bf/dc00c9b9-366d-4632-b955-a9cb4062bc78"
-					(reference "C54")
+					(reference "C52")
 					(unit 1)
 				)
@@
 		(in_pos_files yes)
 		(dnp no)
-		(property "Reference" "C53"
+		(property "Reference" "C51"
 			(at 185.166 33.02 0)
 			(show_name no)
@@
 			(project "PS-SuppChargerPCB"
 				(path "/bb6ce8fd-e1af-464e-bfef-c3b4f18a2cee/a08c0d72-2b4d-4df5-af0e-616f80f6e7bf/dc00c9b9-366d-4632-b955-a9cb4062bc78"
-					(reference "C53")
+					(reference "C51")
 					(unit 1)
 				)
@@
 		(dnp no)
 		(fields_autoplaced yes)
-		(property "Reference" "C50"
+		(property "Reference" "C48"
 			(at 174.752 57.4039 0)
 			(show_name no)
@@
 			(project "PS-SuppChargerPCB"
 				(path "/bb6ce8fd-e1af-464e-bfef-c3b4f18a2cee/a08c0d72-2b4d-4df5-af0e-616f80f6e7bf/dc00c9b9-366d-4632-b955-a9cb4062bc78"
-					(reference "C50")
+					(reference "C48")
 					(unit 1)
 				)
@@
 		(dnp no)
 		(fields_autoplaced yes)
-		(property "Reference" "C62"
+		(property "Reference" "C60"
 			(at 257.937 57.277 0)
 			(show_name no)
@@
 			(project "PS-SuppChargerPCB"
 				(path "/bb6ce8fd-e1af-464e-bfef-c3b4f18a2cee/a08c0d72-2b4d-4df5-af0e-616f80f6e7bf/dc00c9b9-366d-4632-b955-a9cb4062bc78"
-					(reference "C62")
+					(reference "C60")
 					(unit 1)
 				)
@@
 		(in_pos_files yes)
 		(dnp no)
-		(property "Reference" "C57"
+		(property "Reference" "C55"
 			(at 210.82 32.766 0)
 			(show_name no)
@@
 			(project "PS-SuppChargerPCB"
 				(path "/bb6ce8fd-e1af-464e-bfef-c3b4f18a2cee/a08c0d72-2b4d-4df5-af0e-616f80f6e7bf/dc00c9b9-366d-4632-b955-a9cb4062bc78"
-					(reference "C57")
+					(reference "C55")
 					(unit 1)
 				)
@@
 		(dnp no)
 		(fields_autoplaced yes)
-		(property "Reference" "C59"
+		(property "Reference" "C57"
 			(at 224.028 33.0199 0)
 			(show_name no)
@@
 			(project "PS-SuppChargerPCB"
 				(path "/bb6ce8fd-e1af-464e-bfef-c3b4f18a2cee/a08c0d72-2b4d-4df5-af0e-616f80f6e7bf/dc00c9b9-366d-4632-b955-a9cb4062bc78"
-					(reference "C59")
+					(reference "C57")
 					(unit 1)
 				)
@@
 		(dnp no)
 		(fields_autoplaced yes)
-		(property "Reference" "D22"
+		(property "Reference" "D23"
 			(at 194.31 142.2399 90)
 			(show_name no)
@@
 			(project "PS-SuppChargerPCB"
 				(path "/bb6ce8fd-e1af-464e-bfef-c3b4f18a2cee/a08c0d72-2b4d-4df5-af0e-616f80f6e7bf/dc00c9b9-366d-4632-b955-a9cb4062bc78"
-					(reference "D22")
+					(reference "D23")
 					(unit 1)
 				)
@@
 		(in_pos_files yes)
 		(dnp no)
-		(property "Reference" "R53"
+		(property "Reference" "R52"
 			(at 191.008 154.686 0)
 			(show_name no)
@@
 			(project "PS-SuppChargerPCB"
 				(path "/bb6ce8fd-e1af-464e-bfef-c3b4f18a2cee/a08c0d72-2b4d-4df5-af0e-616f80f6e7bf/dc00c9b9-366d-4632-b955-a9cb4062bc78"
-					(reference "R53")
+					(reference "R52")
 					(unit 1)
 				)
@@
 		(in_pos_files yes)
 		(dnp no)
-		(property "Reference" "R57"
+		(property "Reference" "R56"
 			(at 259.588 110.236 0)
 			(show_name no)
@@
 			(project "PS-SuppChargerPCB"
 				(path "/bb6ce8fd-e1af-464e-bfef-c3b4f18a2cee/a08c0d72-2b4d-4df5-af0e-616f80f6e7bf/dc00c9b9-366d-4632-b955-a9cb4062bc78"
-					(reference "R57")
+					(reference "R56")
 					(unit 1)
 				)
@@
 		(in_pos_files yes)
 		(dnp no)
-		(property "Reference" "C48"
+		(property "Reference" "C46"
 			(at 34.544 39.624 90)
 			(show_name no)
@@
 			(project "PS-SuppChargerPCB"
 				(path "/bb6ce8fd-e1af-464e-bfef-c3b4f18a2cee/a08c0d72-2b4d-4df5-af0e-616f80f6e7bf/dc00c9b9-366d-4632-b955-a9cb4062bc78"
-					(reference "C48")
+					(reference "C46")
 					(unit 1)
 				)
@@
 		(in_pos_files yes)
 		(dnp no)
-		(property "Reference" "C51"
+		(property "Reference" "C49"
 			(at 173.99 33.02 0)
 			(show_name no)
@@
 			(project "PS-SuppChargerPCB"
 				(path "/bb6ce8fd-e1af-464e-bfef-c3b4f18a2cee/a08c0d72-2b4d-4df5-af0e-616f80f6e7bf/dc00c9b9-366d-4632-b955-a9cb4062bc78"
-					(reference "C51")
+					(reference "C49")
 					(unit 1)
 				)
@@
 		(in_pos_files yes)
 		(dnp no)
-		(property "Reference" "R50"
+		(property "Reference" "R49"
 			(at 175.768 154.686 0)
 			(show_name no)
@@
 			(project "PS-SuppChargerPCB"
 				(path "/bb6ce8fd-e1af-464e-bfef-c3b4f18a2cee/a08c0d72-2b4d-4df5-af0e-616f80f6e7bf/dc00c9b9-366d-4632-b955-a9cb4062bc78"
-					(reference "R50")
+					(reference "R49")
 					(unit 1)
 				)
@@
 		(dnp no)
 		(fields_autoplaced yes)
-		(property "Reference" "D24"
+		(property "Reference" "D25"
 			(at 261.62 103.1874 90)
 			(show_name no)
@@
 			(project "PS-SuppChargerPCB"
 				(path "/bb6ce8fd-e1af-464e-bfef-c3b4f18a2cee/a08c0d72-2b4d-4df5-af0e-616f80f6e7bf/dc00c9b9-366d-4632-b955-a9cb4062bc78"
-					(reference "D24")
+					(reference "D25")
 					(unit 1)
 				)
@@
 		(in_pos_files yes)
 		(dnp no)
-		(property "Reference" "C58"
+		(property "Reference" "C56"
 			(at 217.17 56.642 0)
 			(show_name no)
@@
 			(project "PS-SuppChargerPCB"
 				(path "/bb6ce8fd-e1af-464e-bfef-c3b4f18a2cee/a08c0d72-2b4d-4df5-af0e-616f80f6e7bf/dc00c9b9-366d-4632-b955-a9cb4062bc78"
-					(reference "C58")
+					(reference "C56")
 					(unit 1)
 				)
@@
 		(in_pos_files yes)
 		(dnp no)
-		(property "Reference" "R55"
+		(property "Reference" "R54"
 			(at 226.06 149.225 90)
 			(show_name no)
@@
 			(project "PS-SuppChargerPCB"
 				(path "/bb6ce8fd-e1af-464e-bfef-c3b4f18a2cee/a08c0d72-2b4d-4df5-af0e-616f80f6e7bf/dc00c9b9-366d-4632-b955-a9cb4062bc78"
-					(reference "R55")
+					(reference "R54")
 					(unit 1)
 				)
@@
 		(in_pos_files yes)
 		(dnp no)
-		(property "Reference" "C52"
+		(property "Reference" "C50"
 			(at 169.672 106.934 0)
 			(show_name no)
@@
 			(project "PS-SuppChargerPCB"
 				(path "/bb6ce8fd-e1af-464e-bfef-c3b4f18a2cee/a08c0d72-2b4d-4df5-af0e-616f80f6e7bf/dc00c9b9-366d-4632-b955-a9cb4062bc78"
-					(reference "C52")
+					(reference "C50")
 					(unit 1)
 				)
@@
 		(in_pos_files yes)
 		(dnp no)
-		(property "Reference" "R56"
+		(property "Reference" "R55"
 			(at 248.285 101.5999 0)
 			(show_name no)
@@
 			(project "PS-SuppChargerPCB"
 				(path "/bb6ce8fd-e1af-464e-bfef-c3b4f18a2cee/a08c0d72-2b4d-4df5-af0e-616f80f6e7bf/dc00c9b9-366d-4632-b955-a9cb4062bc78"
-					(reference "R56")
+					(reference "R55")
 					(unit 1)
 				)
@@
 		(in_pos_files yes)
 		(dnp no)
-		(property "Reference" "C55"
+		(property "Reference" "C53"
 			(at 197.358 33.02 0)
 			(show_name no)
@@
 			(project "PS-SuppChargerPCB"
 				(path "/bb6ce8fd-e1af-464e-bfef-c3b4f18a2cee/a08c0d72-2b4d-4df5-af0e-616f80f6e7bf/dc00c9b9-366d-4632-b955-a9cb4062bc78"
-					(reference "C55")
+					(reference "C53")
 					(unit 1)
 				)
@@
 		(dnp no)
 		(fields_autoplaced yes)
-		(property "Reference" "C49"
+		(property "Reference" "C47"
 			(at 34.798 58.928 90)
 			(show_name no)
@@
 			(project "PS-SuppChargerPCB"
 				(path "/bb6ce8fd-e1af-464e-bfef-c3b4f18a2cee/a08c0d72-2b4d-4df5-af0e-616f80f6e7bf/dc00c9b9-366d-4632-b955-a9cb4062bc78"
-					(reference "C49")
+					(reference "C47")
 					(unit 1)
 				)
@@
 		(dnp no)
 		(fields_autoplaced yes)
-		(property "Reference" "R54"
+		(property "Reference" "R53"
 			(at 226.06 137.795 90)
 			(show_name no)
@@
 			(project "PS-SuppChargerPCB"
 				(path "/bb6ce8fd-e1af-464e-bfef-c3b4f18a2cee/a08c0d72-2b4d-4df5-af0e-616f80f6e7bf/dc00c9b9-366d-4632-b955-a9cb4062bc78"
-					(reference "R54")
+					(reference "R53")
 					(unit 1)
 				)
@@
 		(in_pos_files yes)
 		(dnp no)
-		(property "Reference" "C60"
+		(property "Reference" "C58"
 			(at 233.172 32.004 0)
 			(show_name no)
@@
 			(project "PS-SuppChargerPCB"
 				(path "/bb6ce8fd-e1af-464e-bfef-c3b4f18a2cee/a08c0d72-2b4d-4df5-af0e-616f80f6e7bf/dc00c9b9-366d-4632-b955-a9cb4062bc78"
-					(reference "C60")
+					(reference "C58")
 					(unit 1)
 				)

Commit message: layout1
Parts:
- C46, C47, C48, C49, C50, C51, C52, C53, C54, C55, C56, C57, C58, C59, C60, D25, FB1, FB2, R49, R50, R51, R52, R53, R54, R55, R56: KiLib_Generator (none) -> SMD_2terminal_chip_molded
- J10: KiLib_Generator (none) -> connector/pin_header_socket

Commit message: layout5
Parts:
- renumbered C59 to C46, C49 to C47, C51 to C48, C53 to C49, C55 to C50, C57 to C51, C58 to C52, C46 to C53, C47 to C54, C60 to C55, C48 to C56, C52 to C57, C54 to C58, C56 to C59, C50 to C60, D24 to D23, D25 to D24, D23 to D25, FB2 to FB1, FB1 to FB2, R50 to R49, R55 to R50, R56 to R51, R53 to R52, R54 to R53, R49 to R54, R51 to R55, R52 to R56, SW2 to SW1, SW1 to SW2
