File: PS-SuppChargerPCB.kicad_sch (KiCad schematic)
At the start: 52 parts, among them J1 PS_Banana_+, J2 PS_Banana_-, J3 CarLVPowerConnector, J4 Supp_Conn_xT30, J5 TP_I2C, J6 TP_USB_CC, J7 TP_DS SPI

Commit message: alayout2
Parts:
- JP1: value SolderJumper_2_Open -> PP_SolderJumper_2_Open
- R11, R12, R13, R14, R5, R6, R7, R8, R9: value 1k -> 4.7k
Connections:
- net +5V: no longer D6.2 (A), TP7.1
- net DS_SCL renamed DS_CLK
- net DS_SDA renamed DS_MOSI
- new net PD_5V_OUT: D6.2 (A), TP7.1
Other:
- sheet Peripherals ports: added DS_CLK, DS_MOSI; removed DS_SCL, DS_SDA
Changed lines of the file:
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@@
 	)
 	(junction
-		(at 153.67 33.02)
-		(diameter 0)
-		(color 0 0 0 0)
-	)
-	(junction
 		(at 67.31 168.91)
 		(diameter 0)
@@
 	(wire
 		(pts
-			(xy 153.67 33.02) (xy 157.48 33.02)
-		)
-		(stroke
-			(width 0)
-			(type default)
-		)
-	)
-	(wire
-		(pts
 			(xy 191.77 128.27) (xy 193.04 128.27)
 		)
@@
 	(wire
 		(pts
-			(xy 260.35 130.81) (xy 262.89 130.81)
+			(xy 260.35 128.27) (xy 262.89 128.27)
 		)
 		(stroke
@@
 	(wire
 		(pts
-			(xy 134.62 33.02) (xy 153.67 33.02)
+			(xy 134.62 33.02) (xy 157.48 33.02)
 		)
 		(stroke
@@
 	(wire
 		(pts
-			(xy 260.35 128.27) (xy 262.89 128.27)
+			(xy 260.35 130.81) (xy 262.89 130.81)
 		)
 		(stroke
@@
 		)
 	)
-	(label "DS_SDA"
+	(label "DS_MOSI"
 		(at 220.98 91.44 0)
 		(effects
@@
 		)
 	)
-	(label "DS_SDA"
-		(at 260.35 130.81 180)
+	(label "DS_MOSI"
+		(at 260.35 128.27 180)
 		(effects
 			(font
@@
 		)
 	)
-	(label "DS_SCL"
+	(label "DS_CLK"
 		(at 191.77 132.08 180)
 		(effects
@@
 		)
 	)
-	(label "DS_SDA"
+	(label "DS_MOSI"
 		(at 191.77 128.27 180)
 		(effects
@@
 		)
 	)
-	(label "DS_SCL"
-		(at 260.35 128.27 180)
+	(label "DS_CLK"
+		(at 260.35 130.81 180)
 		(effects
 			(font
@@
 		)
 	)
-	(label "DS_SCL"
+	(label "DS_CLK"
 		(at 220.98 93.98 0)
 		(effects
@@
 			)
 		)
-		(property "Value" "1k"
+		(property "Value" "4.7k"
 			(at 223.52 24.13 90)
 			(show_name no)
@@
 			)
 		)
-		(property "Value" "1k"
+		(property "Value" "4.7k"
 			(at 215.9 71.12 90)
 			(show_name no)
@@
 			)
 		)
-		(property "Value" "1k"
+		(property "Value" "4.7k"
 			(at 264.16 35.56 90)
 			(show_name no)
@@
 			)
 		)
-		(property "Value" "1k"
+		(property "Value" "4.7k"
 			(at 223.52 46.99 90)
 			(show_name no)
@@
 			)
 		)
-		(property "Value" "1k"
+		(property "Value" "4.7k"
 			(at 223.52 58.42 90)
 			(show_name no)
@@
 			)
 		)
-		(property "Value" "1k"
+		(property "Value" "4.7k"
 			(at 264.16 24.13 90)
 			(show_name no)
@@
 			)
 		)
-		(property "Value" "1k"
+		(property "Value" "4.7k"
 			(at 264.16 46.99 90)
 			(show_name no)
@@
 			)
 		)
-		(property "Value" "SolderJumper_2_Open"
-			(at 64.643 105.283 0)
+		(property "Value" "PP_SolderJumper_2_Open"
+			(at 63.246 104.902 0)
 			(show_name no)
 			(do_not_autoplace no)
@@
 			)
 		)
-		(property "Value" "+3V3A"
+		(property "Value" "+3V3"
 			(at 258.572 117.856 0)
 			(show_name no)
@@
 			)
 		)
-		(property "Value" "1k"
+		(property "Value" "4.7k"
 			(at 264.16 58.42 90)
 			(show_name no)
@@
 			)
 		)
-		(property "Value" "1k"
+		(property "Value" "4.7k"
 			(at 223.52 35.56 90)
 			(show_name no)
@@
 	)
 	(symbol
-		(lib_id "power:+5V")
-		(at 153.67 33.02 0)
-		(unit 1)
-		(body_style 1)
-		(exclude_from_sim no)
-		(in_bom yes)
-		(on_board yes)
-		(in_pos_files yes)
-		(dnp no)
-		(property "Reference" "#PWR015"
-			(at 153.67 36.83 0)
-			(hide yes)
-			(show_name no)
-			(do_not_autoplace no)
-			(effects
-				(font
-					(size 1.27 1.27)
-				)
-			)
-		)
-		(property "Value" "+5V"
-			(at 153.416 29.21 0)
-			(show_name no)
-			(do_not_autoplace no)
-			(effects
-				(font
-					(size 1.27 1.27)
-				)
-			)
-		)
-		(property "Footprint" ""
-			(at 153.67 33.02 0)
-			(hide yes)
-			(show_name no)
-			(do_not_autoplace no)
-			(effects
-				(font
-					(size 1.27 1.27)
-				)
-			)
-		)
-		(property "Datasheet" ""
-			(at 153.67 33.02 0)
-			(hide yes)
-			(show_name no)
-			(do_not_autoplace no)
-			(effects
-				(font
-					(size 1.27 1.27)
-				)
-			)
-		)
-		(property "Description" "Power symbol creates a global label with name \"+5V\""
-			(at 153.67 33.02 0)
-			(hide yes)
-			(show_name no)
-			(do_not_autoplace no)
-			(effects
-				(font
-					(size 1.27 1.27)
-				)
-			)
-		)
-		(pin "1"
-		)
-		(instances
-			(project "PS-SuppChargerPCB"
-				(path "/bb6ce8fd-e1af-464e-bfef-c3b4f18a2cee"
-					(reference "#PWR015")
-					(unit 1)
-				)
-			)
-		)
-	)
-	(symbol
 		(lib_id "power:GND")
 		(at 43.18 100.33 0)
@@
 			)
 		)
-		(pin "SCL" input
-			(at 262.89 128.27 180)
+		(pin "DS_Vin" input
+			(at 262.89 124.46 180)
 			(effects
 				(font
@@
 			)
 		)
-		(pin "SDA" input
+		(pin "SCL" input
 			(at 262.89 130.81 180)
 			(effects
@@
 			)
 		)
-		(pin "DS_Vin" input
-			(at 262.89 124.46 180)
+		(pin "SDA" input
+			(at 262.89 128.27 180)
 			(effects
 				(font
@@
 			)
 		)
-		(pin "DS_SCL" bidirectional
+		(pin "DS_CLK" bidirectional
 			(at 193.04 132.08 180)
 			(effects
@@
 			)
 		)
-		(pin "DS_SDA" bidirectional
+		(pin "DS_MOSI" bidirectional
 			(at 193.04 128.27 180)
 			(effects
