File: PS-SuppChargerPCB.kicad_sch (KiCad schematic)
At the start: 51 parts, among them J1 PS_Banana_+, J2 PS_Banana_-, J3 TP_I2C, J4 TP_DS SPI, J5 CarLVPowerConnector, J7 Supp_Conn_xT30

Commit message: idealdiodeschematic
Parts:
- removed D12, D13: B540C-13-F, LHRS_Power:B540C-13-F, symbol lhrs_power:B540C-13-F
Other:
- added sheet DiodeOR (DiodeOR.kicad_sch)
- note removed: "Voltage/current rating: 40V 5A"
- moved on the sheet: TP5
