File: Peripherals.kicad_sch (KiCad schematic)
At the start: 4 parts

Commit message: halleffectsense
Parts:
- renumbered R53 to R58, R54 to R59, R48 to R60, R49 to R61
Changed lines of the file:
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@@
 		(dnp no)
 		(fields_autoplaced yes)
-		(property "Reference" "R54"
+		(property "Reference" "R59"
 			(at 135.89 73.6599 0)
 			(show_name no)
@@
 			(project "PS-SuppChargerPCB"
 				(path "/bb6ce8fd-e1af-464e-bfef-c3b4f18a2cee/a08c0d72-2b4d-4df5-af0e-616f80f6e7bf"
-					(reference "R54")
+					(reference "R59")
 					(unit 1)
 				)
@@
 		(dnp no)
 		(fields_autoplaced yes)
-		(property "Reference" "R53"
+		(property "Reference" "R58"
 			(at 135.89 57.1499 0)
 			(show_name no)
@@
 			(project "PS-SuppChargerPCB"
 				(path "/bb6ce8fd-e1af-464e-bfef-c3b4f18a2cee/a08c0d72-2b4d-4df5-af0e-616f80f6e7bf"
-					(reference "R53")
+					(reference "R58")
 					(unit 1)
 				)
@@
 		(dnp no)
 		(fields_autoplaced yes)
-		(property "Reference" "R49"
+		(property "Reference" "R61"
 			(at 167.64 72.3899 0)
 			(show_name no)
@@
 			(project "PS-SuppChargerPCB"
 				(path "/bb6ce8fd-e1af-464e-bfef-c3b4f18a2cee/a08c0d72-2b4d-4df5-af0e-616f80f6e7bf"
-					(reference "R49")
+					(reference "R61")
 					(unit 1)
 				)
@@
 		(dnp no)
 		(fields_autoplaced yes)
-		(property "Reference" "R48"
+		(property "Reference" "R60"
 			(at 167.64 57.1499 0)
 			(show_name no)
@@
 			(project "PS-SuppChargerPCB"
 				(path "/bb6ce8fd-e1af-464e-bfef-c3b4f18a2cee/a08c0d72-2b4d-4df5-af0e-616f80f6e7bf"
-					(reference "R48")
-					(unit 1)
-				)
+					(reference "R60")
+					(unit 1)
+				)

Commit message: newcvsense
Parts:
- added R63, R64: 4.7k, symbol Device:R
Connections:
- net +3V3: now also R63.1, R64.1
- new net INA_SCL: R63.2
- new net INA_SDA: R64.2
- no-connect marks 14 -> 13
Other:
- note added: "CV Sense SCL/SDA Pullup"
- moved on the sheet: R60, R61

Commit message: shuntschem2
Parts:
- removed R58, R59: 4.7k, symbol Device:R
Connections:
- net INA_SCL renamed I2C_SCL
- net INA_SDA renamed I2C_SDA
- no-connect marks 13 -> 15
Other:
- note added: "I2C Pullups"
- note removed: "CV Sense SCL/SDA Pullup"
- note removed: "Display SCL/SDA Pullup"
- moved on the sheet: R60, R61, R63, R64

Commit message: shuntschem3
Other:
- note added: "PD Controller I2C Address: 0x08"
- moved on the sheet: R60, R61, R63, R64
Changed lines of the file:
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@@
 	(paper "A4")
 	(rectangle
-		(start 114.3 40.64)
-		(end 148.59 86.36)
+		(start 114.3 27.94)
+		(end 148.59 73.66)
 		(stroke
 			(width 0)
@@
 	)
 	(rectangle
-		(start 148.59 40.64)
-		(end 182.88 86.36)
+		(start 148.59 27.94)
+		(end 182.88 73.66)
 		(stroke
 			(width 0)
@@
 		)
 	)
+	(text "PD Controller I2C Address: 0x08\n"
+		(exclude_from_sim no)
+		(at 131.572 76.2 0)
+		(effects
+			(font
+				(size 1.27 1.27)
+			)
+		)
+	)
 	(text "I2C Pullups"
 		(exclude_from_sim no)
-		(at 122.174 43.18 0)
+		(at 122.174 30.48 0)
 		(effects
 			(font
@@
 	(text "Buck Boost CC/PG Pullup"
 		(exclude_from_sim no)
-		(at 162.814 42.926 0)
+		(at 162.814 30.226 0)
 		(effects
 			(font
@@
 	(wire
 		(pts
-			(xy 166.37 62.23) (xy 168.91 62.23)
+			(xy 166.37 49.53) (xy 168.91 49.53)
 		)
 		(stroke
@@
 	(wire
 		(pts
-			(xy 129.54 78.74) (xy 133.35 78.74)
+			(xy 129.54 66.04) (xy 133.35 66.04)
 		)
 		(stroke
@@
 	(wire
 		(pts
-			(xy 129.54 62.23) (xy 133.35 62.23)
+			(xy 129.54 49.53) (xy 133.35 49.53)
 		)
 		(stroke
@@
 	(wire
 		(pts
-			(xy 166.37 77.47) (xy 168.91 77.47)
+			(xy 166.37 64.77) (xy 168.91 64.77)
 		)
 		(stroke
@@
 	)
 	(image
-		(at 148.59 124.46)
+		(at 147.32 128.27)
 		(scale 0.327539)
 		(data "iVBORw0KGgoAAAANSUhEUgAABHAAAASKCAYAAAA2f5mlAAAMTGlDQ1BJQ0MgUHJvZmlsZQAASImV"
@@
 	(hierarchical_label "I2C_SDA"
 		(shape bidirectional)
-		(at 129.54 78.74 180)
+		(at 129.54 66.04 180)
 		(effects
 			(font
@@
 	(hierarchical_label "I2C_SCL"
 		(shape bidirectional)
-		(at 129.54 62.23 180)
+		(at 129.54 49.53 180)
 		(effects
 			(font
@@
 	(hierarchical_label "12VBB_PG"
 		(shape bidirectional)
-		(at 166.37 77.47 180)
+		(at 166.37 64.77 180)
 		(effects
 			(font
@@
 	(hierarchical_label "12VBB_CC"
 		(shape bidirectional)
-		(at 166.37 62.23 180)
+		(at 166.37 49.53 180)
 		(effects
 			(font
@@
 	(symbol
 		(lib_id "power:+3.3V")
-		(at 168.91 54.61 0)
+		(at 168.91 41.91 0)
 		(unit 1)
 		(body_style 1)
@@
 		(dnp no)
 		(property "Reference" "#PWR019"
-			(at 168.91 58.42 0)
+			(at 168.91 45.72 0)
 			(hide yes)
 			(show_name no)
@@
 		)
 		(property "Value" "+3V3"
-			(at 168.402 50.8 0)
+			(at 168.402 38.1 0)
 			(show_name no)
 			(do_not_autoplace no)
@@
 		)
 		(property "Footprint" ""
-			(at 168.91 54.61 0)
+			(at 168.91 41.91 0)
 			(hide yes)
 			(show_name no)
@@
 		)
 		(property "Datasheet" ""
-			(at 168.91 54.61 0)
+			(at 168.91 41.91 0)
 			(hide yes)
 			(show_name no)
@@
 		)
 		(property "Description" "Power symbol creates a global label with name \"+3.3V\""
-			(at 168.91 54.61 0)
+			(at 168.91 41.91 0)
 			(hide yes)
 			(show_name no)
@@
 	(symbol
 		(lib_id "Device:R")
-		(at 168.91 73.66 0)
+		(at 168.91 60.96 0)
 		(unit 1)
 		(body_style 1)
@@
 		(fields_autoplaced yes)
 		(property "Reference" "R61"
-			(at 171.45 72.3899 0)
+			(at 171.45 59.6899 0)
 			(show_name no)
 			(do_not_autoplace no)
@@
 		)
 		(property "Value" "100k"
-			(at 171.45 74.9299 0)
+			(at 171.45 62.2299 0)
 			(show_name no)
 			(do_not_autoplace no)
@@
 		)
 		(property "Footprint" ""
-			(at 167.132 73.66 90)
+			(at 167.132 60.96 90)
 			(hide yes)
 			(show_name no)
@@
 		)
 		(property "Datasheet" ""
-			(at 168.91 73.66 0)
+			(at 168.91 60.96 0)
 			(hide yes)
 			(show_name no)
@@
 		)
 		(property "Description" "Resistor"
-			(at 168.91 73.66 0)
+			(at 168.91 60.96 0)
 			(hide yes)
 			(show_name no)
@@
 	(symbol
 		(lib_id "Device:R")
-		(at 133.35 74.93 0)
+		(at 133.35 62.23 0)
 		(unit 1)
 		(body_style 1)
@@
 		(fields_autoplaced yes)
 		(property "Reference" "R64"
-			(at 135.89 73.6599 0)
+			(at 135.89 60.9599 0)
 			(show_name no)
 			(do_not_autoplace no)
@@
 		)
 		(property "Value" "4.7k"
-			(at 135.89 76.1999 0)
+			(at 135.89 63.4999 0)
 			(show_name no)
 			(do_not_autoplace no)
@@
 		)
 		(property "Footprint" ""
-			(at 131.572 74.93 90)
+			(at 131.572 62.23 90)
 			(hide yes)
 			(show_name no)
@@
 		)
 		(property "Datasheet" ""
-			(at 133.35 74.93 0)
+			(at 133.35 62.23 0)
 			(hide yes)
 			(show_name no)
@@
 		)
 		(property "Description" "Resistor"
-			(at 133.35 74.93 0)
+			(at 133.35 62.23 0)
 			(hide yes)
 			(show_name no)
@@
 	(symbol
 		(lib_id "power:+3.3V")
-		(at 133.35 54.61 0)
+		(at 133.35 41.91 0)
 		(unit 1)
 		(body_style 1)
@@
 		(dnp no)
 		(property "Reference" "#PWR042"
-			(at 133.35 58.42 0)
+			(at 133.35 45.72 0)
 			(hide yes)
 			(show_name no)
@@
 		)
 		(property "Value" "+3V3"
-			(at 133.096 50.8 0)
+			(at 133.096 38.1 0)
 			(show_name no)
 			(do_not_autoplace no)
@@
 		)
 		(property "Footprint" ""
-			(at 133.35 54.61 0)
+			(at 133.35 41.91 0)
 			(hide yes)
 			(show_name no)
@@
 		)
 		(property "Datasheet" ""
-			(at 133.35 54.61 0)
+			(at 133.35 41.91 0)
 			(hide yes)
 			(show_name no)
@@
 		)
 		(property "Description" "Power symbol creates a global label with name \"+3.3V\""
-			(at 133.35 54.61 0)
+			(at 133.35 41.91 0)
 			(hide yes)
 			(show_name no)
@@
 	(symbol
 		(lib_id "power:+3.3V")
-		(at 168.91 69.85 0)
+		(at 168.91 57.15 0)
 		(unit 1)
 		(body_style 1)
@@
 		(dnp no)
 		(property "Reference" "#PWR020"
-			(at 168.91 73.66 0)
+			(at 168.91 60.96 0)
 			(hide yes)
 			(show_name no)
@@
 		)
 		(property "Value" "+3V3"
-			(at 168.656 65.786 0)
+			(at 168.656 53.086 0)
 			(show_name no)
 			(do_not_autoplace no)
@@
 		)
 		(property "Footprint" ""
-			(at 168.91 69.85 0)
+			(at 168.91 57.15 0)
 			(hide yes)
 			(show_name no)
@@
 		)
 		(property "Datasheet" ""
-			(at 168.91 69.85 0)
+			(at 168.91 57.15 0)
 			(hide yes)
 			(show_name no)
@@
 		)
 		(property "Description" "Power symbol creates a global label with name \"+3.3V\""
-			(at 168.91 69.85 0)
+			(at 168.91 57.15 0)
 			(hide yes)
 			(show_name no)
@@
 	(symbol
 		(lib_id "Device:R")
-		(at 168.91 58.42 0)
+		(at 168.91 45.72 0)
 		(unit 1)
 		(body_style 1)
@@
 		(fields_autoplaced yes)
 		(property "Reference" "R60"
-			(at 171.45 57.1499 0)
+			(at 171.45 44.4499 0)
 			(show_name no)
 			(do_not_autoplace no)
@@
 		)
 		(property "Value" "100k"
-			(at 171.45 59.6899 0)
+			(at 171.45 46.9899 0)
 			(show_name no)
 			(do_not_autoplace no)
@@
 		)
 		(property "Footprint" ""
-			(at 167.132 58.42 90)
+			(at 167.132 45.72 90)
 			(hide yes)
 			(show_name no)
@@
 		)
 		(property "Datasheet" ""
-			(at 168.91 58.42 0)
+			(at 168.91 45.72 0)
 			(hide yes)
 			(show_name no)
@@
 		)
 		(property "Description" "Resistor"
-			(at 168.91 58.42 0)
+			(at 168.91 45.72 0)
 			(hide yes)
 			(show_name no)
@@
 	(symbol
 		(lib_id "power:+3.3V")
-		(at 133.35 71.12 0)
+		(at 133.35 58.42 0)
 		(unit 1)
 		(body_style 1)
@@
 		(dnp no)
 		(property "Reference" "#PWR043"
-			(at 133.35 74.93 0)
+			(at 133.35 62.23 0)
 			(hide yes)
 			(show_name no)
@@
 		)
 		(property "Value" "+3V3"
-			(at 132.842 67.056 0)
+			(at 132.842 54.356 0)
 			(show_name no)
 			(do_not_autoplace no)
@@
 		)
 		(property "Footprint" ""
-			(at 133.35 71.12 0)
+			(at 133.35 58.42 0)
 			(hide yes)
 			(show_name no)
@@
 		)
 		(property "Datasheet" ""
-			(at 133.35 71.12 0)
+			(at 133.35 58.42 0)
 			(hide yes)
 			(show_name no)
@@
 		)
 		(property "Description" "Power symbol creates a global label with name \"+3.3V\""
-			(at 133.35 71.12 0)
+			(at 133.35 58.42 0)
 			(hide yes)
 			(show_name no)
@@
 	(symbol
 		(lib_id "Device:R")
-		(at 133.35 58.42 0)
+		(at 133.35 45.72 0)
 		(unit 1)
 		(body_style 1)
@@
 		(fields_autoplaced yes)
 		(property "Reference" "R63"
-			(at 135.89 57.1499 0)
+			(at 135.89 44.4499 0)
 			(show_name no)
 			(do_not_autoplace no)
@@
 		)
 		(property "Value" "4.7k"
-			(at 135.89 59.6899 0)
+			(at 135.89 46.9899 0)
 			(show_name no)
 			(do_not_autoplace no)
@@
 		)
 		(property "Footprint" ""
-			(at 131.572 58.42 90)
+			(at 131.572 45.72 90)
 			(hide yes)
 			(show_name no)
@@
 		)
 		(property "Datasheet" ""
-			(at 133.35 58.42 0)
+			(at 133.35 45.72 0)
 			(hide yes)
 			(show_name no)
@@
 		)
 		(property "Description" "Resistor"
-			(at 133.35 58.42 0)
+			(at 133.35 45.72 0)
 			(hide yes)
 			(show_name no)

Commit message: footprints1
Parts:
- R57: renamed from R63; footprint (none) -> Resistor_SMD:R_0603_1608Metric_Pad0.98x0.95mm_HandSolder
- R58: renamed from R64; footprint (none) -> Resistor_SMD:R_0603_1608Metric_Pad0.98x0.95mm_HandSolder
- R59: renamed from R60; footprint (none) -> Resistor_SMD:R_0603_1608Metric_Pad0.98x0.95mm_HandSolder
- R60: renamed from R61; footprint (none) -> Resistor_SMD:R_0603_1608Metric_Pad0.98x0.95mm_HandSolder
Changed lines of the file:
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@@
 		(dnp no)
 		(fields_autoplaced yes)
-		(property "Reference" "R61"
+		(property "Reference" "R60"
 			(at 171.45 59.6899 0)
 			(show_name no)
@@
 			)
 		)
-		(property "Footprint" ""
+		(property "Footprint" "Resistor_SMD:R_0603_1608Metric_Pad0.98x0.95mm_HandSolder"
 			(at 167.132 60.96 90)
 			(hide yes)
@@
 			(project "PS-SuppChargerPCB"
 				(path "/bb6ce8fd-e1af-464e-bfef-c3b4f18a2cee/a08c0d72-2b4d-4df5-af0e-616f80f6e7bf"
-					(reference "R61")
+					(reference "R60")
 					(unit 1)
 				)
@@
 		(dnp no)
 		(fields_autoplaced yes)
-		(property "Reference" "R64"
+		(property "Reference" "R58"
 			(at 135.89 60.9599 0)
 			(show_name no)
@@
 			)
 		)
-		(property "Footprint" ""
+		(property "Footprint" "Resistor_SMD:R_0603_1608Metric_Pad0.98x0.95mm_HandSolder"
 			(at 131.572 62.23 90)
 			(hide yes)
@@
 			(project "PS-SuppChargerPCB"
 				(path "/bb6ce8fd-e1af-464e-bfef-c3b4f18a2cee/a08c0d72-2b4d-4df5-af0e-616f80f6e7bf"
-					(reference "R64")
+					(reference "R58")
 					(unit 1)
 				)
@@
 		(dnp no)
 		(fields_autoplaced yes)
-		(property "Reference" "R60"
+		(property "Reference" "R59"
 			(at 171.45 44.4499 0)
 			(show_name no)
@@
 			)
 		)
-		(property "Footprint" ""
+		(property "Footprint" "Resistor_SMD:R_0603_1608Metric_Pad0.98x0.95mm_HandSolder"
 			(at 167.132 45.72 90)
 			(hide yes)
@@
 			(project "PS-SuppChargerPCB"
 				(path "/bb6ce8fd-e1af-464e-bfef-c3b4f18a2cee/a08c0d72-2b4d-4df5-af0e-616f80f6e7bf"
-					(reference "R60")
+					(reference "R59")
 					(unit 1)
 				)
@@
 		(dnp no)
 		(fields_autoplaced yes)
-		(property "Reference" "R63"
+		(property "Reference" "R57"
 			(at 135.89 44.4499 0)
 			(show_name no)
@@
 			)
 		)
-		(property "Footprint" ""
+		(property "Footprint" "Resistor_SMD:R_0603_1608Metric_Pad0.98x0.95mm_HandSolder"
 			(at 131.572 45.72 90)
 			(hide yes)
@@
 			(project "PS-SuppChargerPCB"
 				(path "/bb6ce8fd-e1af-464e-bfef-c3b4f18a2cee/a08c0d72-2b4d-4df5-af0e-616f80f6e7bf"
-					(reference "R63")
-					(unit 1)
-				)
+					(reference "R57")
+					(unit 1)
+				)

Commit message: layout1
Parts:
- R57, R58, R59, R60: KiLib_Generator (none) -> SMD_2terminal_chip_molded
Changed lines of the file:
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@@
+			)
+		)
+		(property "KiLib_Generator" "SMD_2terminal_chip_molded"
+			(at 168.91 60.96 0)
+			(hide yes)
+			(show_name no)
+			(do_not_autoplace no)
+			(effects
+				(font
+					(size 1.27 1.27)
+				)
 			)
 		)
@@
 			)
 		)
+		(property "KiLib_Generator" "SMD_2terminal_chip_molded"
+			(at 133.35 62.23 0)
+			(hide yes)
+			(show_name no)
+			(do_not_autoplace no)
+			(effects
+				(font
+					(size 1.27 1.27)
+				)
+			)
+		)
 		(pin "2"
 		)
@@
 			)
 		)
+		(property "KiLib_Generator" "SMD_2terminal_chip_molded"
+			(at 168.91 45.72 0)
+			(hide yes)
+			(show_name no)
+			(do_not_autoplace no)
+			(effects
+				(font
+					(size 1.27 1.27)
+				)
+			)
+		)
 		(pin "2"
 		)
@@
 			(at 133.35 45.72 0)
 			(hide yes)
+			(show_name no)
+			(do_not_autoplace no)
+			(effects
+				(font
+					(size 1.27 1.27)
+				)
+			)
+		)
+		(property "KiLib_Generator" "SMD_2terminal_chip_molded"
+			(at 133.35 45.72 0)
+			(hide yes)
