File: Peripherals.kicad_sch (KiCad schematic)
At the start: 4 parts

Commit message: alayout2
Connections:
- no-connect marks 15 -> 16

Commit message: layout5
Parts:
- renumbered R59 to R58, R60 to R59, R58 to R60
Changed lines of the file:
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@@
 	)
 	(no_connect
-		(at 80.01 46.99)
+		(at 80.01 39.37)
 	)
 	(no_connect
@@
 	)
 	(no_connect
-		(at 38.1 100.33)
+		(at 80.01 57.15)
+	)
+	(no_connect
+		(at 80.01 41.91)
 	)
 	(no_connect
-		(at 38.1 80.01)
+		(at 38.1 100.33)
 	)
 	(no_connect
@@
 		(at 38.1 92.71)
 	)
-	(no_connect
-		(at 38.1 102.87)
-	)
 	(wire
 		(pts
@@
 	(wire
 		(pts
-			(xy 80.01 57.15) (xy 81.28 57.15)
+			(xy 35.56 80.01) (xy 38.1 80.01)
 		)
 		(stroke
@@
 	(wire
 		(pts
-			(xy 36.83 82.55) (xy 38.1 82.55)
+			(xy 36.83 102.87) (xy 38.1 102.87)
 		)
 		(stroke
@@
 	(wire
 		(pts
-			(xy 36.83 67.31) (xy 38.1 67.31)
+			(xy 72.39 113.03) (xy 72.39 110.49)
 		)
 		(stroke
@@
 	(wire
 		(pts
-			(xy 36.83 85.09) (xy 38.1 85.09)
+			(xy 80.01 73.66) (xy 82.55 73.66)
 		)
 		(stroke
@@
 	(wire
 		(pts
-			(xy 36.83 74.93) (xy 38.1 74.93)
+			(xy 35.56 67.31) (xy 38.1 67.31)
 		)
 		(stroke
@@
 	(wire
 		(pts
-			(xy 72.39 113.03) (xy 72.39 110.49)
+			(xy 129.54 49.53) (xy 133.35 49.53)
 		)
 		(stroke
@@
 	(wire
 		(pts
-			(xy 36.83 72.39) (xy 38.1 72.39)
+			(xy 80.01 49.53) (xy 81.28 49.53)
 		)
 		(stroke
@@
 	(wire
 		(pts
-			(xy 80.01 73.66) (xy 82.55 73.66)
+			(xy 80.01 46.99) (xy 81.28 46.99)
 		)
 		(stroke
@@
 	(wire
 		(pts
-			(xy 129.54 49.53) (xy 133.35 49.53)
+			(xy 35.56 72.39) (xy 38.1 72.39)
 		)
 		(stroke
@@
 	(wire
 		(pts
-			(xy 80.01 49.53) (xy 81.28 49.53)
+			(xy 80.01 52.07) (xy 81.28 52.07)
 		)
 		(stroke
@@
 	(wire
 		(pts
-			(xy 80.01 52.07) (xy 81.28 52.07)
+			(xy 80.01 54.61) (xy 81.28 54.61)
 		)
 		(stroke
@@
 	(wire
 		(pts
-			(xy 80.01 54.61) (xy 81.28 54.61)
+			(xy 35.56 77.47) (xy 38.1 77.47)
 		)
 		(stroke
@@
 	(wire
 		(pts
-			(xy 36.83 77.47) (xy 38.1 77.47)
+			(xy 166.37 64.77) (xy 168.91 64.77)
 		)
 		(stroke
@@
 	(wire
 		(pts
-			(xy 80.01 39.37) (xy 81.28 39.37)
+			(xy 80.01 76.2) (xy 82.55 76.2)
 		)
 		(stroke
@@
 	(wire
 		(pts
-			(xy 166.37 64.77) (xy 168.91 64.77)
+			(xy 35.56 74.93) (xy 38.1 74.93)
 		)
 		(stroke
@@
 	(wire
 		(pts
-			(xy 80.01 76.2) (xy 82.55 76.2)
+			(xy 35.56 82.55) (xy 38.1 82.55)
 		)
 		(stroke
@@
 	(wire
 		(pts
-			(xy 36.83 69.85) (xy 38.1 69.85)
+			(xy 35.56 85.09) (xy 38.1 85.09)
 		)
 		(stroke
@@
 	(wire
 		(pts
-			(xy 80.01 41.91) (xy 81.28 41.91)
+			(xy 35.56 69.85) (xy 38.1 69.85)
 		)
 		(stroke
@@
 		)
 	)
-	(hierarchical_label "DS_BLK"
-		(shape bidirectional)
-		(at 36.83 74.93 180)
-		(effects
-			(font
-				(size 1.27 1.27)
-			)
-			(justify right)
-		)
-	)
-	(hierarchical_label "12VBB_PG"
+	(hierarchical_label "PD_GPIO_1"
 		(shape bidirectional)
-		(at 36.83 69.85 180)
+		(at 35.56 85.09 180)
 		(effects
 			(font
@@
 		)
 	)
-	(hierarchical_label "EN"
+	(hierarchical_label "DS_MOSI"
 		(shape bidirectional)
-		(at 36.83 72.39 180)
+		(at 81.28 49.53 0)
 		(effects
 			(font
 				(size 1.27 1.27)
 			)
-			(justify right)
+			(justify left)
 		)
 	)
-	(hierarchical_label "INA_ALERT"
+	(hierarchical_label "USB_DP"
 		(shape bidirectional)
-		(at 81.28 57.15 0)
+		(at 82.55 73.66 0)
 		(effects
 			(font
@@
 		)
 	)
-	(hierarchical_label "USB_DP"
+	(hierarchical_label "I2C_SCL"
 		(shape bidirectional)
-		(at 82.55 73.66 0)
+		(at 81.28 54.61 0)
 		(effects
 			(font
@@
 		)
 	)
-	(hierarchical_label "USB_DM"
+	(hierarchical_label "I2C_SDA"
 		(shape bidirectional)
-		(at 82.55 76.2 0)
+		(at 81.28 52.07 0)
 		(effects
 			(font
@@
 		)
 	)
-	(hierarchical_label "I2C_SCL"
+	(hierarchical_label "DS_BLK"
 		(shape bidirectional)
-		(at 81.28 54.61 0)
+		(at 35.56 72.39 180)
 		(effects
 			(font
 				(size 1.27 1.27)
 			)
-			(justify left)
+			(justify right)
 		)
 	)
-	(hierarchical_label "DS_RES"
+	(hierarchical_label "12VBB_CC"
 		(shape bidirectional)
-		(at 36.83 85.09 180)
+		(at 35.56 80.01 180)
 		(effects
 			(font
@@
 		)
 	)
-	(hierarchical_label "PD_FAULT"
+	(hierarchical_label "USB_DM"
 		(shape bidirectional)
-		(at 81.28 41.91 0)
+		(at 82.55 76.2 0)
 		(effects
 			(font
@@
 		)
 	)
-	(hierarchical_label "DS_MOSI"
+	(hierarchical_label "EN"
 		(shape bidirectional)
-		(at 81.28 49.53 0)
+		(at 35.56 74.93 180)
+		(effects
+			(font
+				(size 1.27 1.27)
+			)
+			(justify right)
+		)
+	)
+	(hierarchical_label "DS_RES"
+		(shape bidirectional)
+		(at 81.28 46.99 0)
 		(effects
 			(font
@@
 		)
 	)
-	(hierarchical_label "12VBB_PG"
+	(hierarchical_label "DS_CS"
 		(shape bidirectional)
-		(at 166.37 64.77 180)
+		(at 35.56 69.85 180)
 		(effects
 			(font
@@
 		)
 	)
-	(hierarchical_label "DS_DC"
+	(hierarchical_label "12VBB_PG"
 		(shape bidirectional)
-		(at 36.83 82.55 180)
+		(at 166.37 64.77 180)
 		(effects
 			(font
@@
 		)
 	)
-	(hierarchical_label "12VBB_CC"
+	(hierarchical_label "PD_FAULT"
 		(shape bidirectional)
-		(at 166.37 49.53 180)
+		(at 35.56 82.55 180)
 		(effects
 			(font
@@
 		)
 	)
-	(hierarchical_label "DS_CS"
+	(hierarchical_label "12VBB_CC"
 		(shape bidirectional)
-		(at 36.83 77.47 180)
+		(at 166.37 49.53 180)
 		(effects
 			(font
@@
 		)
 	)
-	(hierarchical_label "PD_GPIO_1"
+	(hierarchical_label "INA_ALERT"
 		(shape bidirectional)
-		(at 81.28 39.37 0)
+		(at 36.83 102.87 180)
 		(effects
 			(font
 				(size 1.27 1.27)
 			)
-			(justify left)
+			(justify right)
 		)
 	)
-	(hierarchical_label "12VBB_CC"
+	(hierarchical_label "12VBB_PG"
 		(shape bidirectional)
-		(at 36.83 67.31 180)
+		(at 35.56 77.47 180)
 		(effects
 			(font
@@
 		)
 	)
-	(hierarchical_label "I2C_SDA"
+	(hierarchical_label "DS_DC"
 		(shape bidirectional)
-		(at 81.28 52.07 0)
+		(at 35.56 67.31 180)
 		(effects
 			(font
 				(size 1.27 1.27)
 			)
-			(justify left)
+			(justify right)
 		)
 	)
@@
 		(dnp no)
 		(fields_autoplaced yes)
-		(property "Reference" "R60"
+		(property "Reference" "R59"
 			(at 171.45 59.6899 0)
 			(show_name no)
@@
 			(project "PS-SuppChargerPCB"
 				(path "/bb6ce8fd-e1af-464e-bfef-c3b4f18a2cee/a08c0d72-2b4d-4df5-af0e-616f80f6e7bf"
-					(reference "R60")
+					(reference "R59")
 					(unit 1)
 				)
@@
 		(dnp no)
 		(fields_autoplaced yes)
-		(property "Reference" "R58"
+		(property "Reference" "R60"
 			(at 135.89 60.9599 0)
 			(show_name no)
@@
 			(project "PS-SuppChargerPCB"
 				(path "/bb6ce8fd-e1af-464e-bfef-c3b4f18a2cee/a08c0d72-2b4d-4df5-af0e-616f80f6e7bf"
-					(reference "R58")
+					(reference "R60")
 					(unit 1)
 				)
@@
 		(dnp no)
 		(fields_autoplaced yes)
-		(property "Reference" "R59"
+		(property "Reference" "R58"
 			(at 171.45 44.4499 0)
 			(show_name no)
@@
 			(project "PS-SuppChargerPCB"
 				(path "/bb6ce8fd-e1af-464e-bfef-c3b4f18a2cee/a08c0d72-2b4d-4df5-af0e-616f80f6e7bf"
-					(reference "R59")
+					(reference "R58")
 					(unit 1)
 				)
