File: USB-C_Connector.kicad_sch (KiCad schematic)
At the start: 6 parts, among them J3 USB_C_Receptacle_USB2.0_16P

Commit message: reviewnotes
Connections:
- net USB_DM: no longer J3.A7 (D-), J3.B7 (D-)
- net USB_DP: no longer J3.A6 (D+), J3.B6 (D+)
- new net USB_D+: J3.A6 (D+), J3.B6 (D+)
- new net USB_D-: J3.A7 (D-), J3.B7 (D-)
Changed lines of the file:
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@@
 		)
 	)
-	(hierarchical_label "USB_DP"
+	(hierarchical_label "USB_D+"
 		(shape bidirectional)
 		(at 55.88 49.53 0)
@@
 		)
 	)
-	(hierarchical_label "USB_DM"
+	(hierarchical_label "USB_D-"
 		(shape bidirectional)
 		(at 55.88 44.45 0)

Commit message: schematic2
Other:
- note added: "fix usb DM and usb DP net labels"
Changed lines of the file:
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@@
+		)
+	)
+	(text "fix usb DM and usb DP net labels"
+		(exclude_from_sim no)
+		(at 125.476 72.39 0)
+		(effects
+			(font
+				(size 1.27 1.27)
+			)
 		)
 	)

Commit message: schematic6
Parts:
- removed R26, R27: 5.1k, Resistor_SMD:R_0603_1608Metric_Pad0.98x0.95mm_HandSolder, symbol Device:R
Connections:
- net USB_D+ is gone; now on net USB_DP: J3.A6 (D+), J3.B6 (D+)
- net USB_D- is gone; now on net USB_DM: J3.A7 (D-), J3.B7 (D-)
- no-connect marks 4 -> 2
Other:
- note removed: "If using USB-C PD, remove CC1 and CC2 pull down resistor, if not using USB-C PD, keep them"
- note removed: "fix usb DM and usb DP net labels"
- moved on the sheet: C31, D8, D9

Commit message: fixedsharepoint
Parts:
- removed D9: TPD2EUSB30DRTR, LHRS_ICs:TPD2EUSB30DRTR, symbol lhrs_ics:TPD2EUSB30DRTR
- added D9: SP0503BAHT, Package_TO_SOT_SMD:SOT-143, symbol lhrs_ics:SP0503BAH
- C31: value 10uF -> 10u
Connections:
- net GND: now also D9.1 (A)
- net VBUS_IN: now also D9.4 (K)
- net USB_DM renamed USB_D-
- net USB_D-: now also D9.3 (K)
- net USB_DP renamed USB_D+
- net USB_D+: now also D9.2 (K)
Other:
- note removed: "5.5V working 7V breakdown 8V clamping"
- moved on the sheet: C31, D8

Commit message: schematic10
Other:
- moved on the sheet: C31, D8, D9, J3

Commit message: halleffectsense
Parts:
- renumbered C31 to C2, D8 to D13, D9 to D14, J3 to J8
Changed lines of the file:
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@@
 		(dnp no)
 		(fields_autoplaced yes)
-		(property "Reference" "D9"
+		(property "Reference" "D14"
 			(at 115.57 76.2 90)
 			(show_name no)
@@
 			(project "PS-SuppChargerPCB"
 				(path "/bb6ce8fd-e1af-464e-bfef-c3b4f18a2cee/ec016523-8b34-47f1-ab1c-e2da371f5914"
-					(reference "D9")
+					(reference "D14")
 					(unit 1)
 				)
@@
 		(dnp no)
 		(fields_autoplaced yes)
-		(property "Reference" "J3"
+		(property "Reference" "J8"
 			(at 44.45 34.29 0)
 			(show_name no)
@@
 			(project "PS-SuppChargerPCB"
 				(path "/bb6ce8fd-e1af-464e-bfef-c3b4f18a2cee/ec016523-8b34-47f1-ab1c-e2da371f5914"
-					(reference "J3")
+					(reference "J8")
 					(unit 1)
 				)
@@
 		(in_pos_files yes)
 		(dnp no)
-		(property "Reference" "D8"
+		(property "Reference" "D13"
 			(at 68.58 36.195 0)
 			(show_name no)
@@
 			(project "PS-SuppChargerPCB"
 				(path "/bb6ce8fd-e1af-464e-bfef-c3b4f18a2cee/ec016523-8b34-47f1-ab1c-e2da371f5914"
-					(reference "D8")
+					(reference "D13")
 					(unit 1)
 				)
@@
 		(in_pos_files yes)
 		(dnp no)
-		(property "Reference" "C31"
+		(property "Reference" "C2"
 			(at 73.2028 49.4284 0)
 			(show_name no)
@@
 			(project "PS-SuppChargerPCB"
 				(path "/bb6ce8fd-e1af-464e-bfef-c3b4f18a2cee/ec016523-8b34-47f1-ab1c-e2da371f5914"
-					(reference "C31")
-					(unit 1)
-				)
+					(reference "C2")
+					(unit 1)
+				)

Commit message: footprints1
Parts:
- J8: footprint LHRS_ICs:USB_C_Receptacle_GCT_USB4105-xx-A_16P_TopMnt_Horizontal -> LHRS_Connectors:USB_C_Receptacle_GCT_USB4105-xx-A_16P_TopMnt_Horizontal
- renumbered D13 to D14, D14 to D15
Changed lines of the file:
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@@
 		(dnp no)
 		(fields_autoplaced yes)
-		(property "Reference" "D14"
+		(property "Reference" "D15"
 			(at 115.57 76.2 90)
 			(show_name no)
@@
 			(project "PS-SuppChargerPCB"
 				(path "/bb6ce8fd-e1af-464e-bfef-c3b4f18a2cee/ec016523-8b34-47f1-ab1c-e2da371f5914"
-					(reference "D14")
+					(reference "D15")
 					(unit 1)
 				)
@@
 			)
 		)
-		(property "Footprint" "LHRS_ICs:USB_C_Receptacle_GCT_USB4105-xx-A_16P_TopMnt_Horizontal"
+		(property "Footprint" "LHRS_Connectors:USB_C_Receptacle_GCT_USB4105-xx-A_16P_TopMnt_Horizontal"
 			(at 48.26 57.15 0)
 			(hide yes)
@@
 		(in_pos_files yes)
 		(dnp no)
-		(property "Reference" "D13"
+		(property "Reference" "D14"
 			(at 68.58 36.195 0)
 			(show_name no)
@@
 			(project "PS-SuppChargerPCB"
 				(path "/bb6ce8fd-e1af-464e-bfef-c3b4f18a2cee/ec016523-8b34-47f1-ab1c-e2da371f5914"
-					(reference "D13")
-					(unit 1)
-				)
+					(reference "D14")
+					(unit 1)
+				)

Commit message: layout1
Parts:
- C2: KiLib_Generator (none) -> SMD_2terminal_chip_molded
Changed lines of the file:
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@@
+			)
+		)
+		(property "KiLib_Generator" "SMD_2terminal_chip_molded"
+			(at 76.2 48.26 0)
+			(hide yes)
+			(show_name no)
+			(do_not_autoplace no)
+			(effects
+				(font
+					(size 1.27 1.27)
+				)
 			)
 		)
