File: USB_PD.kicad_sch (KiCad schematic)
At the start: 38 parts, among them IC1 CYPD3177-24LQXQ, Q1 SI7997DP-T1-GE3, Q2 SI7997DP-T1-GE3, Q3 IRLML0030

Commit message: reviewnotes
Other:
- note added: "i2c needs pullup resistors in general"
- note added: "put on mcu i2c"
Changed lines of the file:
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@@
+		)
+	)
+	(text "i2c needs pullup resistors in general\n"
+		(exclude_from_sim no)
+		(at 222.758 62.992 0)
+		(effects
+			(font
+				(size 1.27 1.27)
+			)
 		)
 	)
@@
 		)
 	)
+	(text "put on mcu i2c\n"
+		(exclude_from_sim no)
+		(at 202.946 65.278 0)
+		(effects
+			(font
+				(size 1.27 1.27)
+			)
+		)
+	)

Commit message: fixedsharepoint
Parts:
- C63: renamed from C1; Mfg GRM21BR61H106KE43K -> (none)
- D1: Height 2.44 -> (none); Manufacturer_Name Vishay -> (none); Mouser Part Number 625-SMBJ24A-E3 -> (none); Mouser Price/Stock https://www.mouser.co.uk/ProductDetail/Vishay-General-Semic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 -> (none)
- D16: renamed from D4; Color Red -> (none); Mfg NCD0603R1 -> (none)
- D2, D3: Height 2.44 -> (none); Manufacturer_Name Vishay -> (none); Mouser Part Number 625-SMBJ10A-E3 -> (none); Mouser Price/Stock https://www.mouser.co.uk/ProductDetail/Vishay-General-Semic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 -> (none)
- IC4: renamed from IC1; Height 0.6 -> (none); Manufacturer_Name Infineon -> (none); Mouser Part Number 727-CYPD3177-24LQXQ -> (none); Mouser Price/Stock https://www.mouser.co.uk/ProductDetail/Infineon-Technologie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 -> (none)
- Q6: renamed from Q1; Manufacturer_Name Vishay -> (none); Mouser Part Number 781-SI7997DP-T1-GE3 -> (none); Mouser Price/Stock https://www.mouser.co.uk/ProductDetail/Vishay-Semiconductor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 -> (none)
- Q7: renamed from Q2; Manufacturer_Name Vishay -> (none); Mouser Part Number 781-SI7997DP-T1-GE3 -> (none); Mouser Price/Stock https://www.mouser.co.uk/ProductDetail/Vishay-Semiconductor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 -> (none)
- R15: renamed from R2; Mfg CRCW06035K10FKEC -> (none)
- R7: renamed from R1; Mfg CRCW06035K10FKEC -> (none)
- renumbered C2 to C64, C3 to C65, C4 to C66, C5 to C67, C6 to C68, C7 to C69, C8 to C70, C9 to C71, Q3 to Q8, R3 to R46, R4 to R47, R5 to R57, R6 to R58, R7 to R59, R8 to R60, R9 to R61, R10 to R62, R11 to R63, R12 to R64, R13 to R65, R14 to R66, R15 to R67, TP6 to TP12, TP3 to TP4, TP4 to TP5, TP5 to TP6
Other:
- note removed: "i2c needs pullup resistors in general"
- note removed: "put on mcu i2c"

Commit message: schematic9
Parts:
- TP1, TP2, TP4, TP5, TP6: footprint Connector_PinHeader_2.54mm:PinHeader_1x01_P2.54mm_Vertical -> TestPoint:TestPoint_Loop_D1.80mm_Drill1.0mm_Beaded; symbol Connector:TestPoint -> lhrs_misc:Multimeter_TP; now in the parts list
- TP12: footprint TestPoint:TestPoint_Pad_1.0x1.0mm -> TestPoint:TestPoint_Loop_D1.80mm_Drill1.0mm_Beaded; symbol Connector:TestPoint -> lhrs_misc:Multimeter_TP; now in the parts list
Connections:
- net PD_1V8: no longer TP5.1
- net PD_5V_OUT: no longer TP4.1
- net PD_FAULT: no longer TP12.1
- net PD_VBUS_OUT: no longer TP2.1
- net VBUS_MAX: no longer TP6.1
Changed lines of the file:
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@@
 	)
 	(junction
-		(at 138.43 171.45)
-		(diameter 0)
-		(color 0 0 0 0)
-	)
-	(junction
 		(at 95.25 189.23)
 		(diameter 0)
@@
 	)
 	(junction
-		(at 44.45 46.99)
-		(diameter 0)
-		(color 0 0 0 0)
-	)
-	(junction
 		(at 72.39 189.23)
 		(diameter 0)
@@
 	)
 	(junction
-		(at 138.43 138.43)
-		(diameter 0)
-		(color 0 0 0 0)
-	)
-	(junction
 		(at 72.39 156.21)
 		(diameter 0)
@@
 	(wire
 		(pts
-			(xy 138.43 171.45) (xy 140.97 171.45)
-		)
-		(stroke
-			(width 0)
-			(type default)
-		)
-	)
-	(wire
-		(pts
 			(xy 187.96 68.58) (xy 187.96 72.39)
 		)
@@
 	(wire
 		(pts
-			(xy 125.73 171.45) (xy 138.43 171.45)
+			(xy 125.73 171.45) (xy 140.97 171.45)
 		)
 		(stroke
@@
 	(wire
 		(pts
-			(xy 125.73 138.43) (xy 138.43 138.43)
+			(xy 125.73 138.43) (xy 140.97 138.43)
 		)
 		(stroke
@@
 	(wire
 		(pts
-			(xy 138.43 138.43) (xy 140.97 138.43)
-		)
-		(stroke
-			(width 0)
-			(type default)
-		)
-	)
-	(wire
-		(pts
 			(xy 240.03 52.07) (xy 240.03 57.15)
 		)
@@
 	)
 	(symbol
-		(lib_id "Connector:TestPoint")
+		(lib_id "lhrs_misc:Multimeter_TP")
 		(at 236.22 102.87 180)
 		(unit 1)
 		(body_style 1)
 		(exclude_from_sim no)
-		(in_bom no)
+		(in_bom yes)
 		(on_board yes)
 		(in_pos_files yes)
@@
 			)
 		)
-		(property "Footprint" "TestPoint:TestPoint_Pad_1.0x1.0mm"
-			(at 231.14 102.87 0)
+		(property "Footprint" "TestPoint:TestPoint_Loop_D1.80mm_Drill1.0mm_Beaded"
+			(at 236.22 102.87 0)
 			(hide yes)
 			(show_name no)
@@
 		)
 		(property "Datasheet" ""
-			(at 231.14 102.87 0)
+			(at 236.22 102.87 0)
 			(hide yes)
 			(show_name no)
@@
 	)
 	(symbol
-		(lib_id "Connector:TestPoint")
+		(lib_id "lhrs_misc:Multimeter_TP")
 		(at 138.43 171.45 0)
 		(unit 1)
 		(body_style 1)
 		(exclude_from_sim no)
-		(in_bom no)
+		(in_bom yes)
 		(on_board yes)
 		(in_pos_files yes)
@@
 			)
 		)
-		(property "Footprint" "Connector_PinHeader_2.54mm:PinHeader_1x01_P2.54mm_Vertical"
-			(at 143.51 171.45 0)
+		(property "Footprint" "TestPoint:TestPoint_Loop_D1.80mm_Drill1.0mm_Beaded"
+			(at 138.43 171.45 0)
 			(hide yes)
 			(show_name no)
@@
 		)
 		(property "Datasheet" ""
-			(at 143.51 171.45 0)
+			(at 138.43 171.45 0)
 			(hide yes)
 			(show_name no)
@@
 	)
 	(symbol
-		(lib_id "Connector:TestPoint")
+		(lib_id "lhrs_misc:Multimeter_TP")
 		(at 138.43 138.43 0)
 		(unit 1)
 		(body_style 1)
 		(exclude_from_sim no)
-		(in_bom no)
+		(in_bom yes)
 		(on_board yes)
 		(in_pos_files yes)
@@
 			)
 		)
-		(property "Footprint" "Connector_PinHeader_2.54mm:PinHeader_1x01_P2.54mm_Vertical"
-			(at 143.51 138.43 0)
+		(property "Footprint" "TestPoint:TestPoint_Loop_D1.80mm_Drill1.0mm_Beaded"
+			(at 138.43 138.43 0)
 			(hide yes)
 			(show_name no)
@@
 		)
 		(property "Datasheet" ""
-			(at 143.51 138.43 0)
+			(at 138.43 138.43 0)
 			(hide yes)
 			(show_name no)
@@
 	)
 	(symbol
-		(lib_id "Connector:TestPoint")
+		(lib_id "lhrs_misc:Multimeter_TP")
 		(at 44.45 46.99 0)
 		(unit 1)
 		(body_style 1)
 		(exclude_from_sim no)
-		(in_bom no)
+		(in_bom yes)
 		(on_board yes)
 		(in_pos_files yes)
@@
 		)
 		(property "Value" "VBUS_IN"
-			(at 46.99 43.6879 0)
+			(at 46.99 48.7679 0)
 			(show_name no)
 			(do_not_autoplace no)
@@
 			)
 		)
-		(property "Footprint" "Connector_PinHeader_2.54mm:PinHeader_1x01_P2.54mm_Vertical"
-			(at 49.53 46.99 0)
+		(property "Footprint" "TestPoint:TestPoint_Loop_D1.80mm_Drill1.0mm_Beaded"
+			(at 44.45 46.99 0)
 			(hide yes)
 			(show_name no)
@@
 		)
 		(property "Datasheet" ""
-			(at 49.53 46.99 0)
+			(at 44.45 46.99 0)
 			(hide yes)
 			(show_name no)
@@
 	)
 	(symbol
-		(lib_id "Connector:TestPoint")
+		(lib_id "lhrs_misc:Multimeter_TP")
 		(at 163.83 48.26 270)
 		(unit 1)
 		(body_style 1)
 		(exclude_from_sim no)
-		(in_bom no)
+		(in_bom yes)
 		(on_board yes)
 		(in_pos_files yes)
@@
 			)
 		)
-		(property "Footprint" "Connector_PinHeader_2.54mm:PinHeader_1x01_P2.54mm_Vertical"
-			(at 163.83 53.34 0)
+		(property "Footprint" "TestPoint:TestPoint_Loop_D1.80mm_Drill1.0mm_Beaded"
+			(at 163.83 48.26 0)
 			(hide yes)
 			(show_name no)
@@
 		)
 		(property "Datasheet" ""
-			(at 163.83 53.34 0)
+			(at 163.83 48.26 0)
 			(hide yes)
 			(show_name no)
@@
 	)
 	(symbol
-		(lib_id "Connector:TestPoint")
+		(lib_id "lhrs_misc:Multimeter_TP")
 		(at 151.13 48.26 90)
 		(unit 1)
 		(body_style 1)
 		(exclude_from_sim no)
-		(in_bom no)
+		(in_bom yes)
 		(on_board yes)
 		(in_pos_files yes)
@@
 			)
 		)
-		(property "Footprint" "Connector_PinHeader_2.54mm:PinHeader_1x01_P2.54mm_Vertical"
-			(at 151.13 43.18 0)
+		(property "Footprint" "TestPoint:TestPoint_Loop_D1.80mm_Drill1.0mm_Beaded"
+			(at 151.13 48.26 0)
 			(hide yes)
 			(show_name no)
@@
 		)
 		(property "Datasheet" ""
-			(at 151.13 43.18 0)
+			(at 151.13 48.26 0)
 			(hide yes)
 			(show_name no)

Commit message: schematic10
Connections:
- net PD_1V8: now also TP5.1
- net PD_5V_OUT: now also TP4.1
- net PD_FAULT: now also TP12.1
- net PD_VBUS_OUT: now also TP2.1
- net VBUS_MAX: now also TP6.1
Changed lines of the file:
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@@
 	)
 	(junction
-		(at 151.13 48.26)
+		(at 240.03 52.07)
 		(diameter 0)
 		(color 0 0 0 0)
 	)
 	(junction
-		(at 240.03 52.07)
+		(at 138.43 171.45)
 		(diameter 0)
 		(color 0 0 0 0)
@@
 	)
 	(junction
+		(at 241.3 102.87)
+		(diameter 0)
+		(color 0 0 0 0)
+	)
+	(junction
 		(at 35.56 66.04)
 		(diameter 0)
@@
 	)
 	(junction
+		(at 151.13 48.26)
+		(diameter 0)
+		(color 0 0 0 0)
+	)
+	(junction
 		(at 95.25 156.21)
 		(diameter 0)
@@
 		(color 0 0 0 0)
 	)
+	(junction
+		(at 138.43 138.43)
+		(diameter 0)
+		(color 0 0 0 0)
+	)
 	(no_connect
 		(at 137.16 82.55)
@@
 	(wire
 		(pts
-			(xy 177.8 69.85) (xy 184.15 69.85)
+			(xy 151.13 48.26) (xy 151.13 49.53)
 		)
 		(stroke
@@
 	(wire
 		(pts
-			(xy 46.99 182.88) (xy 46.99 189.23)
+			(xy 177.8 69.85) (xy 184.15 69.85)
 		)
 		(stroke
@@
 	(wire
 		(pts
-			(xy 72.39 179.07) (xy 72.39 189.23)
+			(xy 46.99 182.88) (xy 46.99 189.23)
 		)
 		(stroke
@@
 	(wire
 		(pts
-			(xy 151.13 48.26) (xy 151.13 49.53)
+			(xy 72.39 179.07) (xy 72.39 189.23)
 		)
 		(stroke
@@
 	(wire
 		(pts
+			(xy 241.3 102.87) (xy 246.38 102.87)
+		)
+		(stroke
+			(width 0)
+			(type default)
+		)
+	)
+	(wire
+		(pts
 			(xy 44.45 46.99) (xy 44.45 52.07)
 		)
@@
 	(wire
 		(pts
-			(xy 236.22 102.87) (xy 246.38 102.87)
+			(xy 236.22 102.87) (xy 241.3 102.87)
 		)
 		(stroke
@@
 	(wire
 		(pts
+			(xy 138.43 171.45) (xy 140.97 171.45)
+		)
+		(stroke
+			(width 0)
+			(type default)
+		)
+	)
+	(wire
+		(pts
 			(xy 184.15 68.58) (xy 184.15 69.85)
 		)
@@
 	(wire
 		(pts
-			(xy 125.73 171.45) (xy 140.97 171.45)
+			(xy 125.73 171.45) (xy 138.43 171.45)
 		)
 		(stroke
@@
 	(wire
 		(pts
+			(xy 138.43 138.43) (xy 140.97 138.43)
+		)
+		(stroke
+			(width 0)
+			(type default)
+		)
+	)
+	(wire
+		(pts
 			(xy 77.47 171.45) (xy 95.25 171.45)
 		)
@@
 	(wire
 		(pts
-			(xy 125.73 138.43) (xy 140.97 138.43)
+			(xy 125.73 138.43) (xy 138.43 138.43)
 		)
 		(stroke
@@
 	(symbol
 		(lib_id "lhrs_misc:Multimeter_TP")
-		(at 236.22 102.87 180)
+		(at 241.3 107.95 180)
 		(unit 1)
 		(body_style 1)
@@
 		(dnp no)
 		(property "Reference" "TP12"
-			(at 238.76 104.9019 0)
+			(at 243.84 109.9819 0)
 			(hide yes)
 			(show_name no)
@@
 		)
 		(property "Value" "PD_FAULT"
-			(at 246.634 106.172 0)
+			(at 246.38 108.458 0)
 			(show_name no)
 			(do_not_autoplace no)
@@
 		)
 		(property "Footprint" "TestPoint:TestPoint_Loop_D1.80mm_Drill1.0mm_Beaded"
-			(at 236.22 102.87 0)
+			(at 241.3 107.95 0)
 			(hide yes)
 			(show_name no)
@@
 		)
 		(property "Datasheet" ""
-			(at 236.22 102.87 0)
+			(at 241.3 107.95 0)
 			(hide yes)
 			(show_name no)
@@
 		)
 		(property "Description" "test point"
-			(at 236.22 102.87 0)
+			(at 241.3 107.95 0)
 			(hide yes)
 			(show_name no)
@@
 	(symbol
 		(lib_id "lhrs_misc:Multimeter_TP")
-		(at 138.43 171.45 0)
+		(at 138.43 166.37 0)
 		(unit 1)
 		(body_style 1)
@@
 		(dnp no)
 		(property "Reference" "TP4"
-			(at 135.89 169.4181 0)
+			(at 135.89 164.3381 0)
 			(hide yes)
 			(show_name no)
@@
 		)
 		(property "Footprint" "TestPoint:TestPoint_Loop_D1.80mm_Drill1.0mm_Beaded"
-			(at 138.43 171.45 0)
+			(at 138.43 166.37 0)
 			(hide yes)
 			(show_name no)
@@
 		)
 		(property "Datasheet" ""
-			(at 138.43 171.45 0)
+			(at 138.43 166.37 0)
 			(hide yes)
 			(show_name no)
@@
 		)
 		(property "Description" "test point"
-			(at 138.43 171.45 0)
+			(at 138.43 166.37 0)
 			(hide yes)
 			(show_name no)
@@
 	(symbol
 		(lib_id "lhrs_misc:Multimeter_TP")
-		(at 138.43 138.43 0)
+		(at 138.43 133.35 0)
 		(unit 1)
 		(body_style 1)
@@
 		(dnp no)
 		(property "Reference" "TP2"
-			(at 135.89 136.3981 0)
+			(at 135.89 131.3181 0)
 			(hide yes)
 			(show_name no)
@@
 		)
 		(property "Value" "PD_VBUS_OUT"
-			(at 132.08 132.842 0)
+			(at 132.08 132.588 0)
 			(show_name no)
 			(do_not_autoplace no)
@@
 		)
 		(property "Footprint" "TestPoint:TestPoint_Loop_D1.80mm_Drill1.0mm_Beaded"
-			(at 138.43 138.43 0)
+			(at 138.43 133.35 0)
 			(hide yes)
 			(show_name no)
@@
 		)
 		(property "Datasheet" ""
-			(at 138.43 138.43 0)
+			(at 138.43 133.35 0)
 			(hide yes)
 			(show_name no)
@@
 		)
 		(property "Description" "test point"
-			(at 138.43 138.43 0)
+			(at 138.43 133.35 0)
 			(hide yes)
 			(show_name no)
@@
 	(symbol
 		(lib_id "lhrs_misc:Multimeter_TP")
-		(at 163.83 48.26 270)
+		(at 168.91 48.26 270)
 		(unit 1)
 		(body_style 1)
@@
 		(dnp no)
 		(property "Reference" "TP6"
-			(at 165.8619 45.72 0)
+			(at 170.9419 45.72 0)
 			(hide yes)
 			(show_name no)
@@
 		)
 		(property "Value" "PD_3V3"
-			(at 168.91 48.2599 90)
+			(at 167.894 48.26 90)
 			(show_name no)
 			(do_not_autoplace no)
@@
 		)
 		(property "Footprint" "TestPoint:TestPoint_Loop_D1.80mm_Drill1.0mm_Beaded"
-			(at 163.83 48.26 0)
+			(at 168.91 48.26 0)
 			(hide yes)
 			(show_name no)
@@
 		)
 		(property "Datasheet" ""
-			(at 163.83 48.26 0)
+			(at 168.91 48.26 0)
 			(hide yes)
 			(show_name no)
@@
 		)
 		(property "Description" "test point"
-			(at 163.83 48.26 0)
+			(at 168.91 48.26 0)
 			(hide yes)
 			(show_name no)
@@
 	(symbol
 		(lib_id "lhrs_misc:Multimeter_TP")
-		(at 151.13 48.26 90)
+		(at 146.05 48.26 90)
 		(unit 1)
 		(body_style 1)
@@
 		(dnp no)
 		(property "Reference" "TP5"
-			(at 149.0981 50.8 0)
+			(at 144.0181 50.8 0)
 			(hide yes)
 			(show_name no)
@@
 		)
 		(property "Value" "PD_1V8"
-			(at 146.05 48.2601 90)
+			(at 146.558 48.006 90)
 			(show_name no)
 			(do_not_autoplace no)
@@
 		)
 		(property "Footprint" "TestPoint:TestPoint_Loop_D1.80mm_Drill1.0mm_Beaded"
-			(at 151.13 48.26 0)
+			(at 146.05 48.26 0)
 			(hide yes)
 			(show_name no)
@@
 		)
 		(property "Datasheet" ""
-			(at 151.13 48.26 0)
+			(at 146.05 48.26 0)
 			(hide yes)
 			(show_name no)
@@
 		)
 		(property "Description" "test point"
-			(at 151.13 48.26 0)
+			(at 146.05 48.26 0)
 			(hide yes)
 			(show_name no)

Commit message: halleffectsense
Parts:
- renumbered C63 to C10, C64 to C11, C65 to C12, C66 to C13, C67 to C14, C68 to C15, C69 to C16, C70 to C17, C71 to C18, D1 to D17, D2 to D18, D3 to D19, D16 to D20, IC4 to IC2, Q6 to Q3, Q7 to Q4, Q8 to Q5, R7 to R21, R15 to R22, R46 to R23, R47 to R24, R57 to R25, R58 to R26, R59 to R27, R60 to R28, R61 to R29, R62 to R30, R63 to R31, R64 to R32, R65 to R33, R66 to R34, R67 to R35, TP1 to TP13, TP2 to TP14, TP4 to TP15, TP5 to TP16, TP6 to TP17, TP12 to TP18

Commit message: shuntschem2
Parts:
- removed R33, R34: 2.2k, Resistor_SMD:R_0603_1608Metric_Pad0.98x0.95mm_HandSolder, symbol Device:R_Small

Commit message: footprints1
Parts:
- renumbered D17 to D18, D18 to D19, D19 to D20, D20 to D21, R21 to R22, R22 to R23, R23 to R24, R24 to R25, R25 to R26, R26 to R27, R27 to R28, R28 to R29, R29 to R30, R30 to R31, R31 to R32, R32 to R33, R35 to R34, TP13 to TP11, TP14 to TP12, TP15 to TP13, TP16 to TP14, TP17 to TP15, TP18 to TP16
Changed lines of the file:
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@@
 		(in_pos_files yes)
 		(dnp no)
-		(property "Reference" "D18"
+		(property "Reference" "D19"
 			(at 99.06 145.5419 90)
 			(show_name no)
@@
 			(project "PS-SuppChargerPCB"
 				(path "/bb6ce8fd-e1af-464e-bfef-c3b4f18a2cee/0c013a70-ec03-4913-a24e-33c4630278d4"
-					(reference "D18")
+					(reference "D19")
 					(unit 1)
 				)
@@
 		(in_pos_files yes)
 		(dnp no)
-		(property "Reference" "R35"
+		(property "Reference" "R34"
 			(at 255.27 83.82 0)
 			(show_name no)
@@
 			(project "PS-SuppChargerPCB"
 				(path "/bb6ce8fd-e1af-464e-bfef-c3b4f18a2cee/0c013a70-ec03-4913-a24e-33c4630278d4"
-					(reference "R35")
+					(reference "R34")
 					(unit 1)
 				)
@@
 		(in_pos_files yes)
 		(dnp no)
-		(property "Reference" "R25"
+		(property "Reference" "R26"
 			(at 49.53 146.0499 0)
 			(show_name no)
@@
 			(project "PS-SuppChargerPCB"
 				(path "/bb6ce8fd-e1af-464e-bfef-c3b4f18a2cee/0c013a70-ec03-4913-a24e-33c4630278d4"
-					(reference "R25")
+					(reference "R26")
 					(unit 1)
 				)
@@
 		(dnp no)
 		(fields_autoplaced yes)
-		(property "Reference" "R22"
+		(property "Reference" "R23"
 			(at 43.18 93.9799 0)
 			(show_name no)
@@
 			(project "PS-SuppChargerPCB"
 				(path "/bb6ce8fd-e1af-464e-bfef-c3b4f18a2cee/0c013a70-ec03-4913-a24e-33c4630278d4"
-					(reference "R22")
+					(reference "R23")
 					(unit 1)
 				)
@@
 		(in_pos_files yes)
 		(dnp no)
-		(property "Reference" "TP18"
+		(property "Reference" "TP16"
 			(at 243.84 109.9819 0)
 			(hide yes)
@@
 			(project "PS-SuppChargerPCB"
 				(path "/bb6ce8fd-e1af-464e-bfef-c3b4f18a2cee/0c013a70-ec03-4913-a24e-33c4630278d4"
-					(reference "TP18")
+					(reference "TP16")
 					(unit 1)
 				)
@@
 		(in_pos_files yes)
 		(dnp no)
-		(property "Reference" "TP15"
+		(property "Reference" "TP13"
 			(at 135.89 164.3381 0)
 			(hide yes)
@@
 			(project "PS-SuppChargerPCB"
 				(path "/bb6ce8fd-e1af-464e-bfef-c3b4f18a2cee/0c013a70-ec03-4913-a24e-33c4630278d4"
-					(reference "TP15")
+					(reference "TP13")
 					(unit 1)
 				)
@@
 		(dnp no)
 		(fields_autoplaced yes)
-		(property "Reference" "R24"
+		(property "Reference" "R25"
 			(at 41.91 184.15 90)
 			(show_name no)
@@
 			(project "PS-SuppChargerPCB"
 				(path "/bb6ce8fd-e1af-464e-bfef-c3b4f18a2cee/0c013a70-ec03-4913-a24e-33c4630278d4"
-					(reference "R24")
+					(reference "R25")
 					(unit 1)
 				)
@@
 		(in_pos_files yes)
 		(dnp no)
-		(property "Reference" "R29"
+		(property "Reference" "R30"
 			(at 82.55 60.96 0)
 			(show_name no)
@@
 			(project "PS-SuppChargerPCB"
 				(path "/bb6ce8fd-e1af-464e-bfef-c3b4f18a2cee/0c013a70-ec03-4913-a24e-33c4630278d4"
-					(reference "R29")
+					(reference "R30")
 					(unit 1)
 				)
@@
 		(in_pos_files yes)
 		(dnp no)
-		(property "Reference" "R32"
+		(property "Reference" "R33"
 			(at 177.8 58.42 0)
 			(show_name no)
@@
 			(project "PS-SuppChargerPCB"
 				(path "/bb6ce8fd-e1af-464e-bfef-c3b4f18a2cee/0c013a70-ec03-4913-a24e-33c4630278d4"
-					(reference "R32")
+					(reference "R33")
 					(unit 1)
 				)
@@
 		(in_pos_files yes)
 		(dnp no)
-		(property "Reference" "D17"
+		(property "Reference" "D18"
 			(at 38.862 54.102 90)
 			(show_name no)
@@
 			(project "PS-SuppChargerPCB"
 				(path "/bb6ce8fd-e1af-464e-bfef-c3b4f18a2cee/0c013a70-ec03-4913-a24e-33c4630278d4"
-					(reference "D17")
+					(reference "D18")
 					(unit 1)
 				)
@@
 		(dnp no)
 		(fields_autoplaced yes)
-		(property "Reference" "D20"
+		(property "Reference" "D21"
 			(at 257.81 93.0274 90)
 			(show_name no)
@@
 			(project "PS-SuppChargerPCB"
 				(path "/bb6ce8fd-e1af-464e-bfef-c3b4f18a2cee/0c013a70-ec03-4913-a24e-33c4630278d4"
-					(reference "D20")
+					(reference "D21")
 					(unit 1)
 				)
@@
 		(in_pos_files yes)
 		(dnp no)
-		(property "Reference" "R30"
+		(property "Reference" "R31"
 			(at 82.55 92.71 0)
 			(show_name no)
@@
 			(project "PS-SuppChargerPCB"
 				(path "/bb6ce8fd-e1af-464e-bfef-c3b4f18a2cee/0c013a70-ec03-4913-a24e-33c4630278d4"
-					(reference "R30")
+					(reference "R31")
 					(unit 1)
 				)
@@
 		(in_pos_files yes)
 		(dnp no)
-		(property "Reference" "R27"
+		(property "Reference" "R28"
 			(at 74.93 63.5 90)
 			(show_name no)
@@
 			(project "PS-SuppChargerPCB"
 				(path "/bb6ce8fd-e1af-464e-bfef-c3b4f18a2cee/0c013a70-ec03-4913-a24e-33c4630278d4"
-					(reference "R27")
+					(reference "R28")
 					(unit 1)
 				)
@@
 		(in_pos_files yes)
 		(dnp no)
-		(property "Reference" "TP14"
+		(property "Reference" "TP12"
 			(at 135.89 131.3181 0)
 			(hide yes)
@@
 			(project "PS-SuppChargerPCB"
 				(path "/bb6ce8fd-e1af-464e-bfef-c3b4f18a2cee/0c013a70-ec03-4913-a24e-33c4630278d4"
-					(reference "TP14")
+					(reference "TP12")
 					(unit 1)
 				)
@@
 		(dnp no)
 		(fields_autoplaced yes)
-		(property "Reference" "R23"
+		(property "Reference" "R24"
 			(at 41.91 151.13 90)
 			(show_name no)
@@
 			(project "PS-SuppChargerPCB"
 				(path "/bb6ce8fd-e1af-464e-bfef-c3b4f18a2cee/0c013a70-ec03-4913-a24e-33c4630278d4"
-					(reference "R23")
+					(reference "R24")
 					(unit 1)
 				)
@@
 		(dnp no)
 		(fields_autoplaced yes)
-		(property "Reference" "R21"
+		(property "Reference" "R22"
 			(at 27.94 93.9799 0)
 			(show_name no)
@@
 			(project "PS-SuppChargerPCB"
 				(path "/bb6ce8fd-e1af-464e-bfef-c3b4f18a2cee/0c013a70-ec03-4913-a24e-33c4630278d4"
-					(reference "R21")
+					(reference "R22")
 					(unit 1)
 				)
@@
 		(dnp no)
 		(fields_autoplaced yes)
-		(property "Reference" "TP13"
+		(property "Reference" "TP11"
 			(at 41.91 44.9581 0)
 			(hide yes)
@@
 			(project "PS-SuppChargerPCB"
 				(path "/bb6ce8fd-e1af-464e-bfef-c3b4f18a2cee/0c013a70-ec03-4913-a24e-33c4630278d4"
-					(reference "TP13")
+					(reference "TP11")
 					(unit 1)
 				)
@@
 		(in_pos_files yes)
 		(dnp no)
-		(property "Reference" "TP17"
+		(property "Reference" "TP15"
 			(at 170.9419 45.72 0)
 			(hide yes)
@@
 			(project "PS-SuppChargerPCB"
 				(path "/bb6ce8fd-e1af-464e-bfef-c3b4f18a2cee/0c013a70-ec03-4913-a24e-33c4630278d4"
-					(reference "TP17")
+					(reference "TP15")
 					(unit 1)
 				)
@@
 		(dnp no)
 		(fields_autoplaced yes)
-		(property "Reference" "R26"
+		(property "Reference" "R27"
 			(at 49.53 179.0699 0)
 			(show_name no)
@@
 			(project "PS-SuppChargerPCB"
 				(path "/bb6ce8fd-e1af-464e-bfef-c3b4f18a2cee/0c013a70-ec03-4913-a24e-33c4630278d4"
-					(reference "R26")
+					(reference "R27")
 					(unit 1)
 				)
@@
 		(in_pos_files yes)
 		(dnp no)
-		(property "Reference" "R31"
+		(property "Reference" "R32"
 			(at 86.36 146.0499 0)
 			(show_name no)
@@
 			(project "PS-SuppChargerPCB"
 				(path "/bb6ce8fd-e1af-464e-bfef-c3b4f18a2cee/0c013a70-ec03-4913-a24e-33c4630278d4"
-					(reference "R31")
+					(reference "R32")
 					(unit 1)
 				)
@@
 		(in_pos_files yes)
 		(dnp no)
-		(property "Reference" "TP16"
+		(property "Reference" "TP14"
 			(at 144.0181 50.8 0)
 			(hide yes)
@@
 			(project "PS-SuppChargerPCB"
 				(path "/bb6ce8fd-e1af-464e-bfef-c3b4f18a2cee/0c013a70-ec03-4913-a24e-33c4630278d4"
-					(reference "TP16")
+					(reference "TP14")
 					(unit 1)
 				)
@@
 		(in_pos_files yes)
 		(dnp no)
-		(property "Reference" "D19"
+		(property "Reference" "D20"
 			(at 99.06 178.5619 90)
 			(show_name no)
@@
 			(project "PS-SuppChargerPCB"
 				(path "/bb6ce8fd-e1af-464e-bfef-c3b4f18a2cee/0c013a70-ec03-4913-a24e-33c4630278d4"
-					(reference "D19")
+					(reference "D20")
 					(unit 1)
 				)
@@
 		(in_pos_files yes)
 		(dnp no)
-		(property "Reference" "R28"
+		(property "Reference" "R29"
 			(at 74.93 95.25 90)
 			(show_name no)
@@
 			(project "PS-SuppChargerPCB"
 				(path "/bb6ce8fd-e1af-464e-bfef-c3b4f18a2cee/0c013a70-ec03-4913-a24e-33c4630278d4"
-					(reference "R28")
+					(reference "R29")
 					(unit 1)
 				)

Commit message: layout1
Parts:
- C10, C11, C12, C13, C14, C15, C16, C17, C18, D21, R22, R23, R24, R25, R26, R27, R28, R29, R30, R31, R32, R33, R34: KiLib_Generator (none) -> SMD_2terminal_chip_molded
- Q5: KiLib_Generator (none) -> package/gullwing
