File: USB_PD.kicad_sch (KiCad schematic)
At the start: 36 parts, among them IC2 CYPD3177-24LQXQ, Q3 SI7997DP-T1-GE3, Q4 SI7997DP-T1-GE3, Q5 IRLML0030

Commit message: layout5
Parts:
- removed TP12: PD_VBUS_OUT, TestPoint:TestPoint_Loop_D1.80mm_Drill1.0mm_Beaded, symbol lhrs_misc:Multimeter_TP
- removed TP13: PD_5V_OUT, TestPoint:TestPoint_Loop_D1.80mm_Drill1.0mm_Beaded, symbol lhrs_misc:Multimeter_TP
- renumbered C15 to C10, C16 to C11, C17 to C12, C18 to C13, C10 to C14, C11 to C15, C13 to C16, C12 to C17, C14 to C18, D21 to D19, D19 to D20, D20 to D21, Q5 to Q3, Q3 to Q4, Q4 to Q5, R28 to R22, R33 to R23, R30 to R24, R34 to R25, R29 to R26, R31 to R27, R22 to R28, R23 to R29, R26 to R30, R32 to R31, R24 to R32, R27 to R33, R25 to R34, TP14 to TP12, TP15 to TP13, TP16 to TP14

Commit message: layout6
Parts:
- removed TP11: VBUS_IN, TestPoint:TestPoint_Loop_D1.80mm_Drill1.0mm_Beaded, symbol lhrs_misc:Multimeter_TP
Changed lines of the file:
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@@
 	)
 	(junction
-		(at 44.45 46.99)
-		(diameter 0)
-		(color 0 0 0 0)
-	)
-	(junction
 		(at 157.48 107.95)
 		(diameter 0)
@@
 					(unit 1)
 				)
-			)
-		)
-	)
-	(symbol
-		(lib_id "lhrs_misc:Multimeter_TP")
-		(at 44.45 41.91 0)
-		(unit 1)
-		(body_style 1)
-		(exclude_from_sim no)
-		(in_bom yes)
-		(on_board yes)
-		(in_pos_files yes)
-		(dnp no)
-		(property "Reference" "TP11"
-			(at 41.91 39.8781 0)
-			(hide yes)
-			(show_name no)
-			(do_not_autoplace no)
-			(effects
-				(font
-					(size 1.27 1.27)
-				)
-				(justify right)
-			)
-		)
-		(property "Value" "VBUS_IN"
-			(at 46.228 43.688 0)
-			(show_name no)
-			(do_not_autoplace no)
-			(effects
-				(font
-					(size 1.27 1.27)
-				)
-				(justify left)
-			)
-		)
-		(property "Footprint" "TestPoint:TestPoint_Loop_D1.80mm_Drill1.0mm_Beaded"
-			(at 44.45 41.91 0)
-			(hide yes)
-			(show_name no)
-			(do_not_autoplace no)
-			(effects
-				(font
-					(size 1.27 1.27)
-				)
-			)
-		)
-		(property "Datasheet" ""
-			(at 44.45 41.91 0)
-			(hide yes)
-			(show_name no)
-			(do_not_autoplace no)
-			(effects
-				(font
-					(size 1.27 1.27)
-				)
-			)
-		)
-		(property "Description" "test point"
-			(at 44.45 41.91 0)
-			(hide yes)
-			(show_name no)
-			(do_not_autoplace no)
-			(effects
-				(font
-					(size 1.27 1.27)
-				)
-			)
-		)
-		(pin "1"
-		)
-		(instances
-			(project "PS-SuppChargerPCB"
-				(path "/bb6ce8fd-e1af-464e-bfef-c3b4f18a2cee/0c013a70-ec03-4913-a24e-33c4630278d4"
-					(reference "TP11")
-					(unit 1)
-				)
-			)
-			(project "USB_PD"
-				(path "/f5eb7f8f-b132-4f9a-b322-f4fca6115cc9"
-					(reference "TP3")
-					(unit 1)
-				)
