File: 12VBuck.kicad_sch (KiCad schematic)
At the start: 14 parts, among them U1 LMR51635XDDCR

Commit message: schematic5
Changed lines of the file:
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@@
-	(wire
-		(pts
-			(xy 1.3462 1.3462) (xy 2.6162 1.3462)
-		)
-		(stroke
-			(width 0)
-			(type default)
-		)
-	)
 	(wire
 		(pts
@@
 		)
 		(stroke
-			(width 0)
-			(type default)
-		)
-	)
-	(wire
-		(pts
-			(xy 0.0762 0.0762) (xy 1.3462 0.0762)
-		)
-		(stroke

Commit message: schematic7
Parts:
- U1: footprint DDC0006A-MFG -> LHRS_ICs:DDC0006A-MFG
Changed lines of the file:
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@@
 			)
 		)
-		(property "Footprint" "DDC0006A-MFG"
+		(property "Footprint" "LHRS_ICs:DDC0006A-MFG"
 			(at 114.3 81.28 0)
 			(hide yes)

Commit message: fixedsharepoint
Parts:
- removed TP10: SW, TestPoint:TestPoint_THTPad_D3.0mm_Drill1.5mm, symbol Connector:TestPoint
- removed TP7: V_in_12V, TestPoint:TestPoint_THTPad_D3.0mm_Drill1.5mm, symbol Connector:TestPoint
- removed TP8: CB, TestPoint:TestPoint_THTPad_D3.0mm_Drill1.5mm, symbol Connector:TestPoint
- removed TP9: FB, TestPoint:TestPoint_THTPad_D3.0mm_Drill1.5mm, symbol Connector:TestPoint
- L1: footprint LHRS_Passives:74439369082 -> LHRS_Power:XAL5050822MEC; LCSC P/N (none) -> C5309356; P/N 74439369082 -> XAL5050-822MEC
- U1: footprint LHRS_ICs:DDC0006A-MFG -> DDC0006A-MFG; LCSC P/N (none) -> C42432812; P/N (none) -> LMR51635XDDCR
- renumbered R16 to R8, R17 to R9
Other:
- note added: "Vin: 4.6V to 60V"
- note removed: "Test Points"

Commit message: schematic9
Parts:
- U1: footprint DDC0006A-MFG -> LHRS_ICs:DDC0006A-MFG
Changed lines of the file:
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@@
 			)
 		)
-		(property "Footprint" "DDC0006A-MFG"
+		(property "Footprint" "LHRS_ICs:DDC0006A-MFG"
 			(at 114.3 81.28 0)
 			(hide yes)

Commit message: halleffectsense
Parts:
- renumbered C10 to C39, C11 to C40, C12 to C41, C13 to C42, C14 to C43, C15 to C44, L1 to L2, R8 to R47, R9 to R48, U1 to U3
Changed lines of the file:
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@@
 		(dnp no)
 		(fields_autoplaced yes)
-		(property "Reference" "C10"
+		(property "Reference" "C39"
 			(at 96.52 85.0962 0)
 			(show_name no)
@@
 			(project "PS-SuppChargerPCB"
 				(path "/bb6ce8fd-e1af-464e-bfef-c3b4f18a2cee/aebf5d4f-ef40-4f0d-9b6a-e87c6af87ba8"
-					(reference "C10")
+					(reference "C39")
 					(unit 1)
 				)
@@
 		(in_pos_files yes)
 		(dnp no)
-		(property "Reference" "L1"
+		(property "Reference" "L2"
 			(at 161.29 87.884 90)
 			(show_name no)
@@
 			(project "PS-SuppChargerPCB"
 				(path "/bb6ce8fd-e1af-464e-bfef-c3b4f18a2cee/aebf5d4f-ef40-4f0d-9b6a-e87c6af87ba8"
-					(reference "L1")
+					(reference "L2")
 					(unit 1)
 				)
@@
 		(in_pos_files yes)
 		(dnp no)
-		(property "Reference" "C13"
+		(property "Reference" "C42"
 			(at 164.084 93.98 0)
 			(show_name no)
@@
 			(project "PS-SuppChargerPCB"
 				(path "/bb6ce8fd-e1af-464e-bfef-c3b4f18a2cee/aebf5d4f-ef40-4f0d-9b6a-e87c6af87ba8"
-					(reference "C13")
+					(reference "C42")
 					(unit 1)
 				)
@@
 		(in_pos_files yes)
 		(dnp no)
-		(property "Reference" "C15"
+		(property "Reference" "C44"
 			(at 189.992 93.98 0)
 			(show_name no)
@@
 			(project "PS-SuppChargerPCB"
 				(path "/bb6ce8fd-e1af-464e-bfef-c3b4f18a2cee/aebf5d4f-ef40-4f0d-9b6a-e87c6af87ba8"
-					(reference "C15")
+					(reference "C44")
 					(unit 1)
 				)
@@
 		(in_pos_files yes)
 		(dnp no)
-		(property "Reference" "C12"
+		(property "Reference" "C41"
 			(at 156.718 80.01 0)
 			(show_name no)
@@
 			(project "PS-SuppChargerPCB"
 				(path "/bb6ce8fd-e1af-464e-bfef-c3b4f18a2cee/aebf5d4f-ef40-4f0d-9b6a-e87c6af87ba8"
-					(reference "C12")
+					(reference "C41")
 					(unit 1)
 				)
@@
 		(dnp no)
 		(fields_autoplaced yes)
-		(property "Reference" "R8"
+		(property "Reference" "R47"
 			(at 227.33 85.0899 0)
 			(show_name no)
@@
 			(project "PS-SuppChargerPCB"
 				(path "/bb6ce8fd-e1af-464e-bfef-c3b4f18a2cee/aebf5d4f-ef40-4f0d-9b6a-e87c6af87ba8"
-					(reference "R8")
+					(reference "R47")
 					(unit 1)
 				)
@@
 		(dnp no)
 		(fields_autoplaced yes)
-		(property "Reference" "C11"
+		(property "Reference" "C40"
 			(at 105.41 87.6362 0)
 			(show_name no)
@@
 			(project "PS-SuppChargerPCB"
 				(path "/bb6ce8fd-e1af-464e-bfef-c3b4f18a2cee/aebf5d4f-ef40-4f0d-9b6a-e87c6af87ba8"
-					(reference "C11")
+					(reference "C40")
 					(unit 1)
 				)
@@
 		(dnp no)
 		(fields_autoplaced yes)
-		(property "Reference" "R9"
+		(property "Reference" "R48"
 			(at 227.33 92.7099 0)
 			(show_name no)
@@
 			(project "PS-SuppChargerPCB"
 				(path "/bb6ce8fd-e1af-464e-bfef-c3b4f18a2cee/aebf5d4f-ef40-4f0d-9b6a-e87c6af87ba8"
-					(reference "R9")
+					(reference "R48")
 					(unit 1)
 				)
@@
 		(in_pos_files yes)
 		(dnp no)
-		(property "Reference" "C14"
+		(property "Reference" "C43"
 			(at 173.482 94.234 0)
 			(show_name no)
@@
 			(project "PS-SuppChargerPCB"
 				(path "/bb6ce8fd-e1af-464e-bfef-c3b4f18a2cee/aebf5d4f-ef40-4f0d-9b6a-e87c6af87ba8"
-					(reference "C14")
+					(reference "C43")
 					(unit 1)
 				)
@@
 		(dnp no)
 		(fields_autoplaced yes)
-		(property "Reference" "U1"
+		(property "Reference" "U3"
 			(at 129.54 71.12 0)
 			(show_name no)
@@
 			(project "PS-SuppChargerPCB"
 				(path "/bb6ce8fd-e1af-464e-bfef-c3b4f18a2cee/aebf5d4f-ef40-4f0d-9b6a-e87c6af87ba8"
-					(reference "U1")
-					(unit 1)
-				)
+					(reference "U3")
+					(unit 1)
+				)

Commit message: footprints1
Parts:
- renumbered C39 to C37, C40 to C38, C41 to C39, C42 to C40, C43 to C41, C44 to C42, R47 to R46, R48 to R47
Changed lines of the file:
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@@
 		(dnp no)
 		(fields_autoplaced yes)
-		(property "Reference" "C39"
+		(property "Reference" "C37"
 			(at 96.52 85.0962 0)
 			(show_name no)
@@
 			(project "PS-SuppChargerPCB"
 				(path "/bb6ce8fd-e1af-464e-bfef-c3b4f18a2cee/aebf5d4f-ef40-4f0d-9b6a-e87c6af87ba8"
-					(reference "C39")
+					(reference "C37")
 					(unit 1)
 				)
@@
 		(in_pos_files yes)
 		(dnp no)
-		(property "Reference" "C42"
+		(property "Reference" "C40"
 			(at 164.084 93.98 0)
 			(show_name no)
@@
 			(project "PS-SuppChargerPCB"
 				(path "/bb6ce8fd-e1af-464e-bfef-c3b4f18a2cee/aebf5d4f-ef40-4f0d-9b6a-e87c6af87ba8"
-					(reference "C42")
+					(reference "C40")
 					(unit 1)
 				)
@@
 		(in_pos_files yes)
 		(dnp no)
-		(property "Reference" "C44"
+		(property "Reference" "C42"
 			(at 189.992 93.98 0)
 			(show_name no)
@@
 			(project "PS-SuppChargerPCB"
 				(path "/bb6ce8fd-e1af-464e-bfef-c3b4f18a2cee/aebf5d4f-ef40-4f0d-9b6a-e87c6af87ba8"
-					(reference "C44")
+					(reference "C42")
 					(unit 1)
 				)
@@
 		(in_pos_files yes)
 		(dnp no)
-		(property "Reference" "C41"
+		(property "Reference" "C39"
 			(at 156.718 80.01 0)
 			(show_name no)
@@
 			(project "PS-SuppChargerPCB"
 				(path "/bb6ce8fd-e1af-464e-bfef-c3b4f18a2cee/aebf5d4f-ef40-4f0d-9b6a-e87c6af87ba8"
-					(reference "C41")
+					(reference "C39")
 					(unit 1)
 				)
@@
 		(dnp no)
 		(fields_autoplaced yes)
-		(property "Reference" "R47"
+		(property "Reference" "R46"
 			(at 227.33 85.0899 0)
 			(show_name no)
@@
 			(project "PS-SuppChargerPCB"
 				(path "/bb6ce8fd-e1af-464e-bfef-c3b4f18a2cee/aebf5d4f-ef40-4f0d-9b6a-e87c6af87ba8"
-					(reference "R47")
+					(reference "R46")
 					(unit 1)
 				)
@@
 		(dnp no)
 		(fields_autoplaced yes)
-		(property "Reference" "C40"
+		(property "Reference" "C38"
 			(at 105.41 87.6362 0)
 			(show_name no)
@@
 			(project "PS-SuppChargerPCB"
 				(path "/bb6ce8fd-e1af-464e-bfef-c3b4f18a2cee/aebf5d4f-ef40-4f0d-9b6a-e87c6af87ba8"
-					(reference "C40")
+					(reference "C38")
 					(unit 1)
 				)
@@
 		(dnp no)
 		(fields_autoplaced yes)
-		(property "Reference" "R48"
+		(property "Reference" "R47"
 			(at 227.33 92.7099 0)
 			(show_name no)
@@
 			(project "PS-SuppChargerPCB"
 				(path "/bb6ce8fd-e1af-464e-bfef-c3b4f18a2cee/aebf5d4f-ef40-4f0d-9b6a-e87c6af87ba8"
-					(reference "R48")
+					(reference "R47")
 					(unit 1)
 				)
@@
 		(in_pos_files yes)
 		(dnp no)
-		(property "Reference" "C43"
+		(property "Reference" "C41"
 			(at 173.482 94.234 0)
 			(show_name no)
@@
 			(project "PS-SuppChargerPCB"
 				(path "/bb6ce8fd-e1af-464e-bfef-c3b4f18a2cee/aebf5d4f-ef40-4f0d-9b6a-e87c6af87ba8"
-					(reference "C43")
-					(unit 1)
-				)
+					(reference "C41")
+					(unit 1)
+				)

Commit message: layout1
Parts:
- C37, C38, C39, C40, C41, C42, R46, R47: KiLib_Generator (none) -> SMD_2terminal_chip_molded
Changed lines of the file:
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@@
+			)
+		)
+		(property "KiLib_Generator" "SMD_2terminal_chip_molded"
+			(at 93.98 86.36 0)
+			(hide yes)
+			(show_name no)
+			(do_not_autoplace no)
+			(effects
+				(font
+					(size 1.27 1.27)
+				)
 			)
 		)
@@
 			)
 		)
+		(property "KiLib_Generator" "SMD_2terminal_chip_molded"
+			(at 170.18 95.25 0)
+			(hide yes)
+			(show_name no)
+			(do_not_autoplace no)
+			(effects
+				(font
+					(size 1.27 1.27)
+				)
+			)
+		)
 		(pin "2"
 		)
@@
 			)
 		)
+		(property "KiLib_Generator" "SMD_2terminal_chip_molded"
+			(at 186.69 95.25 0)
+			(hide yes)
+			(show_name no)
+			(do_not_autoplace no)
+			(effects
+				(font
+					(size 1.27 1.27)
+				)
+			)
+		)
 		(pin "2"
 		)
@@
 		)
 		(property "LCSC P/N" "C6666325"
+			(at 153.67 83.82 0)
+			(hide yes)
+			(show_name no)
+			(do_not_autoplace no)
+			(effects
+				(font
+					(size 1.27 1.27)
+				)
+			)
+		)
+		(property "KiLib_Generator" "SMD_2terminal_chip_molded"
 			(at 153.67 83.82 0)
 			(hide yes)
@@
 			)
 		)
+		(property "KiLib_Generator" "SMD_2terminal_chip_molded"
+			(at 224.79 86.36 0)
+			(hide yes)
+			(show_name no)
+			(do_not_autoplace no)
+			(effects
+				(font
+					(size 1.27 1.27)
+				)
+			)
+		)
 		(pin "1"
 		)
@@
 			)
 		)
+		(property "KiLib_Generator" "SMD_2terminal_chip_molded"
+			(at 102.87 88.9 0)
+			(hide yes)
+			(show_name no)
+			(do_not_autoplace no)
+			(effects
+				(font
+					(size 1.27 1.27)
+				)
+			)
+		)
 		(pin "1"
 		)
@@
 			)
 		)
+		(property "KiLib_Generator" "SMD_2terminal_chip_molded"
+			(at 224.79 93.98 0)
+			(hide yes)
+			(show_name no)
+			(do_not_autoplace no)
+			(effects
+				(font
+					(size 1.27 1.27)
+				)
+			)
+		)
 		(pin "1"
 		)
@@
 			(at 179.07 95.25 0)
 			(hide yes)
+			(show_name no)
+			(do_not_autoplace no)
+			(effects
+				(font
+					(size 1.27 1.27)
+				)
+			)
+		)
+		(property "KiLib_Generator" "SMD_2terminal_chip_molded"
+			(at 179.07 95.25 0)
+			(hide yes)

Commit message: layout5
Parts:
- renumbered C39 to C37, C37 to C38, C38 to C39
Changed lines of the file:
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@@
 		(dnp no)
 		(fields_autoplaced yes)
-		(property "Reference" "C37"
+		(property "Reference" "C38"
 			(at 96.52 85.0962 0)
 			(show_name no)
@@
 			(project "PS-SuppChargerPCB"
 				(path "/bb6ce8fd-e1af-464e-bfef-c3b4f18a2cee/aebf5d4f-ef40-4f0d-9b6a-e87c6af87ba8"
-					(reference "C37")
+					(reference "C38")
 					(unit 1)
 				)
@@
 		(in_pos_files yes)
 		(dnp no)
-		(property "Reference" "C39"
+		(property "Reference" "C37"
 			(at 156.718 80.01 0)
 			(show_name no)
@@
 			(project "PS-SuppChargerPCB"
 				(path "/bb6ce8fd-e1af-464e-bfef-c3b4f18a2cee/aebf5d4f-ef40-4f0d-9b6a-e87c6af87ba8"
-					(reference "C39")
+					(reference "C37")
 					(unit 1)
 				)
@@
 		(dnp no)
 		(fields_autoplaced yes)
-		(property "Reference" "C38"
+		(property "Reference" "C39"
 			(at 105.41 87.6362 0)
 			(show_name no)
@@
 			(project "PS-SuppChargerPCB"
 				(path "/bb6ce8fd-e1af-464e-bfef-c3b4f18a2cee/aebf5d4f-ef40-4f0d-9b6a-e87c6af87ba8"
-					(reference "C38")
-					(unit 1)
-				)
+					(reference "C39")
+					(unit 1)
+				)
