File: PowerProtection.kicad_sch (KiCad schematic)
At the start: 18 parts, among them IC3 LM74502DDFR, Q4 PSMN012-100YS, Q5 PSMN012-100YS

Commit message: fixedsharepoint
Parts:
- IC3: Manufacturer_Name Texas Instruments -> (none); Manufacturer_Part_Number LM74502DDFR -> (none); Mouser Part Number 595-LM74502DDFR -> (none); Mouser Price/Stock https://www.mouser.co.uk/ProductDetail/Texas-Instruments/LM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 -> (none)
- R29, R35, R36, R43, R44: symbol Device:R_US -> Device:R
- R30: symbol Device:R_US -> Device:R; Mouser Part Number 594-MCT06030C3309FP5 -> (none)
Connections:
- net PS_Vout is gone; now on net Vin: R35.1, R43.1
- net PP_Vout renamed Vout
Other:
- note added: "Supp Battery Range: 10V-14.7V"
- note removed: "Make them bananajacks in footprint"
- note removed: "Two one by one connectors"
- title: (none) -> Power Protection
- moved on the sheet: C34, C47, C58, C60, C61, C62, D13, D14, IC3, Q4, Q5

Commit message: halleffectsense
Parts:
- renumbered C34 to C3, C47 to C4, C58 to C5, C59 to C6, C60 to C7, C61 to C8, C62 to C9, D13 to D15, D14 to D16, IC3 to IC1, Q4 to Q1, Q5 to Q2, R29 to R15, R30 to R16, R35 to R17, R36 to R18, R43 to R19, R44 to R20
Changed lines of the file:
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@@
 		(in_pos_files yes)
 		(dnp no)
-		(property "Reference" "D14"
+		(property "Reference" "D16"
 			(at 40.64 82.296 0)
 			(show_name no)
@@
 			(project "PS-SuppChargerPCB"
 				(path "/bb6ce8fd-e1af-464e-bfef-c3b4f18a2cee/2cf5818b-529e-491f-8ffd-d4b5d2111841"
-					(reference "D14")
+					(reference "D16")
 					(unit 1)
 				)
@@
 		(dnp no)
 		(fields_autoplaced yes)
-		(property "Reference" "C58"
+		(property "Reference" "C5"
 			(at 57.785 80.0099 0)
 			(show_name no)
@@
 			(project "PS-SuppChargerPCB"
 				(path "/bb6ce8fd-e1af-464e-bfef-c3b4f18a2cee/2cf5818b-529e-491f-8ffd-d4b5d2111841"
-					(reference "C58")
+					(reference "C5")
 					(unit 1)
 				)
@@
 		(in_pos_files yes)
 		(dnp no)
-		(property "Reference" "D13"
+		(property "Reference" "D15"
 			(at 22.606 49.276 0)
 			(show_name no)
@@
 			(project "PS-SuppChargerPCB"
 				(path "/bb6ce8fd-e1af-464e-bfef-c3b4f18a2cee/2cf5818b-529e-491f-8ffd-d4b5d2111841"
-					(reference "D13")
+					(reference "D15")
 					(unit 1)
 				)
@@
 		(dnp no)
 		(fields_autoplaced yes)
-		(property "Reference" "R29"
+		(property "Reference" "R15"
 			(at 45.72 60.9599 0)
 			(show_name no)
@@
 			(project "PS-SuppChargerPCB"
 				(path "/bb6ce8fd-e1af-464e-bfef-c3b4f18a2cee/2cf5818b-529e-491f-8ffd-d4b5d2111841"
-					(reference "R29")
+					(reference "R15")
 					(unit 1)
 				)
@@
 		(in_pos_files yes)
 		(dnp no)
-		(property "Reference" "R44"
+		(property "Reference" "R20"
 			(at 137.668 90.17 90)
 			(show_name no)
@@
 			(project "PS-SuppChargerPCB"
 				(path "/bb6ce8fd-e1af-464e-bfef-c3b4f18a2cee/2cf5818b-529e-491f-8ffd-d4b5d2111841"
-					(reference "R44")
+					(reference "R20")
 					(unit 1)
 				)
@@
 		(in_pos_files yes)
 		(dnp no)
-		(property "Reference" "C34"
+		(property "Reference" "C3"
 			(at 38.1 49.5299 0)
 			(show_name no)
@@
 			(project "PS-SuppChargerPCB"
 				(path "/bb6ce8fd-e1af-464e-bfef-c3b4f18a2cee/2cf5818b-529e-491f-8ffd-d4b5d2111841"
-					(reference "C34")
+					(reference "C3")
 					(unit 1)
 				)
@@
 		(in_pos_files yes)
 		(dnp no)
-		(property "Reference" "R30"
+		(property "Reference" "R16"
 			(at 67.31 54.61 90)
 			(show_name no)
@@
 			(project "PS-SuppChargerPCB"
 				(path "/bb6ce8fd-e1af-464e-bfef-c3b4f18a2cee/2cf5818b-529e-491f-8ffd-d4b5d2111841"
-					(reference "R30")
+					(reference "R16")
 					(unit 1)
 				)
@@
 		(in_pos_files yes)
 		(dnp no)
-		(property "Reference" "IC3"
+		(property "Reference" "IC1"
 			(at 75.184 73.66 0)
 			(show_name no)
@@
 			(project "PS-SuppChargerPCB"
 				(path "/bb6ce8fd-e1af-464e-bfef-c3b4f18a2cee/2cf5818b-529e-491f-8ffd-d4b5d2111841"
-					(reference "IC3")
+					(reference "IC1")
 					(unit 1)
 				)
@@
 		(in_pos_files yes)
 		(dnp no)
-		(property "Reference" "Q4"
+		(property "Reference" "Q1"
 			(at 52.578 38.862 90)
 			(show_name no)
@@
 			(project "PS-SuppChargerPCB"
 				(path "/bb6ce8fd-e1af-464e-bfef-c3b4f18a2cee/2cf5818b-529e-491f-8ffd-d4b5d2111841"
-					(reference "Q4")
+					(reference "Q1")
 					(unit 1)
 				)
@@
 		(in_pos_files yes)
 		(dnp no)
-		(property "Reference" "C61"
+		(property "Reference" "C8"
 			(at 113.284 89.154 0)
 			(show_name no)
@@
 			(project "PS-SuppChargerPCB"
 				(path "/bb6ce8fd-e1af-464e-bfef-c3b4f18a2cee/2cf5818b-529e-491f-8ffd-d4b5d2111841"
-					(reference "C61")
+					(reference "C8")
 					(unit 1)
 				)
@@
 		(in_pos_files yes)
 		(dnp no)
-		(property "Reference" "C59"
+		(property "Reference" "C6"
 			(at 54.864 62.23 0)
 			(show_name no)
@@
 			(project "PS-SuppChargerPCB"
 				(path "/bb6ce8fd-e1af-464e-bfef-c3b4f18a2cee/2cf5818b-529e-491f-8ffd-d4b5d2111841"
-					(reference "C59")
+					(reference "C6")
 					(unit 1)
 				)
@@
 		(in_pos_files yes)
 		(dnp no)
-		(property "Reference" "C60"
+		(property "Reference" "C7"
 			(at 112.395 49.5299 0)
 			(show_name no)
@@
 			(project "PS-SuppChargerPCB"
 				(path "/bb6ce8fd-e1af-464e-bfef-c3b4f18a2cee/2cf5818b-529e-491f-8ffd-d4b5d2111841"
-					(reference "C60")
+					(reference "C7")
 					(unit 1)
 				)
@@
 		(in_pos_files yes)
 		(dnp no)
-		(property "Reference" "Q5"
+		(property "Reference" "Q2"
 			(at 100.584 38.608 90)
 			(show_name no)
@@
 			(project "PS-SuppChargerPCB"
 				(path "/bb6ce8fd-e1af-464e-bfef-c3b4f18a2cee/2cf5818b-529e-491f-8ffd-d4b5d2111841"
-					(reference "Q5")
+					(reference "Q2")
 					(unit 1)
 				)
@@
 		(in_pos_files yes)
 		(dnp no)
-		(property "Reference" "R36"
+		(property "Reference" "R18"
 			(at 118.618 90.424 90)
 			(show_name no)
@@
 			(project "PS-SuppChargerPCB"
 				(path "/bb6ce8fd-e1af-464e-bfef-c3b4f18a2cee/2cf5818b-529e-491f-8ffd-d4b5d2111841"
-					(reference "R36")
+					(reference "R18")
 					(unit 1)
 				)
@@
 		(in_pos_files yes)
 		(dnp no)
-		(property "Reference" "C47"
+		(property "Reference" "C4"
 			(at 31.75 82.5499 0)
 			(show_name no)
@@
 			(project "PS-SuppChargerPCB"
 				(path "/bb6ce8fd-e1af-464e-bfef-c3b4f18a2cee/2cf5818b-529e-491f-8ffd-d4b5d2111841"
-					(reference "C47")
+					(reference "C4")
 					(unit 1)
 				)
@@
 		(in_pos_files yes)
 		(dnp no)
-		(property "Reference" "C62"
+		(property "Reference" "C9"
 			(at 132.08 88.9 0)
 			(show_name no)
@@
 			(project "PS-SuppChargerPCB"
 				(path "/bb6ce8fd-e1af-464e-bfef-c3b4f18a2cee/2cf5818b-529e-491f-8ffd-d4b5d2111841"
-					(reference "C62")
+					(reference "C9")
 					(unit 1)
 				)
@@
 		(in_pos_files yes)
 		(dnp no)
-		(property "Reference" "R35"
+		(property "Reference" "R17"
 			(at 118.11 78.74 90)
 			(show_name no)
@@
 			(project "PS-SuppChargerPCB"
 				(path "/bb6ce8fd-e1af-464e-bfef-c3b4f18a2cee/2cf5818b-529e-491f-8ffd-d4b5d2111841"
-					(reference "R35")
+					(reference "R17")
 					(unit 1)
 				)
@@
 		(in_pos_files yes)
 		(dnp no)
-		(property "Reference" "R43"
+		(property "Reference" "R19"
 			(at 137.16 77.47 90)
 			(show_name no)
@@
 			(project "PS-SuppChargerPCB"
 				(path "/bb6ce8fd-e1af-464e-bfef-c3b4f18a2cee/2cf5818b-529e-491f-8ffd-d4b5d2111841"
-					(reference "R43")
-					(unit 1)
-				)
+					(reference "R19")
+					(unit 1)
+				)

Commit message: footprints1
Parts:
- renumbered D15 to D16, D16 to D17, R15 to R16, R16 to R17, R17 to R18, R18 to R19, R19 to R20, R20 to R21
Changed lines of the file:
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@@
 		(in_pos_files yes)
 		(dnp no)
-		(property "Reference" "D16"
+		(property "Reference" "D17"
 			(at 40.64 82.296 0)
 			(show_name no)
@@
 			(project "PS-SuppChargerPCB"
 				(path "/bb6ce8fd-e1af-464e-bfef-c3b4f18a2cee/2cf5818b-529e-491f-8ffd-d4b5d2111841"
-					(reference "D16")
+					(reference "D17")
 					(unit 1)
 				)
@@
 		(in_pos_files yes)
 		(dnp no)
-		(property "Reference" "D15"
+		(property "Reference" "D16"
 			(at 22.606 49.276 0)
 			(show_name no)
@@
 			(project "PS-SuppChargerPCB"
 				(path "/bb6ce8fd-e1af-464e-bfef-c3b4f18a2cee/2cf5818b-529e-491f-8ffd-d4b5d2111841"
-					(reference "D15")
+					(reference "D16")
 					(unit 1)
 				)
@@
 		(dnp no)
 		(fields_autoplaced yes)
-		(property "Reference" "R15"
+		(property "Reference" "R16"
 			(at 45.72 60.9599 0)
 			(show_name no)
@@
 			(project "PS-SuppChargerPCB"
 				(path "/bb6ce8fd-e1af-464e-bfef-c3b4f18a2cee/2cf5818b-529e-491f-8ffd-d4b5d2111841"
-					(reference "R15")
+					(reference "R16")
 					(unit 1)
 				)
@@
 		(in_pos_files yes)
 		(dnp no)
-		(property "Reference" "R20"
+		(property "Reference" "R21"
 			(at 137.668 90.17 90)
 			(show_name no)
@@
 			(project "PS-SuppChargerPCB"
 				(path "/bb6ce8fd-e1af-464e-bfef-c3b4f18a2cee/2cf5818b-529e-491f-8ffd-d4b5d2111841"
-					(reference "R20")
+					(reference "R21")
 					(unit 1)
 				)
@@
 		(in_pos_files yes)
 		(dnp no)
-		(property "Reference" "R16"
+		(property "Reference" "R17"
 			(at 67.31 54.61 90)
 			(show_name no)
@@
 			(project "PS-SuppChargerPCB"
 				(path "/bb6ce8fd-e1af-464e-bfef-c3b4f18a2cee/2cf5818b-529e-491f-8ffd-d4b5d2111841"
-					(reference "R16")
+					(reference "R17")
 					(unit 1)
 				)
@@
 		(in_pos_files yes)
 		(dnp no)
-		(property "Reference" "R18"
+		(property "Reference" "R19"
 			(at 118.618 90.424 90)
 			(show_name no)
@@
 			(project "PS-SuppChargerPCB"
 				(path "/bb6ce8fd-e1af-464e-bfef-c3b4f18a2cee/2cf5818b-529e-491f-8ffd-d4b5d2111841"
-					(reference "R18")
+					(reference "R19")
 					(unit 1)
 				)
@@
 		(in_pos_files yes)
 		(dnp no)
-		(property "Reference" "R17"
+		(property "Reference" "R18"
 			(at 118.11 78.74 90)
 			(show_name no)
@@
 			(project "PS-SuppChargerPCB"
 				(path "/bb6ce8fd-e1af-464e-bfef-c3b4f18a2cee/2cf5818b-529e-491f-8ffd-d4b5d2111841"
-					(reference "R17")
+					(reference "R18")
 					(unit 1)
 				)
@@
 		(in_pos_files yes)
 		(dnp no)
-		(property "Reference" "R19"
+		(property "Reference" "R20"
 			(at 137.16 77.47 90)
 			(show_name no)
@@
 			(project "PS-SuppChargerPCB"
 				(path "/bb6ce8fd-e1af-464e-bfef-c3b4f18a2cee/2cf5818b-529e-491f-8ffd-d4b5d2111841"
-					(reference "R19")
-					(unit 1)
-				)
+					(reference "R20")
+					(unit 1)
+				)

Commit message: layout1
Parts:
- C3, C4, C5, C6, C7, C8, C9, R16, R17, R18, R19, R20, R21: KiLib_Generator (none) -> SMD_2terminal_chip_molded
Changed lines of the file:
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@@
+			)
+		)
+		(property "KiLib_Generator" "SMD_2terminal_chip_molded"
+			(at 54.61 81.28 0)
+			(hide yes)
+			(show_name no)
+			(do_not_autoplace no)
+			(effects
+				(font
+					(size 1.27 1.27)
+				)
 			)
 		)
@@
 			)
 		)
+		(property "KiLib_Generator" "SMD_2terminal_chip_molded"
+			(at 43.18 62.23 0)
+			(hide yes)
+			(show_name no)
+			(do_not_autoplace no)
+			(effects
+				(font
+					(size 1.27 1.27)
+				)
+			)
+		)
 		(pin "1"
 		)
@@
 			)
 		)
+		(property "KiLib_Generator" "SMD_2terminal_chip_molded"
+			(at 139.7 90.17 0)
+			(hide yes)
+			(show_name no)
+			(do_not_autoplace no)
+			(effects
+				(font
+					(size 1.27 1.27)
+				)
+			)
+		)
 		(pin "1"
 		)
@@
 			)
 		)
+		(property "KiLib_Generator" "SMD_2terminal_chip_molded"
+			(at 34.29 50.8 0)
+			(hide yes)
+			(show_name no)
+			(do_not_autoplace no)
+			(effects
+				(font
+					(size 1.27 1.27)
+				)
+			)
+		)
 		(pin "1"
 		)
@@
 			)
 		)
+		(property "KiLib_Generator" "SMD_2terminal_chip_molded"
+			(at 67.31 57.15 0)
+			(hide yes)
+			(show_name no)
+			(do_not_autoplace no)
+			(effects
+				(font
+					(size 1.27 1.27)
+				)
+			)
+		)
 		(pin "1"
 		)
@@
 			)
 		)
+		(property "KiLib_Generator" "SMD_2terminal_chip_molded"
+			(at 110.49 90.17 0)
+			(hide yes)
+			(show_name no)
+			(do_not_autoplace no)
+			(effects
+				(font
+					(size 1.27 1.27)
+				)
+			)
+		)
 		(pin "1"
 		)
@@
 			)
 		)
+		(property "KiLib_Generator" "SMD_2terminal_chip_molded"
+			(at 60.96 63.5 0)
+			(hide yes)
+			(show_name no)
+			(do_not_autoplace no)
+			(effects
+				(font
+					(size 1.27 1.27)
+				)
+			)
+		)
 		(pin "1"
 		)
@@
 		)
 		(property "LCSC P/N" "C440198"
+			(at 109.22 50.8 0)
+			(hide yes)
+			(show_name no)
+			(do_not_autoplace no)
+			(effects
+				(font
+					(size 1.27 1.27)
+				)
+			)
+		)
+		(property "KiLib_Generator" "SMD_2terminal_chip_molded"
 			(at 109.22 50.8 0)
 			(hide yes)
@@
 			)
 		)
+		(property "KiLib_Generator" "SMD_2terminal_chip_molded"
+			(at 120.65 90.17 0)
+			(hide yes)
+			(show_name no)
+			(do_not_autoplace no)
+			(effects
+				(font
+					(size 1.27 1.27)
+				)
+			)
+		)
 		(pin "1"
 		)
@@
 			)
 		)
+		(property "KiLib_Generator" "SMD_2terminal_chip_molded"
+			(at 35.56 83.82 0)
+			(hide yes)
+			(show_name no)
+			(do_not_autoplace no)
+			(effects
+				(font
+					(size 1.27 1.27)
+				)
+			)
+		)
 		(pin "2"
 		)
@@
 			)
 		)
+		(property "KiLib_Generator" "SMD_2terminal_chip_molded"
+			(at 129.54 90.17 0)
+			(hide yes)
+			(show_name no)
+			(do_not_autoplace no)
+			(effects
+				(font
+					(size 1.27 1.27)
+				)
+			)
+		)
 		(pin "1"
 		)
@@
 			)
 		)
+		(property "KiLib_Generator" "SMD_2terminal_chip_molded"
+			(at 115.57 77.47 0)
+			(hide yes)
+			(show_name no)
+			(do_not_autoplace no)
+			(effects
+				(font
+					(size 1.27 1.27)
+				)
+			)
+		)
 		(pin "1"
 		)
@@
 			(at 134.62 77.47 0)
 			(hide yes)
+			(show_name no)
+			(do_not_autoplace no)
+			(effects
+				(font
+					(size 1.27 1.27)
+				)
+			)
+		)
+		(property "KiLib_Generator" "SMD_2terminal_chip_molded"
+			(at 134.62 77.47 0)
+			(hide yes)

Commit message: layout5
Parts:
- renumbered C7 to C4, C6 to C5, C5 to C6, C4 to C7, R17 to R16, R16 to R17, R20 to R19, R19 to R20
Changed lines of the file:
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@@
 		(dnp no)
 		(fields_autoplaced yes)
-		(property "Reference" "C5"
+		(property "Reference" "C6"
 			(at 57.785 80.0099 0)
 			(show_name no)
@@
 			(project "PS-SuppChargerPCB"
 				(path "/bb6ce8fd-e1af-464e-bfef-c3b4f18a2cee/2cf5818b-529e-491f-8ffd-d4b5d2111841"
-					(reference "C5")
+					(reference "C6")
 					(unit 1)
 				)
@@
 		(dnp no)
 		(fields_autoplaced yes)
-		(property "Reference" "R16"
+		(property "Reference" "R17"
 			(at 45.72 60.9599 0)
 			(show_name no)
@@
 			(project "PS-SuppChargerPCB"
 				(path "/bb6ce8fd-e1af-464e-bfef-c3b4f18a2cee/2cf5818b-529e-491f-8ffd-d4b5d2111841"
-					(reference "R16")
+					(reference "R17")
 					(unit 1)
 				)
@@
 		(in_pos_files yes)
 		(dnp no)
-		(property "Reference" "R17"
+		(property "Reference" "R16"
 			(at 67.31 54.61 90)
 			(show_name no)
@@
 			(project "PS-SuppChargerPCB"
 				(path "/bb6ce8fd-e1af-464e-bfef-c3b4f18a2cee/2cf5818b-529e-491f-8ffd-d4b5d2111841"
-					(reference "R17")
+					(reference "R16")
 					(unit 1)
 				)
@@
 		(in_pos_files yes)
 		(dnp no)
-		(property "Reference" "C6"
+		(property "Reference" "C5"
 			(at 54.864 62.23 0)
 			(show_name no)
@@
 			(project "PS-SuppChargerPCB"
 				(path "/bb6ce8fd-e1af-464e-bfef-c3b4f18a2cee/2cf5818b-529e-491f-8ffd-d4b5d2111841"
-					(reference "C6")
+					(reference "C5")
 					(unit 1)
 				)
@@
 		(in_pos_files yes)
 		(dnp no)
-		(property "Reference" "C7"
+		(property "Reference" "C4"
 			(at 112.395 49.5299 0)
 			(show_name no)
@@
 			(project "PS-SuppChargerPCB"
 				(path "/bb6ce8fd-e1af-464e-bfef-c3b4f18a2cee/2cf5818b-529e-491f-8ffd-d4b5d2111841"
-					(reference "C7")
+					(reference "C4")
 					(unit 1)
 				)
@@
 		(in_pos_files yes)
 		(dnp no)
-		(property "Reference" "R19"
+		(property "Reference" "R20"
 			(at 118.618 90.424 90)
 			(show_name no)
@@
 			(project "PS-SuppChargerPCB"
 				(path "/bb6ce8fd-e1af-464e-bfef-c3b4f18a2cee/2cf5818b-529e-491f-8ffd-d4b5d2111841"
-					(reference "R19")
+					(reference "R20")
 					(unit 1)
 				)
@@
 		(in_pos_files yes)
 		(dnp no)
-		(property "Reference" "C4"
+		(property "Reference" "C7"
 			(at 31.75 82.5499 0)
 			(show_name no)
@@
 			(project "PS-SuppChargerPCB"
 				(path "/bb6ce8fd-e1af-464e-bfef-c3b4f18a2cee/2cf5818b-529e-491f-8ffd-d4b5d2111841"
-					(reference "C4")
+					(reference "C7")
 					(unit 1)
 				)
@@
 		(in_pos_files yes)
 		(dnp no)
-		(property "Reference" "R20"
+		(property "Reference" "R19"
 			(at 137.16 77.47 90)
 			(show_name no)
@@
 			(project "PS-SuppChargerPCB"
 				(path "/bb6ce8fd-e1af-464e-bfef-c3b4f18a2cee/2cf5818b-529e-491f-8ffd-d4b5d2111841"
-					(reference "R20")
-					(unit 1)
-				)
+					(reference "R19")
+					(unit 1)
+				)
