File: Power_Mux.kicad_sch (KiCad schematic)
At the start: 8 parts, among them U6 TPS2117DRLR

Commit message: fixedsharepoint
Parts:
- removed R51: 16k, symbol Device:R
- removed R52: 4.7k, symbol Device:R
- C38: renamed from C50; value 0.1uF -> 0.1u; Mfg MLASH168SB7104KTNA01 -> (none)
- C39: renamed from C51; value 0.1uF -> 0.1u; Mfg MLASH168SB7104KTNA01 -> (none)
- C40: renamed from C52; value 0.1uF -> 0.1u; Mfg MLASH168SB7104KTNA01 -> (none)
- C41: renamed from C53; value 0.1uF -> 0.1u; Mfg MLASH168SB7104KTNA01 -> (none)
- U4: renamed from U6; MANUFACTURER Texas Instruments -> (none); MAXIMUM_PACKAGE_HEIGHT 0.6mm -> (none); PARTREV A -> (none); STANDARD IPC-7351B -> (none)
- renumbered R50 to R10

Commit message: schematic10
Changed lines of the file:
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@@
 	(generator "eeschema")
 	(generator_version "10.0")
-	(paper "A4")
+	(paper "A5")
 	(rectangle
 		(start 15.24 81.28)
@@
 	)
 	(rectangle
-		(start 15.24 102.616)
-		(end 95.25 163.576)
+		(start 110.49 31.75)
+		(end 190.5 92.71)
 		(stroke
 			(width 0)
@@
 	(text "Max and min threshold voltage calculations for 3v3 and 5v\n[delete this if you want :^)]"
 		(exclude_from_sim no)
-		(at 54.864 106.934 0)
+		(at 150.114 36.068 0)
 		(effects
 			(font
@@
 	(text "3v3\n"
 		(exclude_from_sim no)
-		(at 20.32 115.57 0)
+		(at 115.57 44.704 0)
 		(effects
 			(font
@@
 	(text "5v "
 		(exclude_from_sim no)
-		(at 58.42 115.316 0)
+		(at 153.67 44.45 0)
 		(effects
 			(font
@@
 	)
 	(image
-		(at 35.56 136.398)
+		(at 130.81 65.532)
 		(scale 0.364641)
 		(data "iVBORw0KGgoAAAANSUhEUgAAAX4AAAGJCAIAAAACL88KAAAAA3NCSVQICAjb4U/gAAAACXBIWXMA"
@@
 	)
 	(image
-		(at 73.66 136.398)
+		(at 168.91 65.532)
 		(scale 0.363383)
 		(data "iVBORw0KGgoAAAANSUhEUgAAAYAAAAGICAIAAADH9qCFAAAAA3NCSVQICAjb4U/gAAAACXBIWXMA"

Commit message: halleffectsense
Parts:
- renumbered C38 to C35, C39 to C36, C40 to C37, C41 to C38, R10 to R46, U4 to U2
Changed lines of the file:
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@@
 		(in_pos_files yes)
 		(dnp no)
-		(property "Reference" "C41"
+		(property "Reference" "C38"
 			(at 91.8972 57.2516 0)
 			(show_name no)
@@
 			(project "PS-SuppChargerPCB"
 				(path "/bb6ce8fd-e1af-464e-bfef-c3b4f18a2cee/a6d476dc-8967-4568-8283-632ab02a8186"
-					(reference "C41")
+					(reference "C38")
 					(unit 1)
 				)
@@
 		(in_pos_files yes)
 		(dnp no)
-		(property "Reference" "R10"
+		(property "Reference" "R46"
 			(at 78.994 67.564 0)
 			(show_name no)
@@
 			(project "PS-SuppChargerPCB"
 				(path "/bb6ce8fd-e1af-464e-bfef-c3b4f18a2cee/a6d476dc-8967-4568-8283-632ab02a8186"
-					(reference "R10")
+					(reference "R46")
 					(unit 1)
 				)
@@
 		(in_pos_files yes)
 		(dnp no)
-		(property "Reference" "C38"
+		(property "Reference" "C35"
 			(at 24.5872 44.5516 0)
 			(show_name no)
@@
 			(project "PS-SuppChargerPCB"
 				(path "/bb6ce8fd-e1af-464e-bfef-c3b4f18a2cee/a6d476dc-8967-4568-8283-632ab02a8186"
-					(reference "C38")
+					(reference "C35")
 					(unit 1)
 				)
@@
 		(dnp no)
 		(fields_autoplaced yes)
-		(property "Reference" "U4"
+		(property "Reference" "U2"
 			(at 60.96 44.45 0)
 			(show_name no)
@@
 			(project "PS-SuppChargerPCB"
 				(path "/bb6ce8fd-e1af-464e-bfef-c3b4f18a2cee/a6d476dc-8967-4568-8283-632ab02a8186"
-					(reference "U4")
+					(reference "U2")
 					(unit 1)
 				)
@@
 		(in_pos_files yes)
 		(dnp no)
-		(property "Reference" "C40"
+		(property "Reference" "C37"
 			(at 42.3672 67.4116 0)
 			(show_name no)
@@
 			(project "PS-SuppChargerPCB"
 				(path "/bb6ce8fd-e1af-464e-bfef-c3b4f18a2cee/a6d476dc-8967-4568-8283-632ab02a8186"
-					(reference "C40")
+					(reference "C37")
 					(unit 1)
 				)
@@
 		(in_pos_files yes)
 		(dnp no)
-		(property "Reference" "C39"
+		(property "Reference" "C36"
 			(at 38.5572 44.5516 0)
 			(show_name no)
@@
 			(project "PS-SuppChargerPCB"
 				(path "/bb6ce8fd-e1af-464e-bfef-c3b4f18a2cee/a6d476dc-8967-4568-8283-632ab02a8186"
-					(reference "C39")
-					(unit 1)
-				)
+					(reference "C36")
+					(unit 1)
+				)

Commit message: footprints1
Parts:
- renumbered C35 to C33, C36 to C34, C37 to C35, C38 to C36, R46 to R45
Changed lines of the file:
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@@
 		(in_pos_files yes)
 		(dnp no)
-		(property "Reference" "C38"
+		(property "Reference" "C36"
 			(at 91.8972 57.2516 0)
 			(show_name no)
@@
 			(project "PS-SuppChargerPCB"
 				(path "/bb6ce8fd-e1af-464e-bfef-c3b4f18a2cee/a6d476dc-8967-4568-8283-632ab02a8186"
-					(reference "C38")
+					(reference "C36")
 					(unit 1)
 				)
@@
 		(in_pos_files yes)
 		(dnp no)
-		(property "Reference" "R46"
+		(property "Reference" "R45"
 			(at 78.994 67.564 0)
 			(show_name no)
@@
 			(project "PS-SuppChargerPCB"
 				(path "/bb6ce8fd-e1af-464e-bfef-c3b4f18a2cee/a6d476dc-8967-4568-8283-632ab02a8186"
-					(reference "R46")
+					(reference "R45")
 					(unit 1)
 				)
@@
 		(in_pos_files yes)
 		(dnp no)
-		(property "Reference" "C35"
+		(property "Reference" "C33"
 			(at 24.5872 44.5516 0)
 			(show_name no)
@@
 			(project "PS-SuppChargerPCB"
 				(path "/bb6ce8fd-e1af-464e-bfef-c3b4f18a2cee/a6d476dc-8967-4568-8283-632ab02a8186"
-					(reference "C35")
+					(reference "C33")
 					(unit 1)
 				)
@@
 		(in_pos_files yes)
 		(dnp no)
-		(property "Reference" "C37"
+		(property "Reference" "C35"
 			(at 42.3672 67.4116 0)
 			(show_name no)
@@
 			(project "PS-SuppChargerPCB"
 				(path "/bb6ce8fd-e1af-464e-bfef-c3b4f18a2cee/a6d476dc-8967-4568-8283-632ab02a8186"
-					(reference "C37")
+					(reference "C35")
 					(unit 1)
 				)
@@
 		(in_pos_files yes)
 		(dnp no)
-		(property "Reference" "C36"
+		(property "Reference" "C34"
 			(at 38.5572 44.5516 0)
 			(show_name no)
@@
 			(project "PS-SuppChargerPCB"
 				(path "/bb6ce8fd-e1af-464e-bfef-c3b4f18a2cee/a6d476dc-8967-4568-8283-632ab02a8186"
-					(reference "C36")
-					(unit 1)
-				)
+					(reference "C34")
+					(unit 1)
+				)

Commit message: layout1
Parts:
- C33, C34, C35, C36, R45: KiLib_Generator (none) -> SMD_2terminal_chip_molded
Changed lines of the file:
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@@
+			)
+		)
+		(property "KiLib_Generator" "SMD_2terminal_chip_molded"
+			(at 88.9 58.42 0)
+			(hide yes)
+			(show_name no)
+			(do_not_autoplace no)
+			(effects
+				(font
+					(size 1.27 1.27)
+				)
 			)
 		)
@@
 			)
 		)
+		(property "KiLib_Generator" "SMD_2terminal_chip_molded"
+			(at 76.2 68.58 0)
+			(hide yes)
+			(show_name no)
+			(do_not_autoplace no)
+			(effects
+				(font
+					(size 1.27 1.27)
+				)
+			)
+		)
 		(pin "1"
 		)
@@
 		)
 		(property "P/N" "MLASH168SB7104KTNA01"
+			(at 21.59 45.72 0)
+			(hide yes)
+			(show_name no)
+			(do_not_autoplace no)
+			(effects
+				(font
+					(size 1.27 1.27)
+				)
+			)
+		)
+		(property "KiLib_Generator" "SMD_2terminal_chip_molded"
 			(at 21.59 45.72 0)
 			(hide yes)
@@
 			)
 		)
+		(property "KiLib_Generator" "SMD_2terminal_chip_molded"
+			(at 39.37 68.58 0)
+			(hide yes)
+			(show_name no)
+			(do_not_autoplace no)
+			(effects
+				(font
+					(size 1.27 1.27)
+				)
+			)
+		)
 		(pin "1"
 		)
@@
 			(at 35.56 45.72 0)
 			(hide yes)
+			(show_name no)
+			(do_not_autoplace no)
+			(effects
+				(font
+					(size 1.27 1.27)
+				)
+			)
+		)
+		(property "KiLib_Generator" "SMD_2terminal_chip_molded"
+			(at 35.56 45.72 0)
+			(hide yes)

Commit message: layout5
Parts:
- renumbered C36 to C35, C35 to C36
Changed lines of the file:
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@@
 		(in_pos_files yes)
 		(dnp no)
-		(property "Reference" "C36"
+		(property "Reference" "C35"
 			(at 91.8972 57.2516 0)
 			(show_name no)
@@
 			(project "PS-SuppChargerPCB"
 				(path "/bb6ce8fd-e1af-464e-bfef-c3b4f18a2cee/a6d476dc-8967-4568-8283-632ab02a8186"
-					(reference "C36")
+					(reference "C35")
 					(unit 1)
 				)
@@
 		(in_pos_files yes)
 		(dnp no)
-		(property "Reference" "C35"
+		(property "Reference" "C36"
 			(at 42.3672 67.4116 0)
 			(show_name no)
@@
 			(project "PS-SuppChargerPCB"
 				(path "/bb6ce8fd-e1af-464e-bfef-c3b4f18a2cee/a6d476dc-8967-4568-8283-632ab02a8186"
-					(reference "C35")
-					(unit 1)
-				)
+					(reference "C36")
+					(unit 1)
+				)
