File: PS-SuppChargerPCB.kicad_pcb (KiCad board)
At the start: 2 copper layers, 199 parts, among them IC1 LM74502DDFR, IC2 CYPD3177-24LQXQ, IC3 TPS552872RYQR, J1 PS_Banana_+, J10 SWD, J2 PS_Banana_-, J3 CarLVPowerConnector, J4 Supp_Conn_xT30, J5 TP_I2C, J6 TP_USB_CC, J7 TP_DS SPI, J8 USB_C_Receptacle_USB2.0_16P, J9 SWD_Header, Q1 PSMN012-100YS, Q2 PSMN012-100YS, Q3 SI7997DP-T1-GE3, Q4 SI7997DP-T1-GE3, Q5 IRLML0030, SW1 Reset, SW2 SW_SPDT, U1 INA226AIDGST, U2 TPS2117DRLR, U3 LMR51635XDDCR, U4 MCP1826S, U5 STM32G473CETx, Y1 Crystal

Commit message: layout1
Parts:
- moved DS1 262.0 mm to (292.1, 192.6)
- moved R44 246.6 mm to (314.1, 70.0)
- moved C32 240.0 mm to (309.1, 70.0)
- moved U1 237.6 mm to (309.9, 63.0)
- moved C45 235.8 mm to (266.1, 185.1)
- moved R48 235.8 mm to (266.1, 187.6)
- moved C31 234.0 mm to (302.1, 64.0)
- moved R42 231.9 mm to (298.1, 62.0)
- moved R43 231.7 mm to (298.1, 65.4)
- moved C44 224.5 mm to (333.0, 117.9)
- moved R41 217.2 mm to (291.0, 64.0)
- moved TP9 213.7 mm to (324.0, 109.9)
- moved U4 213.1 mm to (324.1, 119.0)
- moved J4 210.7 mm to (335.7, 62.0)
- moved D10 206.5 mm to (62.6, 263.2)
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Connections:
- H2 pad 1: unconnected-(H2-Pad1)_2 -> /unconnected-(H2-Pad1)_2_2
- H3 pad 1: unconnected-(H3-Pad1)_1 -> /unconnected-(H3-Pad1)_1_1
- H4 pad 1: unconnected-(H4-Pad1)_2 -> /unconnected-(H4-Pad1)_2_2
- R41 pad 2: Net-(R41-Pad2) -> +14.7V
- R42 pad 2: Net-(R41-Pad2) -> /12VBB_VOUT
- R43 pad 2: Net-(R41-Pad3) -> +14.7V

Commit message: alayout2
Parts:
- JP1: value SolderJumper_2_Open -> PP_SolderJumper_2_Open
- R11, R12, R13, R14, R5, R6, R7, R8, R9: value 1k -> 4.7k
- R41: value 2m -> 10m; footprint PS-Supp-Footprints:PSR100KTQFJ2L00_ROM -> PS-Supp-Footprints:PMR100HZPFU10L0
- moved TP13 91.9 mm to (5.00, 66.5)
- moved TP12 86.6 mm to (10.0, 66.2)
- moved TP14 77.2 mm to (15.2, 66.5)
- moved D21 65.6 mm to (59.5, 73.6), turned to 180 degrees
- moved R34 62.9 mm to (59.5, 70.6), turned to 180 degrees
- moved C18 58.6 mm to (69.8, 74.0), turned to -90 degrees
- moved Q5 57.0 mm to (63.1, 72.0), turned to 180 degrees
- moved C17 56.9 mm to (72.8, 74.0), turned to -90 degrees
- moved C16 53.9 mm to (75.8, 71.0)
- moved C15 53.6 mm to (75.9, 68.0), turned to 180 degrees
- moved R33 42.6 mm to (66.8, 74.1), turned to 90 degrees
- moved C14 40.6 mm to (60.8, 92.8), turned to -90 degrees
- moved TP2 40.1 mm to (20.5, 65.8)
- moved R28 38.4 mm to (78.0, 64.0), turned to 90 degrees
- moved R30 37.7 mm to (75.0, 63.9), turned to 90 degrees
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Connections:
- net /DS_SCL renamed /DS_CLK
- net /DS_SDA renamed /DS_MOSI
- C14 pad 1: +5V -> /PD_5V_OUT
- C34 pad 1: +5V -> /PD_5V_OUT
- C45 pad 1: +3V3A -> +3V3
- C48 pad 1: +3V3A -> /Peripherals/48PinMCU/VDDA
- C52 pad 1: +3V3A -> /Peripherals/48PinMCU/VDDA
- C54 pad 1: +3V3A -> /Peripherals/48PinMCU/VDDA
- C56 pad 1: +3V3A -> /Peripherals/48PinMCU/VDDA
- C60 pad 1: +3V3A -> /Peripherals/48PinMCU/VDDA
- D6 pad 2: +5V -> /PD_5V_OUT
- DS1 pad 2: +3V3A -> +3V3
- FB2 pad 2: +3V3A -> /Peripherals/48PinMCU/VDDA
- H2 pad 1: /unconnected-(H2-Pad1)_2_2 -> unconnected-(H2-Pad1)_2
- H3 pad 1: /unconnected-(H3-Pad1)_1_1 -> unconnected-(H3-Pad1)_1
- H4 pad 1: /unconnected-(H4-Pad1)_2_2 -> unconnected-(H4-Pad1)_2
- Q4 pad 10: +5V -> /PD_5V_OUT
- Q4 pad 12: +5V -> /PD_5V_OUT
- Q4 pad 5: +5V -> /PD_5V_OUT
- Q4 pad 6: +5V -> /PD_5V_OUT
- TP13 pad 1: +5V -> /PD_5V_OUT
- TP7 pad 1: +5V -> /PD_5V_OUT
- U2 pad 6: +5V -> /PD_5V_OUT
- U5 pad 20: +3V3A -> /Peripherals/48PinMCU/VDDA
- U5 pad 21: +3V3A -> /Peripherals/48PinMCU/VDDA
Routing:
- net /USB_PD/VBUS_MIN: track 0.00 -> 7.47 mm
- net /USB_VBUS: track 0.00 -> 6.75 mm
- net /USB_PD/ISINK_COARSE: track 0.00 -> 6.56 mm
- net /USB-C_Connector/VBUS_IN: track 0.00 -> 6.25 mm
- net /USB_DP: track 0.00 -> 2.82 mm
- net /USB_PD/PD_3V3: track 0.00 -> 2.44 mm
- net /USB_DM: track 0.00 -> 2.32 mm

Commit message: layout4
Parts:
- J3: footprint LHRS_Connectors:Molex_Nano-Fit_105309-xx02_1x02_P2.50mm_Vertical -> LHRS_Connectors:Molex_Nano-Fit_105313-xx02_1x02_P2.50mm_Horizontal
- moved TP12 86.8 mm to (89.5, 31.5)
- moved TP13 86.8 mm to (84.5, 31.8)
- moved TP14 86.8 mm to (94.8, 31.8)
- moved TP2 86.8 mm to (100.0, 31.0)
- moved U5 69.9 mm to (232.3, 141.5)
- moved TP7 61.3 mm to (78.8, 39.2)
- moved TP10 57.6 mm to (83.8, 39.8)
- moved TP16 46.2 mm to (96.0, 40.5)
- moved J4 44.6 mm to (291.5, 68.0), turned to -90 degrees
- moved TP6 43.8 mm to (279.2, 49.8)
- moved F1 38.6 mm to (85.3, 153.7), turned to 90 degrees
- moved NT1 36.6 mm to (256.0, 74.5)
- moved C43 36.5 mm to (350.5, 122.0)
- moved C44 36.5 mm to (369.5, 117.0)
- moved D22 36.5 mm to (350.5, 117.0)
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Connections:
- net /PS_JUMPER renamed /PP_VIN
Routing:
- net /12VBB_PG: track 0.00 -> 20.4 mm
- net /I2C_SCL: track 0.00 -> 16.3 mm
- net /12VBB_CC: track 0.00 -> 14.9 mm
- net /I2C_SDA: track 0.00 -> 12.9 mm
- net +3V3: track 0.00 -> 10.0 mm
- net /USB_PD/VBUS_MIN: track 7.47 -> 0.00 mm
- net /USB_VBUS: track 6.75 -> 0.00 mm
- net /USB_PD/ISINK_COARSE: track 6.56 -> 0.00 mm
- net /USB-C_Connector/VBUS_IN: track 6.25 -> 0.00 mm
- net /USB_DP: track 2.82 -> 0.00 mm
- net /USB_PD/PD_3V3: track 2.44 -> 0.00 mm
- net /USB_DM: track 2.32 -> 0.00 mm

Commit message: layout5
Parts:
- moved D13 294.7 mm to (341.4, 114.6), turned to 180 degrees
- moved R15 277.0 mm to (341.5, 117.5), turned to 180 degrees
- moved D11 261.3 mm to (273.1, 68.8), turned to 180 degrees
- moved D8 261.1 mm to (295.2, 111.8), turned to 180 degrees
- moved R13 240.7 mm to (277.3, 68.8)
- moved R10 240.4 mm to (295.2, 114.8), turned to 180 degrees
- moved D10 228.9 mm to (251.1, 90.2), turned to 180 degrees
- moved D12 225.7 mm to (262.2, 114.5), turned to 180 degrees
- moved R12 209.6 mm to (256.1, 90.2)
- moved R14 203.5 mm to (262.2, 117.5), turned to 180 degrees
- moved D4 185.6 mm to (109.9, 59.0)
- moved D5 166.8 mm to (50.6, 78.8)
- moved D9 164.6 mm to (183.9, 111.7)
- moved D6 155.2 mm to (69.8, 91.2), turned to 180 degrees
- moved R11 153.2 mm to (183.8, 109.0)
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Connections:
- net /USB_DM renamed /USB_D-
- net /USB_DP renamed /USB_D+
- U5 pad 11: /PD_GPIO_1 -> /Peripherals/48PinMCU/PA3
- U5 pad 12: /PD_FAULT -> /Peripherals/48PinMCU/PA4
- U5 pad 14: /Peripherals/48PinMCU/PA6 -> /DS_RES
- U5 pad 16: /12VBB_CC -> /DS_DC
- U5 pad 17: /12VBB_PG -> /DS_CS
- U5 pad 18: /EN -> /DS_BLK
- U5 pad 29: /Peripherals/48PinMCU/PB15 -> /INA_ALERT
- U5 pad 32: /INA_ALERT -> /Peripherals/48PinMCU/PA10
- U5 pad 40: /DS_BLK -> /EN
- U5 pad 41: /DS_CS -> /12VBB_PG
- U5 pad 42: /Peripherals/48PinMCU/PB5 -> /12VBB_CC
- U5 pad 43: /DS_DC -> /PD_FAULT
- U5 pad 44: /DS_RES -> /PD_GPIO_1
Routing:
- net /PD_GPIO_1: track 0.00 -> 38.2 mm
- net /PD_FAULT: track 0.00 -> 18.2 mm
- net /I2C_SDA: track 12.9 -> 29.9 mm
- net /I2C_SCL: track 16.3 -> 32.2 mm
- net /USB_D-: track 0.00 -> 2.36 mm
- net /USB_D+: track 0.00 -> 2.33 mm

Commit message: layout6
Parts:
- removed TP11: VBUS_IN, TestPoint:TestPoint_Loop_D1.80mm_Drill1.0mm_Beaded
- removed the TP12 at (89.5, 31.5)
- removed the TP13 at (84.5, 31.8)
- moved TP2 67.9 mm to (70.0, 87.0)
- moved TP14 52.7 mm to (59.0, 78.0)
- moved TP12 49.0 mm to (58.8, 65.0)
- moved TP3 48.2 mm to (54.5, 78.0)
- moved TP13 46.1 mm to (70.0, 82.0)
- moved TP1 37.4 mm to (75.2, 59.0)
- moved R1 34.3 mm to (80.1, 62.8), turned to 180 degrees
- moved J3 32.2 mm to (167.7, 225.0)
- moved J4 32.2 mm to (176.8, 225.0)
- moved J6 32.2 mm to (172.2, 225.0)
- moved C46 31.8 mm to (197.2, 218.3)
- moved C47 31.8 mm to (200.8, 216.6)
- moved C48 31.8 mm to (191.2, 214.1)
- moved C49 31.8 mm to (194.2, 214.2)
- moved C50 31.8 mm to (197.2, 214.2)
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- renumbered C15 to C10, C16 to C11, C17 to C12, C18 to C13, C10 to C14, C11 to C15, C13 to C16, C12 to C17, C14 to C18, C22 to C19, C23 to C20, C19 to C21, C20 to C22, C24 to C23, C25 to C24, C26 to C25, C28 to C26, C30 to C27, C21 to C28, C27 to C29, C29 to C30, C36 to C35, C35 to C36, C39 to C37, C37 to C38, C38 to C39, C7 to C4, C59 to C46, C49 to C47, C51 to C48, C53 to C49, C6 to C5, C55 to C50, C57 to C51, C58 to C52, C46 to C53, C47 to C54, C60 to C55, C48 to C56, C52 to C57, C54 to C58, C56 to C59, C5 to C6, C50 to C60, C4 to C7, D4 to D1, D8 to D10, D13 to D11, D1 to D12, D2 to D13, D21 to D19, D9 to D2, D19 to D20, D20 to D21, D24 to D23, D25 to D24, D23 to D25, D5 to D3, D10 to D4, D6 to D5, D11 to D6, D12 to D8, D3 to D9, FB2 to FB1, FB1 to FB2, H3 to H2, H2 to H3, J5 to J3, J7 to J4, J3 to J5, J4 to J7, Q5 to Q3, Q3 to Q4, Q4 to Q5, R6 to R1, R15 to R11, R1 to R12, R2 to R13, R3 to R14, R4 to R15, R17 to R16, R16 to R17, R20 to R19, R11 to R2, R19 to R20, R28 to R22, R33 to R23, R30 to R24, R34 to R25, R29 to R26, R31 to R27, R22 to R28, R23 to R29, R7 to R3, R26 to R30, R32 to R31, R24 to R32, R27 to R33, R25 to R34, R38 to R35, R39 to R36, R40 to R37, R37 to R38, R36 to R39, R12 to R4, R35 to R40, R44 to R41, R41 to R43, R43 to R44, R50 to R49, R8 to R5, R55 to R50, R56 to R51, R53 to R52, R54 to R53, R49 to R54, R51 to R55, R52 to R56, R59 to R58, R60 to R59, R13 to R6, R58 to R60, R9 to R7, R14 to R8, R5 to R9, SW2 to SW1, SW1 to SW2, TP2 to TP1, TP9 to TP10, TP14 to TP12, TP15 to TP13, TP16 to TP14, TP7 to TP2, TP10 to TP3, TP8 to TP5, TP3 to TP6, TP6 to TP7, TP1 to TP8, TP5 to TP9
Routing:
- net /USB_VBUS: track 0.00 -> 50.7 mm
- net +15V: track 0.00 -> 20.4 mm
- net /USB_PD/PD_3V3: track 0.00 -> 20.1 mm
- net /USB_PD/PD_1V8: track 0.00 -> 13.7 mm
- net /USB_D+: track 2.33 -> 12.7 mm
- net /USB_D-: track 2.36 -> 9.78 mm
- net /USB_PD/VBUS_MIN: track 0.00 -> 6.66 mm
- net /USB_PD/ISINK_COARSE: track 0.00 -> 6.54 mm
- net Net-(D19-K): track 0.00 -> 3.29 mm
- net Net-(D19-A): track 0.00 -> 3.03 mm
- net Net-(D3-K): track 0.00 -> 2.38 mm
- net /PD_FAULT: track 18.2 -> 19.2 mm
- net /USB-C_Connector/VBUS_IN: track 0.00 -> 0.53 mm
