File: PS-SuppChargerPCB.kicad_pcb (KiCad board)
At the start: 2 copper layers, 196 parts, among them IC1 LM74502DDFR, IC2 CYPD3177-24LQXQ, IC3 TPS552872RYQR, J1 PS_Banana_+, J10 SWD, J2 PS_Banana_-, J3 TP_I2C, J4 TP_DS SPI, J5 CarLVPowerConnector, J6 TP_USB_CC, J7 Supp_Conn_xT30, J8 USB_C_Receptacle_USB2.0_16P, J9 SWD_Header, Q1 PSMN012-100YS, Q2 PSMN012-100YS, Q3 IRLML0030, Q4 SI7997DP-T1-GE3, Q5 SI7997DP-T1-GE3, SW1 SW_SPDT, SW2 Reset, U1 INA226AIDGST, U2 TPS2117DRLR, U3 LMR51635XDDCR, U4 MCP1826S, U5 STM32G473CETx, Y1 Crystal

Commit message: layout7
Parts:
- moved U5 149.1 mm to (101.0, 63.5)
- moved C31 109.3 mm to (170.6, 48.2)
- moved C32 109.3 mm to (174.8, 44.0)
- moved D6 109.3 mm to (166.7, 44.0)
- moved J7 109.3 mm to (185.1, 43.2)
- moved R42 109.3 mm to (166.8, 50.2)
- moved R43 109.3 mm to (161.1, 47.6)
- moved R44 109.3 mm to (166.8, 47.2)
- moved TP6 109.3 mm to (166.8, 55.2)
- moved TP7 109.3 mm to (166.8, 39.0)
- moved U1 109.3 mm to (176.6, 47.5)
- moved R41 109.3 mm to (178.7, 44.0)
- moved R6 109.3 mm to (170.9, 44.0)
- moved C1 107.3 mm to (130.6, 83.1)
- moved C19 107.3 mm to (134.8, 76.4)
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Routing:
- net /USB_VBUS: track 50.7 -> 0.00 mm
- net Net-(D20-A): track 0.00 -> 32.4 mm
- net Net-(D21-A): track 0.00 -> 30.5 mm
- net /CC1: track 0.00 -> 24.2 mm
- net +15V: track 20.4 -> 0.00 mm
- net /CC2: track 0.00 -> 18.3 mm, vias 0 -> 2
- net /USB_PD/SAFE_PWR_EN: track 0.00 -> 17.9 mm, vias 0 -> 2
- net /I2C_SDA: track 29.7 -> 12.9 mm
- net /I2C_SCL: track 32.2 -> 16.3 mm
- net Net-(D20-K): track 0.00 -> 15.1 mm
- net /USB_PD/VBUS_FET_EN: track 0.00 -> 13.5 mm, vias 0 -> 2
- net /PD_GPIO_1: track 38.2 -> 24.8 mm
- net /USB_PD/PD_3V3: track 20.1 -> 32.7 mm, vias 0 -> 2
- net /PD_FAULT: track 19.2 -> 30.9 mm
- net Net-(D21-K): track 0.00 -> 9.32 mm
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- added copper zone on F.Cu, net +15V
- added copper zone on F.Cu, net /PD_5V_OUT
- added copper zone on F.Cu, net /USB-C_Connector/VBUS_IN
- added copper zone on F.Cu, net /USB_VBUS
- added copper zone on B.Cu, net GND

Commit message: layout9
Parts:
- moved R30 203.4 mm to (215.0, 179.0), turned to -90 degrees
- moved C14 200.8 mm to (206.2, 179.5), turned to 90 degrees
- moved R31 199.4 mm to (209.2, 178.9), turned to 90 degrees
- moved C15 198.6 mm to (212.2, 179.0), turned to 90 degrees
- moved TP1 198.6 mm to (193.0, 182.0)
- moved D20 194.0 mm to (212.8, 174.3)
- moved D18 193.0 mm to (200.2, 179.3), turned to 0 degrees
- moved R33 191.0 mm to (224.8, 159.6), turned to -90 degrees
- moved R1 190.8 mm to (187.8, 180.3)
- moved Q4 188.5 mm to (212.6, 170.2), turned to 90 degrees
- moved D1 186.5 mm to (187.8, 177.3), turned to 0 degrees
- moved C17 185.6 mm to (224.8, 155.8), turned to -90 degrees
- moved TP12 184.9 mm to (210.0, 183.3)
- moved C2 182.2 mm to (187.8, 174.0)
- moved D21 182.0 mm to (221.0, 157.6), turned to -90 degrees
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Routing:
- net /PD_GPIO_1: track 24.8 -> 1.45 mm, vias 0 -> 1
- net Net-(D20-A): track 32.4 -> 14.7 mm
- net /PD_FAULT: track 30.9 -> 14.9 mm, vias 0 -> 3
- net /USB_PD/SAFE_PWR_EN: track 17.9 -> 2.79 mm, vias 2 -> 0
- net /CC2: track 18.3 -> 29.8 mm, vias 2 -> 0
- net /USB_PD/VBUS_FET_EN: track 13.5 -> 3.00 mm, vias 2 -> 0
- net /USB_PD/PD_1V8: track 14.1 -> 6.24 mm, vias 0 -> 1
- net Net-(D20-K): track 15.1 -> 7.47 mm
- net Net-(D21-A): track 30.5 -> 23.1 mm
- net /USB_D+: track 14.6 -> 9.41 mm, vias 2 -> 0
- net /CC1: track 24.2 -> 19.5 mm
- net Net-(IC2-FLIP): track 7.54 -> 11.6 mm
- net /USB_PD/PD_3V3: track 32.7 -> 28.8 mm
- net /USB_PD/VBUS_MIN: track 7.62 -> 11.2 mm
- net Net-(D3-K): track 3.03 -> 0.00 mm
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- removed copper zone on F.Cu, net +15V
- removed copper zone on F.Cu, net /PD_5V_OUT
- removed copper zone on F.Cu, net /USB-C_Connector/VBUS_IN
- removed copper zone on B.Cu, net GND

Commit message: layout10
Parts:
- moved C60 160.0 mm to (160.6, -50.3)
- moved D25 160.0 mm to (164.4, -24.5)
- moved J3 160.0 mm to (135.4, -58.3)
- moved J4 160.0 mm to (144.6, -58.3)
- moved J9 160.0 mm to (183.1, -25.3)
- moved R49 160.0 mm to (160.6, -46.8)
- moved R52 160.0 mm to (180.1, -18.1)
- moved R53 160.0 mm to (180.1, -14.9)
- moved R54 160.0 mm to (167.2, -20.7)
- moved R55 160.0 mm to (164.2, -20.7)
- moved R56 160.0 mm to (161.2, -20.7)
- moved SW1 160.0 mm to (181.7, -47.5)
- moved SW2 160.0 mm to (165.4, -47.8)
- moved C46 160.0 mm to (165.0, -65.0)
- moved C47 160.0 mm to (168.5, -66.7)
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Routing:
- net Net-(D20-A): track 14.7 -> 45.8 mm, vias 0 -> 2
- net /PD_5V_OUT: track 0.00 -> 24.2 mm, vias 0 -> 2
- net /USB_PD/PD_1V8: track 6.24 -> 20.4 mm
- net /USB_PD/PD_3V3: track 28.8 -> 41.6 mm, vias 2 -> 3
- net /USB_D+: track 9.41 -> 19.5 mm
- net Net-(D21-A): track 23.1 -> 33.2 mm, vias 0 -> 2
- net Net-(D21-K): track 10.4 -> 19.3 mm
- net /CC2: track 29.8 -> 21.6 mm, vias 0 -> 1
- net /USB_D-: track 10.1 -> 17.8 mm
- net +15V: track 0.00 -> 6.68 mm
- net Net-(D20-K): track 7.47 -> 13.6 mm
- net /USB_PD/ISINK_COARSE: track 9.73 -> 14.1 mm, vias 0 -> 2
- net Net-(D5-K): track 3.59 -> 1.84 mm
- net /CC1: track 19.5 -> 19.9 mm, vias 0 -> 2
- net /USB-C_Connector/VBUS_IN: vias 0 -> 6
- added copper zone on F.Cu, net +15V
- added copper zone on F.Cu, net /USB-C_Connector/VBUS_IN

Commit message: layoutpsdone
Parts:
- moved J3 241.7 mm to (335.2, 77.8)
- moved R60 241.7 mm to (383.9, 47.2)
- moved C46 241.7 mm to (364.8, 71.0)
- moved C47 241.7 mm to (368.2, 69.3)
- moved C48 241.7 mm to (358.8, 66.8)
- moved C49 241.7 mm to (361.8, 66.9)
- moved C50 241.7 mm to (364.8, 66.9)
- moved C51 241.7 mm to (358.8, 71.1)
- moved C52 241.7 mm to (361.8, 71.2)
- moved C55 241.7 mm to (384.0, 70.1)
- moved D23 241.7 mm to (380.2, 81.2)
- moved D24 241.7 mm to (383.5, 81.1)
- moved D25 241.7 mm to (364.2, 111.6)
- moved FB1 241.7 mm to (381.0, 70.1)
- moved J10 241.7 mm to (384.7, 119.1)
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Routing:
- net /PowerProtection/gate: track 0.00 -> 28.2 mm
- net /PowerProtection/source: track 0.00 -> 20.1 mm
- net Net-(D17-K): track 0.00 -> 16.6 mm
- net /PowerProtection/EN/UVLO: track 0.00 -> 13.3 mm
- net /PowerProtection/OV: track 0.00 -> 9.02 mm
- net Net-(D7-K): track 0.00 -> 3.32 mm
- net Net-(C5-Pad1): track 0.00 -> 3.03 mm
- net Net-(D9-K): track 0.00 -> 2.52 mm
- net Net-(IC1-VCAP): track 0.00 -> 2.13 mm
- added copper zone on F.Cu, net /PP_VIN
- added copper zone on F.Cu, net /PP_VOUT
- added copper zone on F.Cu, net /PS_VOUT

Commit message: layoutbbdone
Parts:
- moved L1 127.6 mm to (165.2, 216.8)
- moved C27 116.3 mm to (184.3, 219.8)
- moved R37 113.9 mm to (188.8, 218.7)
- moved R39 112.4 mm to (186.1, 204.8)
- moved C28 112.3 mm to (186.3, 202.6)
- moved NT1 112.3 mm to (189.7, 202.6)
- moved C29 112.3 mm to (186.0, 206.6)
- moved C30 112.3 mm to (186.0, 210.6)
- moved R38 112.3 mm to (186.0, 208.6)
- moved C19 112.3 mm to (175.8, 200.8)
- moved R40 111.8 mm to (168.2, 207.6), turned to 0 degrees
- moved IC3 111.8 mm to (178.8, 205.9)
- moved R12 111.8 mm to (172.1, 204.3)
- moved R13 111.8 mm to (168.3, 204.3)
- moved C1 111.8 mm to (172.1, 207.6)
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Routing:
- net Net-(IC3-SW1): track 0.00 -> 31.3 mm, vias 0 -> 2
- net Net-(IC3-ISP): track 0.00 -> 27.9 mm
- net Net-(IC3-SW2): track 0.00 -> 23.9 mm
- net Net-(IC3-FB): track 0.00 -> 15.7 mm
- net /12VBB_PG: track 20.4 -> 10.2 mm
- net Net-(IC3-FSW): track 0.00 -> 9.18 mm
- net /EN: track 0.00 -> 7.48 mm
- net Net-(IC3-COMP): track 0.00 -> 6.18 mm
- net Net-(IC3-CDC): track 0.00 -> 6.18 mm
- net /DIODE_OR_OUT: track 0.00 -> 5.36 mm
- net Net-(IC3-BOOT1): track 0.00 -> 5.36 mm, vias 0 -> 2
- net Net-(IC3-VCC): track 0.00 -> 5.23 mm
- net Net-(IC3-BOOT2): track 0.00 -> 4.86 mm
- net /12VBB_CC: track 14.9 -> 10.1 mm
- net /12VBuckBoost/DITH/SYNC: track 0.00 -> 3.92 mm
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- added copper zone on F.Cu, net /12VBB_VOUT
- added copper zone on F.Cu, net /DIODE_OR_OUT
