File: PS-SuppChargerPCB.kicad_pcb (KiCad board)
At the start: 2 copper layers, 196 parts, among them IC1 LM74502DDFR, IC2 CYPD3177-24LQXQ, IC3 TPS552872RYQR, J1 PS_Banana_+, J10 SWD, J2 PS_Banana_-, J3 TP_I2C, J4 TP_DS SPI, J5 CarLVPowerConnector, J6 TP_USB_CC, J7 Supp_Conn_xT30, J8 USB_C_Receptacle_USB2.0_16P, J9 SWD_Header, Q1 PSMN012-100YS, Q2 PSMN012-100YS, Q3 IRLML0030, Q4 SI7997DP-T1-GE3, Q5 SI7997DP-T1-GE3, SW1 SW_SPDT, SW2 Reset, U1 INA226AIDGST, U2 TPS2117DRLR, U3 LMR51635XDDCR, U4 MCP1826S, U5 STM32G473CETx, Y1 Crystal

Commit message: premosfetflip
Parts:
- removed J6: TP_USB_CC, Connector_PinSocket_2.54mm:PinSocket_1x02_P2.54mm_Vertical
- moved NT1 23.4 mm to (148.6, 153.1)
- moved C26 6.17 mm to (160.8, 209.8), turned to 90 degrees
- moved C14 5.94 mm to (140.4, 188.8), turned to -90 degrees
- moved C18 4.44 mm to (159.3, 163.8), turned to 90 degrees
- moved R5 3.86 mm to (162.4, 162.9)
- moved C24 3.32 mm to (164.4, 209.7)
- moved C23 3.32 mm to (168.2, 209.7)
- moved C25 3.32 mm to (171.9, 209.7)
- moved C27 3.32 mm to (175.2, 209.9)
- moved C22 2.93 mm to (171.7, 204.1)
- moved D18 2.20 mm to (136.5, 188.9)
- moved C21 2.07 mm to (174.8, 204.0)
- moved R40 1.35 mm to (174.2, 199.2)
- moved D5 0.44 mm to (162.4, 164.7), turned to 180 degrees
- moved D15 0.14 mm to (134.8, 173.2)
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Connections:
- C28 pad 2: GND -> GNDA
- C29 pad 2: GND -> GNDA
- C30 pad 2: GND -> GNDA
- H2 pad 1: unconnected-(H2-Pad1)_1 -> /unconnected-(H2-Pad1)_1_1
- H3 pad 1: unconnected-(H3-Pad1)_2 -> /unconnected-(H3-Pad1)_2_2
- H4 pad 1: unconnected-(H4-Pad1)_2 -> /unconnected-(H4-Pad1)_2_2
- IC3 pad 17: GND -> GNDA
- J5 pad 1: /PS_VOUT -> GND
- NT1 pad 2: GND -> GNDA
- R37 pad 2: GND -> GNDA
- R39 pad 1: GND -> GNDA
- R40 pad 1: GND -> GNDA
Routing:
- net /12VBB_VOUT: track 23.3 -> 14.8 mm
- net /PD_5V_OUT: track 72.8 -> 64.6 mm
- net /PowerProtection/source: track 14.7 -> 7.93 mm
- net Net-(IC3-FSW): track 6.58 -> 0.00 mm
- net /USB-C_Connector/VBUS_IN: track 0.00 -> 5.48 mm
- net +14.7V: track 20.7 -> 24.2 mm
- net GND: track 0.00 -> 2.27 mm, vias 0 -> 1
- net Net-(D5-K): track 1.84 -> 0.00 mm
- net Net-(D21-A): track 27.0 -> 25.4 mm, vias 2 -> 1
- net /USB_PD/PD_3V3: track 45.8 -> 44.4 mm
- removed copper zone on F.Cu, net (none)

Commit message: usbpdflipped
Parts:
- moved TP1 154.0 mm to (0.30, 189.0)
- moved TP13 75.7 mm to (87.5, 189.9)
- moved TP12 75.7 mm to (83.2, 189.9)
- moved H1 72.3 mm to (50.0, 102.7)
- moved TP14 68.2 mm to (75.0, 189.6)
- moved R50 26.4 mm to (150.4, 159.5)
- moved R58 26.2 mm to (147.8, 159.5)
- moved C48 26.1 mm to (140.7, 155.8), turned to 180 degrees
- moved R59 26.1 mm to (145.0, 159.5)
- moved R52 26.0 mm to (142.2, 159.5)
- moved C47 25.9 mm to (156.8, 157.0)
- moved R53 25.8 mm to (139.5, 159.5)
- moved C46 25.7 mm to (153.7, 157.7), turned to 0 degrees
- moved C53 25.2 mm to (157.8, 152.8)
- moved C54 25.2 mm to (157.8, 149.3)
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Routing:
- net /12VBB_CC: track 73.8 -> 17.5 mm
- net /12VBB_PG: track 73.7 -> 18.9 mm
- net /EN: track 77.7 -> 23.9 mm
- net /USB_PD/PD_3V3: track 44.4 -> 0.00 mm, vias 3 -> 0
- net Net-(D20-A): track 43.6 -> 0.00 mm, vias 2 -> 0
- net /USB_D+: track 6.71 -> 41.7 mm
- net /USB_D-: track 6.71 -> 41.0 mm
- net /PD_5V_OUT: track 64.6 -> 87.3 mm, vias 4 -> 2
- net Net-(D21-A): track 25.4 -> 3.67 mm, vias 1 -> 0
- net /USB_PD/PD_1V8: track 21.2 -> 0.00 mm, vias 1 -> 0
- net /I2C_SCL: track 105.2 -> 84.2 mm
- net /I2C_SDA: track 93.3 -> 72.5 mm
- net /CC2: track 20.4 -> 0.00 mm, vias 1 -> 0
- net /CC1: track 19.2 -> 0.00 mm, vias 1 -> 0
- net /PD_FAULT: track 15.9 -> 0.00 mm, vias 3 -> 0
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- added copper zone on F.Cu, net /PD_5V_OUT

Commit message: usbpdflipped2
Parts:
- moved TP1 155.0 mm to (155.3, 190.4)
- moved TP14 92.6 mm to (164.9, 167.2)
- moved TP13 86.3 mm to (172.8, 177.0)
- moved TP12 80.8 mm to (164.0, 191.8)
- moved H1 78.8 mm to (120.2, 138.3)
- moved H4 6.11 mm to (258.2, 228.2)
- moved C5 5.10 mm to (156.8, 212.1), turned to -90 degrees
- moved TP2 4.36 mm to (173.2, 167.4)
- moved C22 3.80 mm to (167.8, 204.2)
- moved D2 3.25 mm to (187.4, 173.2)
- moved R2 3.25 mm to (187.4, 170.2)
- moved C21 2.86 mm to (171.9, 204.2)
- moved R40 2.70 mm to (171.6, 199.2)
- moved D12 2.50 mm to (185.1, 178.5)
- moved C43 2.39 mm to (186.1, 154.7)
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Routing:
- net Net-(IC3-ISP): track 38.0 -> 0.00 mm
- net Net-(D22-K): track 15.8 -> 5.28 mm
- net +3V3: track 102.0 -> 91.7 mm
- net +5V: track 23.4 -> 15.7 mm
- net Net-(IC3-FB): track 6.52 -> 0.00 mm
- net /PD_5V_OUT: track 87.3 -> 81.3 mm
- net /DIODE_OR_OUT: track 4.06 -> 0.00 mm
- net Net-(C5-Pad1): track 3.02 -> 0.00 mm
- net /PowerProtection/source: track 7.93 -> 5.38 mm
- net /12VBB_VOUT: track 14.8 -> 12.3 mm
- added copper zone on F.Cu, net Net-(IC3-ISP)

Commit message: idealdiodeschematic
Parts:
- moved J7 5.05 mm to (207.7, 220.6), turned to 180 degrees
- moved F1 3.90 mm to (139.1, 211.0)
- moved R43 1.56 mm to (192.7, 219.1)
- moved C3 1.04 mm to (145.3, 195.9)
Routing:
- net /12VBB_VOUT: track 12.3 -> 24.9 mm
Changed lines of the file:
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@@
 	(footprint "Capacitor_SMD:C_0603_1608Metric_Pad1.08x0.95mm_HandSolder"
 		(layer "F.Cu")
-		(at 145.6 196.95 90)
+		(at 145.3 195.95 90)
 		(descr "Capacitor SMD 0603 (1608 Metric), square (rectangular) end terminal, IPC-7351 nominal with elongated pad for handsoldering. (Body size source: IPC-SM-782 page 76, https://www.pcb-3d.com/wordpress/wp-content/uploads/ipc-sm-782a_amendment_1_and_2.pdf)")
 		(tags "capacitor handsolder")
@@
 	(footprint "LHRS_Connectors:AMASS_XT30UPB-M_1x02_P5.0mm_Vertical"
 		(layer "F.Cu")
-		(at 203.5 217.75)
+		(at 207.7 220.55 180)
 		(descr "Connector XT30 Vertical PCB Male, https://www.tme.eu/en/Document/4acc913878197f8c2e30d4b8cdc47230/XT30UPB%20SPEC.pdf")
 		(tags "RC Connector XT30")
@@
 		(duplicate_pad_numbers_are_jumpers no)
 		(fp_line
-			(start -2.71 -1.41)
-			(end -2.71 1.41)
+			(start 7.71 -2.71)
+			(end 7.71 2.71)
 			(stroke
 				(width 0.12)
@@
 		)
 		(fp_line
-			(start -2.71 -1.41)
-			(end -1.01 -2.71)
+			(start -1.01 2.71)
+			(end 7.71 2.71)
 			(stroke
 				(width 0.12)
@@
 		)
 		(fp_line
-			(start -2.71 1.41)
-			(end -1.01 2.71)
+			(start -1.01 -2.71)
+			(end 7.71 -2.71)
 			(stroke
 				(width 0.12)
@@
 		)
 		(fp_line
-			(start -1.01 -2.71)
-			(end 7.71 -2.71)
+			(start -2.71 1.41)
+			(end -1.01 2.71)
 			(stroke
 				(width 0.12)
@@
 		)
 		(fp_line
-			(start -1.01 2.71)
-			(end 7.71 2.71)
+			(start -2.71 -1.41)
+			(end -1.01 -2.71)
 			(stroke
 				(width 0.12)
@@
 		)
 		(fp_line
-			(start 7.71 -2.71)
-			(end 7.71 2.71)
+			(start -2.71 -1.41)
+			(end -2.71 1.41)
 			(stroke
 				(width 0.12)
@@
 		)
 		(fp_line
-			(start -3.1 -1.8)
-			(end -3.1 1.8)
+			(start 8.1 -3.1)
+			(end 8.1 3.1)
 			(stroke
 				(width 0.05)
@@
 		)
 		(fp_line
-			(start -3.1 -1.8)
-			(end -1.4 -3.1)
+			(start -1.4 3.1)
+			(end 8.1 3.1)
 			(stroke
 				(width 0.05)
@@
 		)
 		(fp_line
-			(start -3.1 1.8)
-			(end -1.4 3.1)
+			(start -1.4 -3.1)
+			(end 8.1 -3.1)
 			(stroke
 				(width 0.05)
@@
 		)
 		(fp_line
-			(start -1.4 -3.1)
-			(end 8.1 -3.1)
+			(start -3.1 1.8)
+			(end -1.4 3.1)
 			(stroke
 				(width 0.05)
@@
 		)
 		(fp_line
-			(start -1.4 3.1)
-			(end 8.1 3.1)
+			(start -3.1 -1.8)
+			(end -1.4 -3.1)
 			(stroke
 				(width 0.05)
@@
 		)
 		(fp_line
-			(start 8.1 -3.1)
-			(end 8.1 3.1)
+			(start -3.1 -1.8)
+			(end -3.1 1.8)
 			(stroke
 				(width 0.05)
@@
 		)
 		(fp_line
-			(start -2.6 -1.3)
-			(end -2.6 1.3)
+			(start 7.6 -2.6)
+			(end 7.6 2.6)
 			(stroke
 				(width 0.1)
@@
 		)
 		(fp_line
-			(start -2.6 -1.3)
-			(end -0.9 -2.6)
+			(start -0.9 2.6)
+			(end 7.6 2.6)
 			(stroke
 				(width 0.1)
@@
 		)
 		(fp_line
-			(start -2.6 1.3)
-			(end -0.9 2.6)
+			(start -0.9 -2.6)
+			(end 7.6 -2.6)
 			(stroke
 				(width 0.1)
@@
 		)
 		(fp_line
-			(start -0.9 -2.6)
-			(end 7.6 -2.6)
+			(start -2.6 1.3)
+			(end -0.9 2.6)
 			(stroke
 				(width 0.1)
@@
 		)
 		(fp_line
-			(start -0.9 2.6)
-			(end 7.6 2.6)
+			(start -2.6 -1.3)
+			(end -0.9 -2.6)
 			(stroke
 				(width 0.1)
@@
 		)
 		(fp_line
-			(start 7.6 -2.6)
-			(end 7.6 2.6)
+			(start -2.6 -1.3)
+			(end -2.6 1.3)
 			(stroke
 				(width 0.1)
@@
 			(layer "F.Fab")
 		)
-		(fp_text user "-"
-			(at -4 0 0)
+		(fp_text user "+"
+			(at 9 0 0)
 			(layer "F.SilkS")
 			(effects
@@
 			)
 		)
-		(fp_text user "+"
-			(at 9 0 0)
+		(fp_text user "-"
+			(at -4 0 0)
 			(layer "F.SilkS")
 			(effects
@@
 		)
 		(pad "1" thru_hole rect
-			(at 0 0)
+			(at 0 0 180)
 			(size 3 3)
 			(drill 1.8)
@@
 		)
 		(pad "2" thru_hole circle
-			(at 5 0)
+			(at 5 0 180)
 			(size 3 3)
 			(drill 1.8)
@@
 	(footprint "PS-Supp-Footprints:PMR100HZPFU10L0"
 		(layer "F.Cu")
-		(at 192.75 217.5375)
+		(at 192.7 219.1)
 		(tags "PMR100HZPFU10L0 ")
 		(property "Reference" "R43"
@@
 			(polygon
 				(pts
-					(xy 191.3022 215.6833) (xy 194.1978 215.6833) (xy 194.1978 219.3917) (xy 191.3022 219.3917)
+					(xy 191.2522 217.2458) (xy 194.1478 217.2458) (xy 194.1478 220.9542) (xy 191.2522 220.9542)
 				)
 			)
@@
 	(footprint "LHRS_Power:Fuse-3557-2"
 		(layer "F.Cu")
-		(at 139.05 214.885 90)
+		(at 139.1 210.985 90)
 		(descr "3557-2")
 		(tags "Connector")
@@
 	)
 	(segment
-		(start 197.96875 215)
-		(end 197.994607 215)
-		(width 0.2)
-		(layer "F.Cu")
-		(net "+14.7V")
-	)
-	(segment
-		(start 201.457106 211.5375)
-		(end 202.925 211.5375)
+		(start 195.34795 214.85205)
+		(end 196.5 213.7)
 		(width 0.2)
 		(layer "F.Cu")
@@
 	)
 	(segment
-		(start 195.39795 217.5375)
-		(end 195.39795 213.65205)
+		(start 202.05 213.7)
+		(end 202.925 212.825)
 		(width 0.2)
 		(layer "F.Cu")
@@
 	)
 	(segment
-		(start 204.5 213.75)
-		(end 207.5 213.75)
-		(width 0.2)
-		(layer "F.Cu")
-		(net "+14.7V")
-	)
-	(segment
-		(start 195.95 213.1)
-		(end 198.15 213.1)
+		(start 195.34795 219.1)
+		(end 195.34795 214.85205)
 		(width 0.2)
 		(layer "F.Cu")
@@
 	)
 	(segment
-		(start 197.994607 215)
-		(end 201.457106 211.5375)
+		(start 204.5 213.75)
+		(end 207.5 213.75)
 		(width 0.2)
 		(layer "F.Cu")
@@
 	)
 	(segment
-		(start 195.39795 217.5375)
-		(end 195.43125 217.5375)
+		(start 196.5 213.7)
+		(end 202.05 213.7)
 		(width 0.2)
 		(layer "F.Cu")
@@
 	)
 	(segment
-		(start 202.925 212.175)
-		(end 204.5 213.75)
-		(width 0.2)
-		(layer "F.Cu")
-		(net "+14.7V")
-	)
-	(segment
-		(start 198.15 213.1)
-		(end 198.3 212.95)
+		(start 202.925 212.825)
+		(end 202.925 211.5375)
 		(width 0.2)
 		(layer "F.Cu")
@@
 	)
 	(segment
-		(start 195.39795 213.65205)
-		(end 195.95 213.1)
+		(start 202.925 212.175)
+		(end 204.5 213.75)
 		(width 0.2)
 		(layer "F.Cu")
@@
 	)
 	(segment
-		(start 195.642893 212.7)
-		(end 195.742894 212.6)
+		(start 201.9 212.45)
+		(end 201.9 206.475)
 		(width 0.2)
 		(layer "F.Cu")
@@
 	)
 	(segment
-		(start 195.742894 212.6)
-		(end 197.942894 212.6)
+		(start 190.05205 219.1)
+		(end 190.05205 214.19795)
 		(width 0.2)
 		(layer "F.Cu")
@@
 	)
 	(segment
-		(start 197.942894 212.6)
-		(end 198.092894 212.45)
+		(start 190.05205 214.19795)
+		(end 190.95 213.3)
 		(width 0.2)
 		(layer "F.Cu")
@@
 	)
 	(segment
-		(start 198.15 212.45)
-		(end 198.25 212.35)
+		(start 201.9 206.475)
+		(end 202.8375 205.5375)
 		(width 0.2)
 		(layer "F.Cu")
@@
 	)
 	(segment
-		(start 190.10205 217.5375)
-		(end 190.10205 214.34795)
+		(start 190.95 213.3)
+		(end 201.05 213.3)
 		(width 0.2)
 		(layer "F.Cu")
@@
 	)
 	(segment
-		(start 198.092894 212.45)
-		(end 198.15 212.45)
-		(width 0.2)
-		(layer "F.Cu")
-		(net "/12VBB_VOUT")
-	)
-	(segment
-		(start 191.75 212.7)
-		(end 195.642893 212.7)
-		(width 0.2)
-		(layer "F.Cu")
-		(net "/12VBB_VOUT")
-	)
-	(segment
-		(start 190.10205 214.34795)
-		(end 191.75 212.7)
+		(start 201.05 213.3)
+		(end 201.9 212.45)
 		(width 0.2)
 		(layer "F.Cu")
@@
 		(start 143.2625 175.6625)
 		(end 140.8125 173.2125)
-		(width 0.2)
+		(width 1)
 		(layer "F.Cu")
 		(net "/PD_5V_OUT")
@@
 		(start 144.3525 175.6625)
 		(end 143.2625 175.6625)
-		(width 0.2)
+		(width 1)
 		(layer "F.Cu")
 		(net "/PD_5V_OUT")
@@
 	)
 	(zone
-		(net "/PP_VIN")
+		(net "+14.7V")
 		(layer "F.Cu")
-		(name "PP_VIN")
+		(name "+14.7V")
 		(hatch edge 0.5)
-		(priority 1)
+		(priority 6)
 		(connect_pads yes
 			(clearance 0.5)
@@
 		(polygon
 			(pts
-				(xy 134.75 194.35777) (xy 149.5 194.35777) (xy 148.6 207.7) (xy 145.25 207.3) (xy 141 209.7) (xy 134.75 210.4)
+				(xy 193.4 217.15) (xy 205.3 217.15) (xy 205.3 224.4) (xy 197.8 224.4) (xy 193.4 224.4)
 			)
 		)
 	)
 	(zone
-		(net "+14.7V")
+		(net "Net-(IC3-ISP)")
 		(layer "F.Cu")
-		(name "+14.7V")
+		(name "Buck_Boost_OUT")
 		(hatch edge 0.5)
-		(priority 6)
+		(priority 14)
 		(connect_pads yes
 			(clearance 0.5)
@@
 			(thermal_gap 0.5)
 			(thermal_bridge_width 0.5)
-			(island_removal_mode 0)
+			(island_removal_mode 1)
 		)
 		(polygon
 			(pts
-				(xy 193.4 213.9) (xy 218.25 213.9) (xy 218.25 222) (xy 197.8 222) (xy 193.4 222)
+				(xy 159.2 212.6) (xy 159.2 210.15) (xy 176.2 210.15) (xy 176.2 212.6)
 			)
 		)
 	)
 	(zone
-		(net "Net-(IC3-ISP)")
+		(net "/PP_VIN")
 		(layer "F.Cu")
-		(name "Buck_Boost_OUT")
+		(name "PP_VIN")
 		(hatch edge 0.5)
-		(priority 14)
+		(priority 1)
 		(connect_pads yes
 			(clearance 0.5)
@@
 		(polygon
 			(pts
-				(xy 159.2 212.6) (xy 159.2 210.15) (xy 176.2 210.15) (xy 176.2 212.6)
+				(xy 138.85 195.75) (xy 138.85 201.3) (xy 135.45 201.3) (xy 135.45 207.6) (xy 149.6 207.6) (xy 149.6 195.75)
 			)
 		)
@@
 		(polygon
 			(pts
-				(xy 174.5 196.95) (xy 174.5 192.75) (xy 149.25 192.75) (xy 149.25 206.25) (xy 160.35 206.25) (xy 160.35 196.95)
+				(xy 174.5 196.95) (xy 174.5 192.75) (xy 149.6 192.75) (xy 149.6 206.25) (xy 160.35 206.25) (xy 160.35 196.95)
 			)
 		)
@@
 		(polygon
 			(pts
-				(xy 123.05 199.75) (xy 134.5 199.75) (xy 134.5 216.25) (xy 143.1 216.25) (xy 143.1 223) (xy 123.05 223)
+				(xy 123.05 203.15) (xy 132.2 203.15) (xy 136.05 211) (xy 143.1 214.3) (xy 143.1 221.25) (xy 123.05 221)
 			)
 		)

Commit message: fixedstuff
Parts:
- added C61: 0.1u, Capacitor_SMD:C_0603_1608Metric_Pad1.08x0.95mm_HandSolder, F.Cu at (179.2, 176.8)
- added C62: 0.1u, Capacitor_SMD:C_0603_1608Metric_Pad1.08x0.95mm_HandSolder, F.Cu at (176.2, 189.7)
- added Q8: NMOS, PS-Supp-Footprints:SOT95P237X112-3N, F.Cu at (177.5, 174.1)
- added Q9: NMOS, PS-Supp-Footprints:SOT95P237X112-3N, F.Cu at (171.4, 187.2)
- added R61: 100, Resistor_SMD:R_0603_1608Metric_Pad0.98x0.95mm_HandSolder, F.Cu at (182.7, 176.8)
- added R62: 100, Resistor_SMD:R_0603_1608Metric_Pad0.98x0.95mm_HandSolder, F.Cu at (180.4, 186.5)
- added U6: LTC4357HDCB-TRMPBF, PS-Supp-Footprints:DFN-6_DCB_LIT, F.Cu at (182.3, 174.1)
- added U7: LTC4357HDCB-TRMPBF, PS-Supp-Footprints:DFN-6_DCB_LIT, F.Cu at (176.0, 187.2)
- J5: footprint LHRS_Connectors:Molex_Nano-Fit_105313-xx02_1x02_P2.50mm_Horizontal -> LHRS_Connectors:Molex_Nano-Fit_105309-xx02_1x02_P2.50mm_Vertical
- moved NT1 74.9 mm to (183.0, 217.1), turned to 90 degrees
- moved R48 39.5 mm to (199.7, 134.6)
- moved TP13 31.5 mm to (142.9, 186.9)
- moved R2 30.1 mm to (197.7, 198.5), turned to 180 degrees
- moved J4 28.1 mm to (196.2, 134.6)
- moved R24 26.0 mm to (147.9, 190.2), turned to 180 degrees
- moved R34 25.9 mm to (172.0, 166.6), turned to -90 degrees
- moved C18 25.8 mm to (164.1, 161.2), turned to 0 degrees
- moved D2 24.7 mm to (197.7, 195.7), turned to 180 degrees
- moved D21 24.7 mm to (168.6, 164.5), turned to -90 degrees
- moved D18 24.7 mm to (149.9, 165.9), turned to 90 degrees
- moved TP1 24.5 mm to (132.0, 182.7), turned to -90 degrees
- moved TP14 24.2 mm to (140.8, 166.9), turned to 180 degrees
- moved TP12 23.1 mm to (142.7, 182.8)
- moved R26 23.0 mm to (151.7, 190.2), turned to 0 degrees
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Connections:
- H2 pad 1: /unconnected-(H2-Pad1)_1_1 -> unconnected-(H2-Pad1)_1
- H3 pad 1: /unconnected-(H3-Pad1)_2_2 -> unconnected-(H3-Pad1)_2
- H4 pad 1: /unconnected-(H4-Pad1)_2_2 -> unconnected-(H4-Pad1)_2
- J5 pad 2: GND -> /PS_VOUT
Routing:
- net /I2C_SCL: track 84.2 -> 3.32 mm
- net /I2C_SDA: track 72.5 -> 3.86 mm
- net +3V3: track 91.7 -> 27.8 mm
- net /INA_ALERT: track 65.8 -> 7.07 mm
- net /DIODE_OR_OUT: track 0.00 -> 45.6 mm
- net /PD_5V_OUT: track 81.3 -> 39.4 mm
- net /USB_VBUS: track 13.9 -> 0.00 mm
- net /PP_VOUT: track 0.00 -> 13.1 mm
- net +15V: track 2.97 -> 14.4 mm
- net /12VBuck/FB: track 11.0 -> 0.00 mm
- net /Power_Mux/PR1: track 14.0 -> 3.51 mm
- net /USB_D+: track 41.7 -> 34.8 mm
- net /USB_D-: track 41.0 -> 34.1 mm
- net Net-(IC3-FSW): track 0.00 -> 6.15 mm
- net Net-(Q8-G): track 0.00 -> 4.64 mm
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- removed copper zone on F.Cu, net /PD_5V_OUT
