File: DiodeOR.kicad_sch (KiCad schematic)
At the start: 8 parts, among them Q6 IRLML0030TRPBF, Q7 IRLML0030TRPBF, U6 LTC4357HDCB-TRMPBF, U7 LTC4357HDCB-TRMPBF

Commit message: fixedstuff
Parts:
- removed Q6, Q7: IRLML0030TRPBF, SOT95P237X112-3N, symbol PS-SuppCharger_Library:IRLML0030TRPBF
- added D12, D13: B540C-13-F, LHRS_Power:B540C-13-F, symbol lhrs_power:B540C-13-F
- added Q8, Q9: NMOS, PS-Supp-Footprints:SOT95P237X112-3N, symbol Simulation_SPICE:NMOS
- C61, C62: value C -> 0.1u; footprint (none) -> Capacitor_SMD:C_0603_1608Metric_Pad1.08x0.95mm_HandSolder
- R61, R62: value R -> 100; footprint (none) -> Resistor_SMD:R_0603_1608Metric_Pad0.98x0.95mm_HandSolder
- U6, U7: footprint DFN-6_DCB_LIT -> PS-Supp-Footprints:DFN-6_DCB_LIT
Connections:
- net DIODE_OR_OUT: now also D12.1 (K), D13.1 (K), Q8.1 (D), Q9.1 (D)
- net IN1: now also D12.2 (A), Q8.3 (S)
- net IN2: now also D13.2 (A), Q9.3 (S)
- net at U6.3 (GATE): now also Q8.2 (G)
- net at U7.3 (GATE): now also Q9.2 (G)
Other:
- note added: "RDS(ON) <= (0.1V)/(3A) RDS(ON) <= 33.3mΩ"
